Commit message: binit tests merging robot and dock at a coincident contacts_link (exists in docking_station.urdf) and charge_port_link (new in SE4, offset is y=18.5cm, z=10.7cm from base_link)

File: stretch4_urdf/SE4_accessories/docking_station/docking_station.urdf (robot description, URDF)
Before this commit: robot URDF_FRANCIS_ASSEM_Docking_Station_V1, 5 links, 4 joints
Joints:
- joint contacts_joint: child contacts_link -> docking_station_link; origin xyz=0 -0.0862 0.1335 rpy=0 0 0 -> xyz=0 0.0862 -0.1335 rpy=0 0 0; parent docking_station_link -> contacts_link

File: stretch4_urdf/SE4_francis/xacro/stretch_main.xacro (robot description, xacro)
@@ -28,4 +28,11 @@
     <parent link="base_footprint" />
     <child link="base_link" />
+    <axis xyz="0 0 0" />
+  </joint>
+  <link name="charge_port_link" />
+  <joint name="charge_port_joint" type="fixed">
+    <origin xyz="0 0.185 0.107" rpy="0 0 0" />
+    <parent link="base_link" />
+    <child link="charge_port_link" />
     <axis xyz="0 0 0" />
   </joint>
