Commit message: Tool URDF updates

File: stretch4_urdf/SE4_tools/eoa_wrist_dw4_tool_calibration/eoa_wrist_dw4_tool_calibration.urdf (robot description, URDF)
Before this commit: robot camera_calibration_board, 1 links, 0 joints
Links:
- link quick_connect_interface_link: geometry collision mesh filename=$(arg tool_mesh_dir)/quick_connect_interface_collision_link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; visual mesh filename=$(arg tool_mesh_dir)/quick_connect_interface_link.STL

File: stretch4_urdf/SE4_tools/eoa_wrist_dw4_tool_pg4/eoa_wrist_dw4_tool_pg4.urdf (robot description, URDF)
Before this commit: robot URDF_DALI_ASSEM_Parallel_Jaw_Gripper_V2, 7 links, 6 joints
Joints:
- joint aruco_fingertip_left_joint: origin xyz=-0.0670399 0.0122506 0.017 rpy=-1.57079 -1.57079 1.57079 -> xyz=-0.01225 -0.0670400491408859 0.0170000000000008 rpy=0 0 0
- joint aruco_fingertip_right_joint: origin xyz=-0.06704 -0.0122502 0.017 rpy=2.65359e-06 1.57079 3.14159 -> xyz=-0.0122499999999998 0.0670400491408858 0.0169999999999987 rpy=0 0 -3.14159265358979
- joint finger_left_joint: axis 0 0 1 -> 1 0 0; origin xyz=0 0.16686 0 rpy=0 0 1.5708 -> xyz=0.166855269271506 0 0 rpy=0 0 -1.5707963267949
- joint finger_right_joint: axis 0 0 1 -> 1 0 0; origin xyz=0 0.16686 0 rpy=0 0 1.5708 -> xyz=0.166855269271506 0 0 rpy=0 0 1.5707963267949
- joint grasp_frame_joint: origin xyz=0 0.166855 0 rpy=0 0 3.67321e-06 -> xyz=0.166855269271506 0 0 rpy=0 0 0
- joint quick_connect_interface_joint: origin xyz=0 0 0 rpy=0 0 -1.5708 -> xyz=0 0 0 rpy=0 0 0

File: stretch4_urdf/SE4_tools/eoa_wrist_dw4_tool_sg4/eoa_wrist_dw4_tool_sg4.urdf (robot description, URDF)
Before this commit: robot URDF_DALI_ASSEM_Stretch_Gripper_V4, 8 links, 7 joints
Links:
- link aruco_fingertip_left_link: mass 0.000123521493853862 -> 0.000123521493853863
- link gripper_finger_left_link: mass 0.0196491261592472 -> 0.0196452088457427
- link gripper_finger_right_link: mass 0.0196451967584484 -> 0.0196451967584486
- link gripper_fingertip_left_link: mass 0.0147998681120424 -> 0.0155504911063414
- link gripper_fingertip_right_link: mass 0.0147998807271023 -> 0.0155505328279169
- link quick_connect_interface_link: mass 0.0917733059735497 -> 0.268266992833353
Joints:
- joint aruco_fingertip_left_joint: origin xyz=0.0335358 0.00675395 3.80134e-05 rpy=1.37881 -2.50583e-06 0.62832 -> xyz=-0.00441710992520833 -0.0320457043432331 0 rpy=1.37881010907552 0 0.698131700797736
- joint aruco_fingertip_right_joint: origin xyz=-0.0335357 0.00675413 3.81175e-05 rpy=1.37881 1.8123e-06 2.51327 -> xyz=-0.00441710992520835 0.0320457043432331 0 rpy=1.37881010907552 0 2.44346095279206
- joint grasp_center_joint: origin xyz=0.234538 0 0 rpy=0 0 -1.5708 -> xyz=0.23496234568483 0 0 rpy=0 0 0
- joint gripper_finger_left_joint: axis 0 1 0 -> 0 -1 0; limit lower=0.0 upper=0.5 effort=0 velocity=0 -> lower=-0.5 upper=0 effort=0 velocity=0; origin xyz=0.0373909 0.0222607 0 rpy=1.5708 0 3.14159 -> xyz=0.0377995041255282 0.0221213818384166 0 rpy=1.5707963267949 0 -1.5707963267949
- joint gripper_finger_right_joint: limit lower=0.0 upper=0.5 effort=0 velocity=0 -> lower=0 upper=0.5 effort=0 velocity=0; origin xyz=0.0373909 -0.0222607 0 rpy=1.5708 0 3.14159 -> xyz=0.0377995041255281 -0.0221213818384166 0 rpy=1.5707963267949 0 -1.5707963267949
- joint gripper_fingertip_left_joint: origin xyz=-0.191008 0 -0.022168 rpy=-1.5708 2.65359e-06 0 -> xyz=0.0221679999883927 0 -0.191008332164325 rpy=-1.5707963267949 0.279252680319088 0
- joint gripper_fingertip_right_joint: origin xyz=-0.191008 0 0.022168 rpy=1.5708 -2.65359e-06 3.14159 -> xyz=-0.0221679999883885 0 -0.191008332164326 rpy=1.5707963267949 0.279252680319109 -3.14159265358979

File: stretch4_urdf/SE4_tools/eoa_wrist_dw4_tool_tablet/eoa_wrist_dw4_tool_tablet.urdf (robot description, URDF)
Before this commit: robot URDF_DALI_ASSEM_Tablet_Mount_V3, 1 links, 0 joints
Links:
- link quick_connect_interface_link: mass 0.774816112828515 -> 0.755969840555698
