Commit message: Finger frame corrections for sg4

File: stretch4_urdf/SE4_tools/eoa_wrist_dw4_tool_sg4/eoa_wrist_dw4_tool_sg4.urdf (robot description, URDF)
Before this commit: robot URDF_FRANCIS_ASSEM_Stretch_Gripper_V3, 8 links, 7 joints
Links:
- link gripper_finger_left_link: mass 0.0196452088457427 -> 0.0196452088457426
- link quick_connect_interface_link: mass 0.268266992833353 -> 0.268266990446664
Joints:
- joint gripper_finger_left_joint: axis 0 -1 0 -> 0 0 1; limit lower=-0.5 upper=0 effort=0 velocity=0 -> lower=0 upper=0.5 effort=0 velocity=0; origin xyz=0.0377995041255282 0.0221213818384166 0 rpy=1.5707963267949 0 -1.5707963267949 -> xyz=0.0378 0.022121 0 rpy=0 0 0
- joint gripper_finger_right_joint: axis 0 -1 0 -> 0 0 1; origin xyz=0.0377995041255281 -0.0221213818384166 0 rpy=1.5707963267949 0 -1.5707963267949 -> xyz=0.0377995041255281 -0.0221213818384166 0 rpy=3.14159265358979 0 0
- joint gripper_fingertip_left_joint: origin xyz=0.0221679999883927 0 -0.191008332164325 rpy=-1.5707963267949 0.279252680319088 0 -> xyz=0.191008332164325 -0.0221679999883927 0 rpy=0 0 -1.29154364647581
- joint gripper_fingertip_right_joint: origin xyz=-0.0221679999883885 0 -0.191008332164326 rpy=1.5707963267949 0.279252680319109 -3.14159265358979 -> xyz=0.191008332164326 -0.0221679999883885 0 rpy=3.14159265358979 0 -1.29154364647579
