Commit message: Bugfix for link ordering

File: stretch4_urdf/SE4_francis/xacro/stretch_main.xacro (robot description, xacro)
@@ -17,5 +17,5 @@
       </material>
     </visual>
-    <collision name="base_collision_link">
+      <collision name="base_collision_link">
       <origin xyz="0 0 0" rpy="0 0 0" />
       <geometry>
@@ -23,5 +23,5 @@
       </geometry>
     </collision>
-  </link>
+</link>
   <joint name="base_ref" type="fixed">
     <origin xyz="0 0 0.028" rpy="0 0 0" />
@@ -171,5 +171,5 @@
       </material>
     </visual>
-    <collision name="head_collision_link">
+      <collision name="head_collision_link">
       <origin xyz="0 0 0" rpy="0 0 0" />
       <geometry>
@@ -177,5 +177,5 @@
       </geometry>
     </collision>
-  </link>
+</link>
   <joint name="head_joint" type="fixed">
     <origin xyz="-0.093 -0.098 1.559" rpy="0 0 0" />
@@ -224,12 +224,4 @@
   </joint>
   <link name="camera_right_optical_link">
-    <visual>
-      <origin xyz="0 0 0" rpy="0 0 3.14159" />
-      <geometry>
-        <box size="0.001 0.001 0.001" /></geometry>
-      <material name="">
-        <color rgba="0.752941176470588 0.752941176470588 0.752941176470588 1" />
-      </material>
-    </visual>
     </link>
   <joint name="camera_right_optical_joint" type="fixed">
@@ -253,12 +245,4 @@
   </joint>
   <link name="camera_left_optical_link">
-    <visual>
-      <origin xyz="0 0 0" rpy="0 0 0" />
-      <geometry>
-        <box size="0.001 0.001 0.001" /></geometry>
-      <material name="">
-        <color rgba="0.752941176470588 0.752941176470588 0.752941176470588 1" />
-      </material>
-    </visual>
     </link>
   <joint name="camera_left_optical_joint" type="fixed">
@@ -282,12 +266,4 @@
   </joint>
   <link name="camera_center_optical_link">
-    <visual>
-      <origin xyz="0 0 0" rpy="0 0 -3.14159" />
-      <geometry>
-        <box size="0.001 0.001 0.001" /></geometry>
-      <material name="">
-        <color rgba="0.792156862745098 0.819607843137255 0.933333333333333 1" />
-      </material>
-    </visual>
     </link>
   <joint name="camera_center_optical_joint" type="fixed">
@@ -354,5 +330,5 @@
     <limit lower="0" upper="1.2" effort="0" velocity="0" />
   </joint>
-  <link name="arm_l0_link">
+  <link name="arm_l4_link">
     <inertial>
       <origin xyz="0.0146277 -0.0397927 0.0182873" rpy="0 1.5708 0" />
@@ -369,5 +345,5 @@
       </material>
     </visual>
-    <collision name="arm_l0_collision_link">
+    <collision name="arm_l4_collision_link">
       <origin xyz="0 0 0" rpy="0 1.5708 0" />
       <geometry>
@@ -376,11 +352,11 @@
     </collision>
   </link>
-  <joint name="arm_l0_joint" type="fixed">
+  <joint name="arm_l4_joint" type="fixed">
     <origin xyz="-0.0295 0.0994 -0.0128595" rpy="0 0 0" />
     <parent link="lift_link" />
-    <child link="arm_l0_link" />
-    <axis xyz="0 0 0" />
-  </joint>
-  <link name="arm_l1_link">
+    <child link="arm_l4_link" />
+    <axis xyz="0 0 0" />
+  </joint>
+  <link name="arm_l3_link">
     <inertial>
       <origin xyz="0.125319 0 0.00214616" rpy="0 1.5708 0" />
@@ -397,77 +373,77 @@
       </material>
     </visual>
+    <collision name="arm_l3_collision_link">
+      <origin xyz="0 0 0" rpy="0 1.5708 0" />
+      <geometry>
+        <mesh filename="$(arg model_mesh_dir)/arm_l3_collision_link.STL" />
+      </geometry>
+    </collision>
+  </link>
+  <joint name="arm_l3_joint" type="prismatic">
+    <origin xyz="0.0055 0 0" rpy="0 0 0" />
+    <parent link="arm_l4_link" />
+    <child link="arm_l3_link" />
+    <axis xyz="1 0 0" />
+    <limit lower="0" upper="0.13" effort="0" velocity="0" />
+  </joint>
+  <link name="arm_l2_link">
+    <inertial>
+      <origin xyz="0.126545 0 0.00212533" rpy="0 1.5708 0" />
+      <mass value="0.197181391808907" />
+      <inertia ixx="0.000701571828521803" ixy="1.70789035181299E-21" ixz="-1.56735722682992E-10" iyy="0.000676905139492615" iyz="1.0639178603614E-19" izz="0.000180704361161813" />
+    </inertial>
+    <visual>
+      <origin xyz="0 0 0" rpy="0 1.5708 0" />
+      <geometry>
+        <mesh filename="$(arg model_mesh_dir)/arm_l2_link.STL" />
+      </geometry>
+      <material name="">
+        <color rgba="0.752941176470588 0.752941176470588 0.752941176470588 1" />
+      </material>
+    </visual>
+    <collision name="arm_l2_collision_link">
+      <origin xyz="0 0 0" rpy="0 1.5708 0" />
+      <geometry>
+        <mesh filename="$(arg model_mesh_dir)/arm_l2_collision_link.STL" />
+      </geometry>
+    </collision>
+  </link>
+  <joint name="arm_l2_joint" type="prismatic">
+    <origin xyz="0.0135 0 0" rpy="0 0 0" />
+    <parent link="arm_l3_link" />
+    <child link="arm_l2_link" />
+    <axis xyz="1 0 0" />
+    <limit lower="0" upper="0.13" effort="0" velocity="0" />
+  </joint>
+  <link name="arm_l1_link">
+    <inertial>
+      <origin xyz="0.127806 0 0.00210076" rpy="0 1.5708 0" />
+      <mass value="0.182379618165529" />
+      <inertia ixx="0.000644687237937216" ixy="1.17464040780326E-20" ixz="-1.68878152441466E-10" iyy="0.00062371110107317" iyz="2.14435350061523E-19" izz="0.000140464382352664" />
+    </inertial>
+    <visual>
+      <origin xyz="0 0 0" rpy="0 1.5708 0" />
+      <geometry>
+        <mesh filename="$(arg model_mesh_dir)/arm_l1_link.STL" />
+      </geometry>
+      <material name="">
+        <color rgba="0.752941176470588 0.752941176470588 0.752941176470588 1" />
+      </material>
+    </visual>
     <collision name="arm_l1_collision_link">
       <origin xyz="0 0 0" rpy="0 1.5708 0" />
       <geometry>
-        <mesh filename="$(arg model_mesh_dir)/arm_l3_collision_link.STL" />
+        <mesh filename="$(arg model_mesh_dir)/arm_l1_collision_link.STL" />
       </geometry>
     </collision>
   </link>
   <joint name="arm_l1_joint" type="prismatic">
-    <origin xyz="0.0055 0 0" rpy="0 0 0" />
-    <parent link="arm_l0_link" />
+    <origin xyz="0.0135 0 0" rpy="0 0 0" />
+    <parent link="arm_l2_link" />
     <child link="arm_l1_link" />
     <axis xyz="1 0 0" />
     <limit lower="0" upper="0.13" effort="0" velocity="0" />
   </joint>
-  <link name="arm_l2_link">
-    <inertial>
-      <origin xyz="0.126545 0 0.00212533" rpy="0 1.5708 0" />
-      <mass value="0.197181391808907" />
-      <inertia ixx="0.000701571828521803" ixy="1.70789035181299E-21" ixz="-1.56735722682992E-10" iyy="0.000676905139492615" iyz="1.0639178603614E-19" izz="0.000180704361161813" />
-    </inertial>
-    <visual>
-      <origin xyz="0 0 0" rpy="0 1.5708 0" />
-      <geometry>
-        <mesh filename="$(arg model_mesh_dir)/arm_l2_link.STL" />
-      </geometry>
-      <material name="">
-        <color rgba="0.752941176470588 0.752941176470588 0.752941176470588 1" />
-      </material>
-    </visual>
-    <collision name="arm_l2_collision_link">
-      <origin xyz="0 0 0" rpy="0 1.5708 0" />
-      <geometry>
-        <mesh filename="$(arg model_mesh_dir)/arm_l2_collision_link.STL" />
-      </geometry>
-    </collision>
-  </link>
-  <joint name="arm_l2_joint" type="prismatic">
-    <origin xyz="0.0135 0 0" rpy="0 0 0" />
-    <parent link="arm_l1_link" />
-    <child link="arm_l2_link" />
-    <axis xyz="1 0 0" />
-    <limit lower="0" upper="0.13" effort="0" velocity="0" />
-  </joint>
-  <link name="arm_l3_link">
-    <inertial>
-      <origin xyz="0.127806 0 0.00210076" rpy="0 1.5708 0" />
-      <mass value="0.182379618165529" />
-      <inertia ixx="0.000644687237937216" ixy="1.17464040780326E-20" ixz="-1.68878152441466E-10" iyy="0.00062371110107317" iyz="2.14435350061523E-19" izz="0.000140464382352664" />
-    </inertial>
-    <visual>
-      <origin xyz="0 0 0" rpy="0 1.5708 0" />
-      <geometry>
-        <mesh filename="$(arg model_mesh_dir)/arm_l1_link.STL" />
-      </geometry>
-      <material name="">
-        <color rgba="0.752941176470588 0.752941176470588 0.752941176470588 1" />
-      </material>
-    </visual>
-    <collision name="arm_l3_collision_link">
-      <origin xyz="0 0 0" rpy="0 1.5708 0" />
-      <geometry>
-        <mesh filename="$(arg model_mesh_dir)/arm_l1_collision_link.STL" />
-      </geometry>
-    </collision>
-  </link>
-  <joint name="arm_l3_joint" type="prismatic">
-    <origin xyz="0.0135 0 0" rpy="0 0 0" />
-    <parent link="arm_l2_link" />
-    <child link="arm_l3_link" />
-    <axis xyz="1 0 0" />
-    <limit lower="0" upper="0.13" effort="0" velocity="0" />
-  </joint>
-  <link name="arm_l4_link">
+  <link name="arm_l0_link">
     <inertial>
       <origin xyz="0.105 0 0.00206007" rpy="0 1.5708 0" />
@@ -484,5 +460,5 @@
       </material>
     </visual>
-    <collision name="arm_l4_collision_link">
+    <collision name="arm_l0_collision_link">
       <origin xyz="0 0 0" rpy="0 1.5708 0" />
       <geometry>
@@ -491,8 +467,8 @@
     </collision>
   </link>
-  <joint name="arm_l4_joint" type="prismatic">
+  <joint name="arm_l0_joint" type="prismatic">
     <origin xyz="0.01375 0 0" rpy="0 0 0" />
-    <parent link="arm_l3_link" />
-    <child link="arm_l4_link" />
+    <parent link="arm_l1_link" />
+    <child link="arm_l0_link" />
     <axis xyz="1 0 0" />
     <limit lower="0" upper="0.13" effort="0" velocity="0" />
@@ -522,5 +498,5 @@
   <joint name="wrist_joint" type="fixed">
     <origin xyz="0.24715 0 -0.03672" rpy="0 0 0" />
-    <parent link="arm_l4_link" />
+    <parent link="arm_l0_link" />
     <child link="wrist_link" />
     <axis xyz="0 0 0" />
@@ -615,10 +591,10 @@
   <link name="gripper_camera_link">
     <inertial>
-      <origin xyz="0.00250349 0.0120203 0" rpy="1.5708 0 -1.5708" />
+      <origin xyz="0 0.0120203 -0.00250349" rpy="0 0 -1.5708" />
       <mass value="0.0447759731526001" />
       <inertia ixx="1.60232107304684E-05" ixy="-8.65767518586304E-22" ixz="2.63946367478605E-08" iyy="6.92267971098109E-06" iyz="-6.09577361235966E-22" izz="1.36247235159961E-05" />
     </inertial>
     <visual>
-      <origin xyz="0 0 0" rpy="1.5708 0 -1.5708" />
+      <origin xyz="0 0 0" rpy="0 0 -1.5708" />
       <geometry>
         <mesh filename="$(arg model_mesh_dir)/gripper_camera_link.STL" />
@@ -628,13 +604,13 @@
       </material>
     </visual>
-    <collision name="gripper_camera_link_collision">
-      <origin xyz="0 0 0" rpy="1.5708 0 -1.5708" />
-      <geometry>
-        <mesh filename="$(arg model_mesh_dir)/gripper_camera_link_collision.STL" />
+    <collision name="gripper_camera_collision_link">
+      <origin xyz="0 0 0" rpy="0 0 -1.5708" />
+      <geometry>
+        <mesh filename="$(arg model_mesh_dir)/gripper_camera_collision_link.STL" />
       </geometry>
     </collision>
   </link>
   <joint name="gripper_camera_joint" type="fixed">
-    <origin xyz="0.0192 0 0.057" rpy="1.5708 -1.5708 0" />
+    <origin xyz="0.0192 0 0.057" rpy="-3.14159 0 -1.5708" />
     <parent link="wrist_roll_link" />
     <child link="gripper_camera_link" />
@@ -643,5 +619,5 @@
   <link name="gripper_stereo_camera_color_optical_frame">
     <visual>
-      <origin xyz="0 0 0" rpy="1.5708 0 1.5708" />
+      <origin xyz="0 0 0" rpy="0 0 1.5708" />
       <geometry>
         <box size="0.001 0.001 0.001" /></geometry>
@@ -659,5 +635,5 @@
   <link name="gripper_right_camera_color_optical_frame">
     <visual>
-      <origin xyz="0 0 0" rpy="1.5708 0 1.5708" />
+      <origin xyz="0 0 0" rpy="0 0 1.5708" />
       <geometry>
         <box size="0.001 0.001 0.001" /></geometry>
@@ -668,5 +644,5 @@
     </link>
   <joint name="gripper_right_camera_color_optical_joint" type="fixed">
-    <origin xyz="0 0 0.01" rpy="3.14159 0 0" />
+    <origin xyz="0.01 0 0" rpy="3.14159 0 0" />
     <parent link="gripper_camera_link" />
     <child link="gripper_right_camera_color_optical_frame" />
@@ -675,5 +651,5 @@
   <link name="gripper_left_camera_color_optical_frame">
     <visual>
-      <origin xyz="0 0 0" rpy="1.5708 0 1.5708" />
+      <origin xyz="0 0 0" rpy="0 0 1.5708" />
       <geometry>
         <box size="0.001 0.001 0.001" /></geometry>
@@ -684,5 +660,5 @@
     </link>
   <joint name="gripper_left_camera_color_optical_joint" type="fixed">
-    <origin xyz="0 0 -0.01" rpy="3.14159 0 0" />
+    <origin xyz="-0.01 0 0" rpy="3.14159 0 0" />
     <parent link="gripper_camera_link" />
     <child link="gripper_left_camera_color_optical_frame" />
