Commit message: Optical and sensor frame updates

File: stretch4_urdf/SE4_francis/xacro/stretch_main.xacro (robot description, xacro)
@@ -1,10 +1,18 @@
 <robot xmlns:xacro="http://www.ros.org/wiki/xacro" name="stretch">
   <link name="base_footprint">
+    <visual>
+      <origin xyz="0 0 0" rpy="0 0 0" />
+      <geometry>
+        <box size="0.001 0.001 0.001" /></geometry>
+      <material name="">
+        <color rgba="0.752941176470588 0.752941176470588 0.752941176470588 1" />
+      </material>
+    </visual>
     </link>
   <link name="base_link">
     <inertial>
-      <origin xyz="0.000438847979969877 -0.00177714773743115 0.096468369649182" rpy="0 0 0" />
-      <mass value="18.9261042191254" />
-      <inertia ixx="0.21499266597667" ixy="0.000833860434673384" ixz="-0.000588719185658632" iyy="0.223010418927279" iyz="-0.00155067412786978" izz="0.327845794874634" />
+      <origin xyz="0.000438847979959605 -0.00177714773743784 0.0964683588787771" rpy="0 0 0" />
+      <mass value="18.9261042191275" />
+      <inertia ixx="0.214992665976689" ixy="0.000833860434661022" ixz="-0.000588719185644055" iyy="0.223010418927309" iyz="-0.00155067412786045" izz="0.327845794874662" />
     </inertial>
     <visual>
@@ -17,5 +25,5 @@
       </material>
     </visual>
-      <collision name="base_collision_link">
+    <collision name="base_collision_link">
       <origin xyz="0 0 0" rpy="0 0 0" />
       <geometry>
@@ -23,5 +31,5 @@
       </geometry>
     </collision>
-</link>
+  </link>
   <joint name="base_ref" type="fixed">
     <origin xyz="0 0 0.028" rpy="0 0 0" />
@@ -32,11 +40,26 @@
   <link name="line_sensor_5_link">
     <inertial>
-      <origin xyz="0.00114502070313138 0.0119761602719027 0.000126774756058469" rpy="0 0 0" />
+      <origin xyz="0.00324936 0.00537451 0.0102622" rpy="1.5708 0.453786 1.0472" />
       <mass value="0.00213836003346436" />
-      <inertia ixx="2.88698160050487E-07" ixy="-7.07831726662329E-09" ixz="5.64135957062393E-10" iyy="6.64615782289848E-08" iyz="2.73972720709968E-10" izz="2.34959277592962E-07" />
-    </inertial>
+      <inertia ixx="2.88698160050487E-07" ixy="-7.07831726662329E-09" ixz="5.64135957062429E-10" iyy="6.64615782289849E-08" iyz="2.73972720709955E-10" izz="2.34959277592962E-07" />
+    </inertial>
+    <visual>
+      <origin xyz="0 0 0" rpy="1.5708 0.453786 1.0472" />
+      <geometry>
+        <mesh filename="$(arg model_mesh_dir)/line_sensor_5_link.STL" />
+      </geometry>
+      <material name="">
+        <color rgba="0.792156862745098 0.819607843137255 0.933333333333333 1" />
+      </material>
+    </visual>
+    <collision name="line_sensor_5_collision_link">
+      <origin xyz="0 0 0" rpy="1.5708 0.453786 1.0472" />
+      <geometry>
+        <mesh filename="$(arg model_mesh_dir)/line_sensor_5_link.STL" />
+      </geometry>
+    </collision>
   </link>
   <joint name="line_sensor_5_joint" type="fixed">
-    <origin xyz="0.0613832 0.178319 0.0527014" rpy="1.5708 0.453786 1.0472" />
+    <origin xyz="0.0613832 0.178319 0.0527014" rpy="0 0 0" />
     <parent link="base_link" />
     <child link="line_sensor_5_link" />
@@ -44,7 +67,15 @@
   </joint>
   <link name="line_sensor_5_optical_link">
+    <visual>
+      <origin xyz="0 0 0" rpy="0.247888 -0.46609 2.62868" />
+      <geometry>
+        <box size="0.001 0.001 0.001" /></geometry>
+      <material name="">
+        <color rgba="0.792156862745098 0.819607843137255 0.933333333333333 1" />
+      </material>
+    </visual>
     </link>
   <joint name="line_sensor_5_optical_joint" type="fixed">
-    <origin xyz="0.00286 0 0" rpy="-1.5708 0 -1.5708" />
+    <origin xyz="0.00128528 0.00222616 -0.00125374" rpy="-1.5708 0 -1.5708" />
     <parent link="line_sensor_5_link" />
     <child link="line_sensor_5_optical_link" />
@@ -53,11 +84,26 @@
   <link name="line_sensor_4_link">
     <inertial>
-      <origin xyz="0.00114502070313141 0.0119761602719027 0.000126774756058476" rpy="0 0 0" />
+      <origin xyz="-0.00302978 0.00550128 0.0102622" rpy="1.5708 0.453786 2.0944" />
       <mass value="0.00213836003346436" />
-      <inertia ixx="2.88698160050488E-07" ixy="-7.07831726662323E-09" ixz="5.64135957060038E-10" iyy="6.6461578228985E-08" iyz="2.73972720708377E-10" izz="2.34959277592962E-07" />
-    </inertial>
+      <inertia ixx="2.88698160050488E-07" ixy="-7.07831726662323E-09" ixz="5.64135957060017E-10" iyy="6.6461578228985E-08" iyz="2.73972720708404E-10" izz="2.34959277592962E-07" />
+    </inertial>
+    <visual>
+      <origin xyz="0 0 0" rpy="1.5708 0.453786 2.0944" />
+      <geometry>
+        <mesh filename="$(arg model_mesh_dir)/line_sensor_4_link.STL" />
+      </geometry>
+      <material name="">
+        <color rgba="0.792156862745098 0.819607843137255 0.933333333333333 1" />
+      </material>
+    </visual>
+    <collision name="line_sensor_4_collision_link">
+      <origin xyz="0 0 0" rpy="1.5708 0.453786 2.0944" />
+      <geometry>
+        <mesh filename="$(arg model_mesh_dir)/line_sensor_4_link.STL" />
+      </geometry>
+    </collision>
   </link>
   <joint name="line_sensor_4_joint" type="fixed">
-    <origin xyz="-0.0613832 0.178319 0.0527014" rpy="1.5708 0.453786 2.0944" />
+    <origin xyz="-0.0613832 0.178319 0.0527014" rpy="0 0 0" />
     <parent link="base_link" />
     <child link="line_sensor_4_link" />
@@ -65,7 +111,15 @@
   </joint>
   <link name="line_sensor_4_optical_link">
+    <visual>
+      <origin xyz="0 0 0" rpy="-0.247888 0.46609 2.62868" />
+      <geometry>
+        <box size="0.001 0.001 0.001" /></geometry>
+      <material name="">
+        <color rgba="0.792156862745098 0.819607843137255 0.933333333333333 1" />
+      </material>
+    </visual>
     </link>
   <joint name="line_sensor_4_optical_joint" type="fixed">
-    <origin xyz="0.00286 0 0" rpy="-1.5708 0 -1.5708" />
+    <origin xyz="-0.00128528 0.00222616 -0.00125374" rpy="-1.5708 0 -1.5708" />
     <parent link="line_sensor_4_link" />
     <child link="line_sensor_4_optical_link" />
@@ -74,11 +128,26 @@
   <link name="line_sensor_3_link">
     <inertial>
-      <origin xyz="0.00114502070313155 0.0119761602719025 0.000126774756058573" rpy="0 0 0" />
+      <origin xyz="-0.00627914 0.000126775 0.0102622" rpy="1.5708 0.453786 -3.14159" />
       <mass value="0.00213836003346444" />
-      <inertia ixx="2.88698160050477E-07" ixy="-7.07831726660265E-09" ixz="5.64135957061257E-10" iyy="6.64615782289998E-08" iyz="2.73972720709266E-10" izz="2.34959277592965E-07" />
-    </inertial>
+      <inertia ixx="2.88698160050477E-07" ixy="-7.07831726660264E-09" ixz="5.64135957061256E-10" iyy="6.64615782289998E-08" iyz="2.73972720709257E-10" izz="2.34959277592965E-07" />
+    </inertial>
+    <visual>
+      <origin xyz="0 0 0" rpy="1.5708 0.453786 -3.14159" />
+      <geometry>
+        <mesh filename="$(arg model_mesh_dir)/line_sensor_3_link.STL" />
+      </geometry>
+      <material name="">
+        <color rgba="0.792156862745098 0.819607843137255 0.933333333333333 1" />
+      </material>
+    </visual>
+    <collision name="line_sensor_3_collision_link">
+      <origin xyz="0 0 0" rpy="1.5708 0.453786 -3.14159" />
+      <geometry>
+        <mesh filename="$(arg model_mesh_dir)/line_sensor_3_link.STL" />
+      </geometry>
+    </collision>
   </link>
   <joint name="line_sensor_3_joint" type="fixed">
-    <origin xyz="-0.18512 -0.036 0.0527014" rpy="1.5708 0.453786 -3.14159" />
+    <origin xyz="-0.18512 -0.036 0.0527014" rpy="0 0 0" />
     <parent link="base_link" />
     <child link="line_sensor_3_link" />
@@ -86,7 +155,15 @@
   </joint>
   <link name="line_sensor_3_optical_link">
+    <visual>
+      <origin xyz="0 0 0" rpy="-1.5708 1.11701 1.5708" />
+      <geometry>
+        <box size="0.001 0.001 0.001" /></geometry>
+      <material name="">
+        <color rgba="0.792156862745098 0.819607843137255 0.933333333333333 1" />
+      </material>
+    </visual>
     </link>
   <joint name="line_sensor_3_optical_joint" type="fixed">
-    <origin xyz="0.00286 0 0" rpy="-1.5708 0 -1.5708" />
+    <origin xyz="-0.00257055 0 -0.00125374" rpy="-1.5708 0 -1.5708" />
     <parent link="line_sensor_3_link" />
     <child link="line_sensor_3_optical_link" />
@@ -95,11 +172,26 @@
   <link name="line_sensor_2_link">
     <inertial>
-      <origin xyz="0.00114502070313149 0.0119761602719027 0.000126774756058545" rpy="0 0 0" />
+      <origin xyz="-0.00324936 -0.00537451 0.0102622" rpy="1.5708 0.453786 -2.0944" />
       <mass value="0.00213836003346437" />
-      <inertia ixx="2.88698160050489E-07" ixy="-7.07831726662341E-09" ixz="5.64135957062458E-10" iyy="6.64615782289852E-08" iyz="2.73972720710036E-10" izz="2.34959277592963E-07" />
-    </inertial>
+      <inertia ixx="2.88698160050488E-07" ixy="-7.07831726662343E-09" ixz="5.64135957062436E-10" iyy="6.64615782289851E-08" iyz="2.73972720710034E-10" izz="2.34959277592963E-07" />
+    </inertial>
+    <visual>
+      <origin xyz="0 0 0" rpy="1.5708 0.453786 -2.0944" />
+      <geometry>
+        <mesh filename="$(arg model_mesh_dir)/line_sensor_2_link.STL" />
+      </geometry>
+      <material name="">
+        <color rgba="0.792156862745098 0.819607843137255 0.933333333333333 1" />
+      </material>
+    </visual>
+    <collision name="line_sensor_2_collision_link">
+      <origin xyz="0 0 0" rpy="1.5708 0.453786 -2.0944" />
+      <geometry>
+        <mesh filename="$(arg model_mesh_dir)/line_sensor_2_link.STL" />
+      </geometry>
+    </collision>
   </link>
   <joint name="line_sensor_2_joint" type="fixed">
-    <origin xyz="-0.123737 -0.142319 0.0527014" rpy="1.5708 0.453786 -2.0944" />
+    <origin xyz="-0.123737 -0.142319 0.0527014" rpy="0 0 0" />
     <parent link="base_link" />
     <child link="line_sensor_2_link" />
@@ -107,7 +199,15 @@
   </joint>
   <link name="line_sensor_2_optical_link">
+    <visual>
+      <origin xyz="0 0 0" rpy="-2.8937 0.46609 0.51291" />
+      <geometry>
+        <box size="0.001 0.001 0.001" /></geometry>
+      <material name="">
+        <color rgba="0.792156862745098 0.819607843137255 0.933333333333333 1" />
+      </material>
+    </visual>
     </link>
   <joint name="line_sensor_2_optical_joint" type="fixed">
-    <origin xyz="0.00286 0 0" rpy="-1.5708 0 -1.5708" />
+    <origin xyz="-0.00128528 -0.00222616 -0.00125374" rpy="-1.5708 0 -1.5708" />
     <parent link="line_sensor_2_link" />
     <child link="line_sensor_2_optical_link" />
@@ -116,11 +216,26 @@
   <link name="line_sensor_1_link">
     <inertial>
-      <origin xyz="0.00114502070313141 0.0119761602719026 0.000126774756058601" rpy="0 0 0" />
+      <origin xyz="0.00302978 -0.00550128 0.0102622" rpy="1.5708 0.453786 -1.0472" />
       <mass value="0.00213836003346436" />
-      <inertia ixx="2.88698160050487E-07" ixy="-7.07831726662332E-09" ixz="5.6413595706002E-10" iyy="6.64615782289848E-08" iyz="2.73972720708439E-10" izz="2.34959277592961E-07" />
-    </inertial>
+      <inertia ixx="2.88698160050487E-07" ixy="-7.07831726662329E-09" ixz="5.64135957059983E-10" iyy="6.64615782289849E-08" iyz="2.73972720708449E-10" izz="2.34959277592962E-07" />
+    </inertial>
+    <visual>
+      <origin xyz="0 0 0" rpy="1.5708 0.453786 -1.0472" />
+      <geometry>
+        <mesh filename="$(arg model_mesh_dir)/line_sensor_1_link.STL" />
+      </geometry>
+      <material name="">
+        <color rgba="0.792156862745098 0.819607843137255 0.933333333333333 1" />
+      </material>
+    </visual>
+    <collision name="line_sensor_1_collision_link">
+      <origin xyz="0 0 0" rpy="1.5708 0.453786 -1.0472" />
+      <geometry>
+        <mesh filename="$(arg model_mesh_dir)/line_sensor_1_link.STL" />
+      </geometry>
+    </collision>
   </link>
   <joint name="line_sensor_1_joint" type="fixed">
-    <origin xyz="0.123737 -0.142319 0.0527014" rpy="1.5708 0.453786 -1.0472" />
+    <origin xyz="0.123737 -0.142319 0.0527014" rpy="0 0 0" />
     <parent link="base_link" />
     <child link="line_sensor_1_link" />
@@ -128,7 +243,15 @@
   </joint>
   <link name="line_sensor_1_optical_link">
+    <visual>
+      <origin xyz="0 0 0" rpy="2.8937 -0.46609 0.51291" />
+      <geometry>
+        <box size="0.001 0.001 0.001" /></geometry>
+      <material name="">
+        <color rgba="0.792156862745098 0.819607843137255 0.933333333333333 1" />
+      </material>
+    </visual>
     </link>
   <joint name="line_sensor_1_optical_joint" type="fixed">
-    <origin xyz="0.00286 0 0" rpy="-1.5708 0 -1.5708" />
+    <origin xyz="0.00128528 -0.00222616 -0.00125374" rpy="-1.5708 0 -1.5708" />
     <parent link="line_sensor_1_link" />
     <child link="line_sensor_1_optical_link" />
@@ -137,11 +260,26 @@
   <link name="line_sensor_0_link">
     <inertial>
-      <origin xyz="0.00114502070313233 0.0119761602719029 0.000126774756058746" rpy="0 0 0" />
+      <origin xyz="0.00627914 -0.000126775 0.0102622" rpy="1.5708 0.453786 0" />
       <mass value="0.00213836003346444" />
-      <inertia ixx="2.88698160050477E-07" ixy="-7.07831726660256E-09" ixz="5.6413595706126E-10" iyy="6.64615782290001E-08" iyz="2.73972720709193E-10" izz="2.34959277592965E-07" />
-    </inertial>
+      <inertia ixx="2.88698160050477E-07" ixy="-7.07831726660252E-09" ixz="5.64135957061258E-10" iyy="6.64615782290001E-08" iyz="2.73972720709191E-10" izz="2.34959277592965E-07" />
+    </inertial>
+    <visual>
+      <origin xyz="0 0 0" rpy="1.5708 0.453786 0" />
+      <geometry>
+        <mesh filename="$(arg model_mesh_dir)/line_sensor_0_link.STL" />
+      </geometry>
+      <material name="">
+        <color rgba="0.792156862745098 0.819607843137255 0.933333333333333 1" />
+      </material>
+    </visual>
+    <collision name="line_sensor_0_collision_link">
+      <origin xyz="0 0 0" rpy="1.5708 0.453786 0" />
+      <geometry>
+        <mesh filename="$(arg model_mesh_dir)/line_sensor_0_link.STL" />
+      </geometry>
+    </collision>
   </link>
   <joint name="line_sensor_0_joint" type="fixed">
-    <origin xyz="0.18512 -0.036 0.0527014" rpy="1.5708 0.453786 0" />
+    <origin xyz="0.18512 -0.036 0.0527014" rpy="0 0 0" />
     <parent link="base_link" />
     <child link="line_sensor_0_link" />
@@ -149,7 +287,15 @@
   </joint>
   <link name="line_sensor_0_optical_link">
+    <visual>
+      <origin xyz="0 0 0" rpy="1.5708 -1.11701 1.5708" />
+      <geometry>
+        <box size="0.001 0.001 0.001" /></geometry>
+      <material name="">
+        <color rgba="0.792156862745098 0.819607843137255 0.933333333333333 1" />
+      </material>
+    </visual>
     </link>
   <joint name="line_sensor_0_optical_joint" type="fixed">
-    <origin xyz="0.00286 0 0" rpy="-1.5708 0 -1.5708" />
+    <origin xyz="0.00257055 0 -0.00125374" rpy="-1.5708 0 -1.5708" />
     <parent link="line_sensor_0_link" />
     <child link="line_sensor_0_optical_link" />
@@ -158,7 +304,7 @@
   <link name="head_link">
     <inertial>
-      <origin xyz="0.0514013580104842 0.0986460644909709 -0.0250866227521696" rpy="0 0 0" />
-      <mass value="5.12944639372071" />
-      <inertia ixx="0.0380731695781352" ixy="0.000202619198715346" ixz="0.000237956614656072" iyy="0.0304351984631137" iyz="5.6169841247061E-05" izz="0.0637978570860214" />
+      <origin xyz="0.0578831464809341 0.0985910077817881 -0.0270263436790745" rpy="0 0 0" />
+      <mass value="5.618435167362" />
+      <inertia ixx="0.0382731622122869" ixy="0.000202623919235895" ixz="0.000231642202175719" iyy="0.0306326706365949" iyz="5.61616354648268E-05" izz="0.0640020784749226" />
     </inertial>
     <visual>
@@ -171,5 +317,5 @@
       </material>
     </visual>
-      <collision name="head_collision_link">
+    <collision name="head_collision_link">
       <origin xyz="0 0 0" rpy="0 0 0" />
       <geometry>
@@ -177,5 +323,5 @@
       </geometry>
     </collision>
-</link>
+  </link>
   <joint name="head_joint" type="fixed">
     <origin xyz="-0.093 -0.098 1.559" rpy="0 0 0" />
@@ -186,11 +332,26 @@
   <link name="lidar_right_link">
     <inertial>
-      <origin xyz="-3.20916615947908E-07 0.000175557811368021 -0.0150548418051187" rpy="0 0 0" />
-      <mass value="0.240802480448075" />
-      <inertia ixx="9.8041898749052E-05" ixy="4.48636958766777E-09" ixz="-3.11098715595503E-10" iyy="9.67162435587801E-05" iyz="1.39381302162429E-06" izz="0.000105657113395344" />
-    </inertial>
+      <origin xyz="0.031314 0.125004 0.0737134" rpy="-2.1317 -0.54633 2.53998" />
+      <mass value="5.62562911534835" />
+      <inertia ixx="0.0492829862682945" ixy="-0.00156447943074778" ixz="0.0149316960757035" iyy="0.0349356510816738" iyz="0.00380036130478219" izz="0.0486907192495753" />
+    </inertial>
+    <visual>
+      <origin xyz="0 0 0" rpy="-2.1317 -0.54633 2.53998" />
+      <geometry>
+        <mesh filename="$(arg model_mesh_dir)/lidar_right_link.STL" />
+      </geometry>
+      <material name="">
+        <color rgba="0.752941176470588 0.752941176470588 0.752941176470588 1" />
+      </material>
+    </visual>
+    <collision name="lidar_right_collision_link">
+      <origin xyz="0 0 0" rpy="-2.1317 -0.54633 2.53998" />
+      <geometry>
+        <mesh filename="$(arg model_mesh_dir)/lidar_right_link.STL" />
+      </geometry>
+    </collision>
   </link>
   <joint name="lidar_right_joint" type="fixed">
-    <origin xyz="0.131744 -0.0264137 -0.058328" rpy="-3.05466 0.7816 2.39203" />
+    <origin xyz="0.131744 -0.0264137 -0.058328" rpy="0 -1.5708 0" />
     <parent link="head_link" />
     <child link="lidar_right_link" />
@@ -199,11 +360,26 @@
   <link name="lidar_left_link">
     <inertial>
-      <origin xyz="-3.87815889180132E-07 0.000175565758143037 -0.0150548416196863" rpy="0 0 0" />
-      <mass value="0.240802531963034" />
-      <inertia ixx="9.80418920755826E-05" ixy="4.46941117355771E-09" ixz="-3.09741336789929E-10" iyy="9.67162544690224E-05" iyz="1.39381215337495E-06" izz="0.000105657115998718" />
-    </inertial>
+      <origin xyz="0.031314 0.123823 -0.0737134" rpy="1.00989 -0.54633 -0.601617" />
+      <mass value="5.62562911534835" />
+      <inertia ixx="0.0495631509325281" ixy="0.00150375861955282" ixz="-0.0147241234027668" iyy="0.0345419854283597" iyz="0.00388339874340473" izz="0.0488042202386559" />
+    </inertial>
+    <visual>
+      <origin xyz="0 0 0" rpy="1.00989 -0.54633 -0.601617" />
+      <geometry>
+        <mesh filename="$(arg model_mesh_dir)/lidar_left_link.STL" />
+      </geometry>
+      <material name="">
+        <color rgba="0.752941176470588 0.752941176470588 0.752941176470588 1" />
+      </material>
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