Commit message: Processing script refactor

File: stretch4_urdf/SE4_francis/xacro/stretch_main.xacro (robot description, xacro)
@@ -40,10 +40,10 @@
   <link name="line_sensor_5_link">
     <inertial>
-      <origin xyz="0.00324936 0.00537451 0.0102622" rpy="1.5708 0.453786 1.0472" />
+      <origin xyz="0.00114502 0.000126775 -0.0119762" rpy="1.5708 0 0" />
       <mass value="0.00213836003346436" />
       <inertia ixx="2.88698160050487E-07" ixy="-7.07831726662329E-09" ixz="5.64135957062429E-10" iyy="6.64615782289849E-08" iyz="2.73972720709955E-10" izz="2.34959277592962E-07" />
     </inertial>
     <visual>
-      <origin xyz="0 0 0" rpy="1.5708 0.453786 1.0472" />
+      <origin xyz="0 0 0" rpy="1.5708 0 0" />
       <geometry>
         <mesh filename="$(arg model_mesh_dir)/line_sensor_5_link.STL" />
@@ -54,5 +54,5 @@
     </visual>
     <collision name="line_sensor_5_collision_link">
-      <origin xyz="0 0 0" rpy="1.5708 0.453786 1.0472" />
+      <origin xyz="0 0 0" rpy="1.5708 0 0" />
       <geometry>
         <mesh filename="$(arg model_mesh_dir)/line_sensor_5_link.STL" />
@@ -61,5 +61,5 @@
   </link>
   <joint name="line_sensor_5_joint" type="fixed">
-    <origin xyz="0.0613832 0.178319 0.0527014" rpy="0 0 0" />
+    <origin xyz="0.0613832 0.178319 0.0527014" rpy="0 0.453786 1.0472" />
     <parent link="base_link" />
     <child link="line_sensor_5_link" />
@@ -68,5 +68,5 @@
   <link name="line_sensor_5_optical_link">
     <visual>
-      <origin xyz="0 0 0" rpy="0.247888 -0.46609 2.62868" />
+      <origin xyz="0 0 0" rpy="-3.14159 -1.5708 0" />
       <geometry>
         <box size="0.001 0.001 0.001" /></geometry>
@@ -77,5 +77,5 @@
     </link>
   <joint name="line_sensor_5_optical_joint" type="fixed">
-    <origin xyz="0.00128528 0.00222616 -0.00125374" rpy="-1.5708 0 -1.5708" />
+    <origin xyz="0.00286 0 0" rpy="-1.5708 0 -1.5708" />
     <parent link="line_sensor_5_link" />
     <child link="line_sensor_5_optical_link" />
@@ -84,10 +84,10 @@
   <link name="line_sensor_4_link">
     <inertial>
-      <origin xyz="-0.00302978 0.00550128 0.0102622" rpy="1.5708 0.453786 2.0944" />
+      <origin xyz="0.00114502 0.000126775 -0.0119762" rpy="1.5708 0 0" />
       <mass value="0.00213836003346436" />
       <inertia ixx="2.88698160050488E-07" ixy="-7.07831726662323E-09" ixz="5.64135957060017E-10" iyy="6.6461578228985E-08" iyz="2.73972720708404E-10" izz="2.34959277592962E-07" />
     </inertial>
     <visual>
-      <origin xyz="0 0 0" rpy="1.5708 0.453786 2.0944" />
+      <origin xyz="0 0 0" rpy="1.5708 0 0" />
       <geometry>
         <mesh filename="$(arg model_mesh_dir)/line_sensor_4_link.STL" />
@@ -98,5 +98,5 @@
     </visual>
     <collision name="line_sensor_4_collision_link">
-      <origin xyz="0 0 0" rpy="1.5708 0.453786 2.0944" />
+      <origin xyz="0 0 0" rpy="1.5708 0 0" />
       <geometry>
         <mesh filename="$(arg model_mesh_dir)/line_sensor_4_link.STL" />
@@ -105,5 +105,5 @@
   </link>
   <joint name="line_sensor_4_joint" type="fixed">
-    <origin xyz="-0.0613832 0.178319 0.0527014" rpy="0 0 0" />
+    <origin xyz="-0.0613832 0.178319 0.0527014" rpy="0 0.453786 2.0944" />
     <parent link="base_link" />
     <child link="line_sensor_4_link" />
@@ -112,5 +112,5 @@
   <link name="line_sensor_4_optical_link">
     <visual>
-      <origin xyz="0 0 0" rpy="-0.247888 0.46609 2.62868" />
+      <origin xyz="0 0 0" rpy="3.14159 -1.5708 0" />
       <geometry>
         <box size="0.001 0.001 0.001" /></geometry>
@@ -121,5 +121,5 @@
     </link>
   <joint name="line_sensor_4_optical_joint" type="fixed">
-    <origin xyz="-0.00128528 0.00222616 -0.00125374" rpy="-1.5708 0 -1.5708" />
+    <origin xyz="0.00286 0 0" rpy="-1.5708 0 -1.5708" />
     <parent link="line_sensor_4_link" />
     <child link="line_sensor_4_optical_link" />
@@ -128,10 +128,10 @@
   <link name="line_sensor_3_link">
     <inertial>
-      <origin xyz="-0.00627914 0.000126775 0.0102622" rpy="1.5708 0.453786 -3.14159" />
+      <origin xyz="0.00114502 0.000126775 -0.0119762" rpy="1.5708 0 0" />
       <mass value="0.00213836003346444" />
       <inertia ixx="2.88698160050477E-07" ixy="-7.07831726660264E-09" ixz="5.64135957061256E-10" iyy="6.64615782289998E-08" iyz="2.73972720709257E-10" izz="2.34959277592965E-07" />
     </inertial>
     <visual>
-      <origin xyz="0 0 0" rpy="1.5708 0.453786 -3.14159" />
+      <origin xyz="0 0 0" rpy="1.5708 0 0" />
       <geometry>
         <mesh filename="$(arg model_mesh_dir)/line_sensor_3_link.STL" />
@@ -142,5 +142,5 @@
     </visual>
     <collision name="line_sensor_3_collision_link">
-      <origin xyz="0 0 0" rpy="1.5708 0.453786 -3.14159" />
+      <origin xyz="0 0 0" rpy="1.5708 0 0" />
       <geometry>
         <mesh filename="$(arg model_mesh_dir)/line_sensor_3_link.STL" />
@@ -149,5 +149,5 @@
   </link>
   <joint name="line_sensor_3_joint" type="fixed">
-    <origin xyz="-0.18512 -0.036 0.0527014" rpy="0 0 0" />
+    <origin xyz="-0.18512 -0.036 0.0527014" rpy="0 0.453786 -3.14159" />
     <parent link="base_link" />
     <child link="line_sensor_3_link" />
@@ -156,5 +156,5 @@
   <link name="line_sensor_3_optical_link">
     <visual>
-      <origin xyz="0 0 0" rpy="-1.5708 1.11701 1.5708" />
+      <origin xyz="0 0 0" rpy="-3.14159 -1.5708 0" />
       <geometry>
         <box size="0.001 0.001 0.001" /></geometry>
@@ -165,5 +165,5 @@
     </link>
   <joint name="line_sensor_3_optical_joint" type="fixed">
-    <origin xyz="-0.00257055 0 -0.00125374" rpy="-1.5708 0 -1.5708" />
+    <origin xyz="0.00286 0 0" rpy="-1.5708 0 -1.5708" />
     <parent link="line_sensor_3_link" />
     <child link="line_sensor_3_optical_link" />
@@ -172,10 +172,10 @@
   <link name="line_sensor_2_link">
     <inertial>
-      <origin xyz="-0.00324936 -0.00537451 0.0102622" rpy="1.5708 0.453786 -2.0944" />
+      <origin xyz="0.00114502 0.000126775 -0.0119762" rpy="1.5708 0 0" />
       <mass value="0.00213836003346437" />
       <inertia ixx="2.88698160050488E-07" ixy="-7.07831726662343E-09" ixz="5.64135957062436E-10" iyy="6.64615782289851E-08" iyz="2.73972720710034E-10" izz="2.34959277592963E-07" />
     </inertial>
     <visual>
-      <origin xyz="0 0 0" rpy="1.5708 0.453786 -2.0944" />
+      <origin xyz="0 0 0" rpy="1.5708 0 0" />
       <geometry>
         <mesh filename="$(arg model_mesh_dir)/line_sensor_2_link.STL" />
@@ -186,5 +186,5 @@
     </visual>
     <collision name="line_sensor_2_collision_link">
-      <origin xyz="0 0 0" rpy="1.5708 0.453786 -2.0944" />
+      <origin xyz="0 0 0" rpy="1.5708 0 0" />
       <geometry>
         <mesh filename="$(arg model_mesh_dir)/line_sensor_2_link.STL" />
@@ -193,5 +193,5 @@
   </link>
   <joint name="line_sensor_2_joint" type="fixed">
-    <origin xyz="-0.123737 -0.142319 0.0527014" rpy="0 0 0" />
+    <origin xyz="-0.123737 -0.142319 0.0527014" rpy="0 0.453786 -2.0944" />
     <parent link="base_link" />
     <child link="line_sensor_2_link" />
@@ -200,5 +200,5 @@
   <link name="line_sensor_2_optical_link">
     <visual>
-      <origin xyz="0 0 0" rpy="-2.8937 0.46609 0.51291" />
+      <origin xyz="0 0 0" rpy="-3.14159 -1.5708 0" />
       <geometry>
         <box size="0.001 0.001 0.001" /></geometry>
@@ -209,5 +209,5 @@
     </link>
   <joint name="line_sensor_2_optical_joint" type="fixed">
-    <origin xyz="-0.00128528 -0.00222616 -0.00125374" rpy="-1.5708 0 -1.5708" />
+    <origin xyz="0.00286 0 0" rpy="-1.5708 0 -1.5708" />
     <parent link="line_sensor_2_link" />
     <child link="line_sensor_2_optical_link" />
@@ -216,10 +216,10 @@
   <link name="line_sensor_1_link">
     <inertial>
-      <origin xyz="0.00302978 -0.00550128 0.0102622" rpy="1.5708 0.453786 -1.0472" />
+      <origin xyz="0.00114502 0.000126775 -0.0119762" rpy="1.5708 0 0" />
       <mass value="0.00213836003346436" />
       <inertia ixx="2.88698160050487E-07" ixy="-7.07831726662329E-09" ixz="5.64135957059983E-10" iyy="6.64615782289849E-08" iyz="2.73972720708449E-10" izz="2.34959277592962E-07" />
     </inertial>
     <visual>
-      <origin xyz="0 0 0" rpy="1.5708 0.453786 -1.0472" />
+      <origin xyz="0 0 0" rpy="1.5708 0 0" />
       <geometry>
         <mesh filename="$(arg model_mesh_dir)/line_sensor_1_link.STL" />
@@ -230,5 +230,5 @@
     </visual>
     <collision name="line_sensor_1_collision_link">
-      <origin xyz="0 0 0" rpy="1.5708 0.453786 -1.0472" />
+      <origin xyz="0 0 0" rpy="1.5708 0 0" />
       <geometry>
         <mesh filename="$(arg model_mesh_dir)/line_sensor_1_link.STL" />
@@ -237,5 +237,5 @@
   </link>
   <joint name="line_sensor_1_joint" type="fixed">
-    <origin xyz="0.123737 -0.142319 0.0527014" rpy="0 0 0" />
+    <origin xyz="0.123737 -0.142319 0.0527014" rpy="0 0.453786 -1.0472" />
     <parent link="base_link" />
     <child link="line_sensor_1_link" />
@@ -244,5 +244,5 @@
   <link name="line_sensor_1_optical_link">
     <visual>
-      <origin xyz="0 0 0" rpy="2.8937 -0.46609 0.51291" />
+      <origin xyz="0 0 0" rpy="-3.14159 -1.5708 0" />
       <geometry>
         <box size="0.001 0.001 0.001" /></geometry>
@@ -253,5 +253,5 @@
     </link>
   <joint name="line_sensor_1_optical_joint" type="fixed">
-    <origin xyz="0.00128528 -0.00222616 -0.00125374" rpy="-1.5708 0 -1.5708" />
+    <origin xyz="0.00286 0 0" rpy="-1.5708 0 -1.5708" />
     <parent link="line_sensor_1_link" />
     <child link="line_sensor_1_optical_link" />
@@ -260,10 +260,10 @@
   <link name="line_sensor_0_link">
     <inertial>
-      <origin xyz="0.00627914 -0.000126775 0.0102622" rpy="1.5708 0.453786 0" />
+      <origin xyz="0.00114502 0.000126775 -0.0119762" rpy="1.5708 0 0" />
       <mass value="0.00213836003346444" />
       <inertia ixx="2.88698160050477E-07" ixy="-7.07831726660252E-09" ixz="5.64135957061258E-10" iyy="6.64615782290001E-08" iyz="2.73972720709191E-10" izz="2.34959277592965E-07" />
     </inertial>
     <visual>
-      <origin xyz="0 0 0" rpy="1.5708 0.453786 0" />
+      <origin xyz="0 0 0" rpy="1.5708 0 0" />
       <geometry>
         <mesh filename="$(arg model_mesh_dir)/line_sensor_0_link.STL" />
@@ -274,5 +274,5 @@
     </visual>
     <collision name="line_sensor_0_collision_link">
-      <origin xyz="0 0 0" rpy="1.5708 0.453786 0" />
+      <origin xyz="0 0 0" rpy="1.5708 0 0" />
       <geometry>
         <mesh filename="$(arg model_mesh_dir)/line_sensor_0_link.STL" />
@@ -281,5 +281,5 @@
   </link>
   <joint name="line_sensor_0_joint" type="fixed">
-    <origin xyz="0.18512 -0.036 0.0527014" rpy="0 0 0" />
+    <origin xyz="0.18512 -0.036 0.0527014" rpy="0 0.453786 0" />
     <parent link="base_link" />
     <child link="line_sensor_0_link" />
@@ -288,5 +288,5 @@
   <link name="line_sensor_0_optical_link">
     <visual>
-      <origin xyz="0 0 0" rpy="1.5708 -1.11701 1.5708" />
+      <origin xyz="0 0 0" rpy="-3.14159 -1.5708 0" />
       <geometry>
         <box size="0.001 0.001 0.001" /></geometry>
@@ -297,5 +297,5 @@
     </link>
   <joint name="line_sensor_0_optical_joint" type="fixed">
-    <origin xyz="0.00257055 0 -0.00125374" rpy="-1.5708 0 -1.5708" />
+    <origin xyz="0.00286 0 0" rpy="-1.5708 0 -1.5708" />
     <parent link="line_sensor_0_link" />
     <child link="line_sensor_0_optical_link" />
@@ -332,10 +332,10 @@
   <link name="lidar_right_link">
     <inertial>
-      <origin xyz="0.031314 0.125004 0.0737134" rpy="-2.1317 -0.54633 2.53998" />
+      <origin xyz="0.0766909447572703 0.0306840677846499 -0.12335811389925" rpy="0 0 0" />
       <mass value="5.62562911534835" />
       <inertia ixx="0.0492829862682945" ixy="-0.00156447943074778" ixz="0.0149316960757035" iyy="0.0349356510816738" iyz="0.00380036130478219" izz="0.0486907192495753" />
     </inertial>
     <visual>
-      <origin xyz="0 0 0" rpy="-2.1317 -0.54633 2.53998" />
+      <origin xyz="0 0 0" rpy="0 0 0" />
       <geometry>
         <mesh filename="$(arg model_mesh_dir)/lidar_right_link.STL" />
@@ -346,5 +346,5 @@
     </visual>
     <collision name="lidar_right_collision_link">
-      <origin xyz="0 0 0" rpy="-2.1317 -0.54633 2.53998" />
+      <origin xyz="0 0 0" rpy="0 0 0" />
       <geometry>
         <mesh filename="$(arg model_mesh_dir)/lidar_right_link.STL" />
@@ -353,5 +353,5 @@
   </link>
   <joint name="lidar_right_joint" type="fixed">
-    <origin xyz="0.131744 -0.0264137 -0.058328" rpy="0 -1.5708 0" />
+    <origin xyz="0.131744 -0.0264137 -0.058328" rpy="-3.05466 0.7816 2.39203" />
     <parent link="head_link" />
     <child link="lidar_right_link" />
@@ -360,10 +360,10 @@
   <link name="lidar_left_link">
     <inertial>
-      <origin xyz="0.031314 0.123823 -0.0737134" rpy="1.00989 -0.54633 -0.601617" />
+      <origin xyz="-0.0761200632210846 0.0298724102181261 -0.122718664121595" rpy="0 0 0" />
       <mass value="5.62562911534835" />
       <inertia ixx="0.0495631509325281" ixy="0.00150375861955282" ixz="-0.0147241234027668" iyy="0.0345419854283597" iyz="0.00388339874340473" izz="0.0488042202386559" />
     </inertial>
     <visual>
-      <origin xyz="0 0 0" rpy="1.00989 -0.54633 -0.601617" />
+      <origin xyz="0 0 0" rpy="0 0 0" />
       <geometry>
         <mesh filename="$(arg model_mesh_dir)/lidar_left_link.STL" />
@@ -374,5 +374,5 @@
     </visual>
     <collision name="lidar_left_collision_link">
-      <origin xyz="0 0 0" rpy="1.00989 -0.54633 -0.601617" />
+      <origin xyz="0 0 0" rpy="0 0 0" />
       <geometry>
         <mesh filename="$(arg model_mesh_dir)/lidar_left_link.STL" />
@@ -381,5 +381,5 @@
   </link>
   <joint name="lidar_left_joint" type="fixed">
-    <origin xyz="0.131744 0.222414 -0.058328" rpy="-3.14159 -1.5708 0" />
+    <origin xyz="0.131744 0.222414 -0.058328" rpy="-3.05466 -0.7816 0.749563" />
     <parent link="head_link" />
     <child link="lidar_left_link" />
@@ -388,10 +388,10 @@
   <link name="camera_right_link">
     <inertial>
-      <origin xyz="-0.11381 -0.0112573 -0.0755903" rpy="-1.5708 0 -2.3911" />
+      <origin xyz="0.0693851 0.0755903 0.0909127" rpy="0 1.5708 0" />
       <mass value="5.62562911534835" />
       <inertia ixx="0.0504717539490822" ixy="-0.000186491896655228" ixz="0.0128492795010695" iyy="0.0306330356066479" iyz="9.71151606421086E-05" izz="0.0518045670438135" />
     </inertial>
     <visual>
-      <origin xyz="0 0 0" rpy="-1.5708 0 -2.3911" />
+      <origin xyz="0 0 0" rpy="0 1.5708 0" />
       <geometry>
         <mesh filename="$(arg model_mesh_dir)/camera_right_link.STL" />
@@ -402,5 +402,5 @@
     </visual>
     <collision name="camera_right_collision_link">
-      <origin xyz="0 0 0" rpy="-1.5708 0 -2.3911" />
+      <origin xyz="0 0 0" rpy="0 1.5708 0" />
       <geometry>
         <mesh filename="$(arg model_mesh_dir)/camera_right_link.STL" />
@@ -409,5 +409,5 @@
   </link>
   <joint name="camera_right_joint" type="fixed">
-    <origin xyz="0.171841 0.023 -0.0157567" rpy="1.5708 0 0" />
+    <origin xyz="0.171841 0.023 -0.0157567" rpy="0 0.820305 0" />
     <parent link="head_link" />
     <child link="camera_right_link" />
@@ -416,5 +416,5 @@
   <link name="camera_right_optical_link">
     <visual>
-      <origin xyz="0 0 0" rpy="-0.820305 0 -1.5708" />
+      <origin xyz="0 0 0" rpy="0 0 1.5708" />
       <geometry>
         <box size="0.001 0.001 0.001" /></geometry>
@@ -425,5 +425,5 @@
     </link>
   <joint name="camera_right_optical_joint" type="fixed">
-    <origin xyz="0.0144584 -0.0155047 0" rpy="-1.5708 0 -1.5708" />
+    <origin xyz="0.0212 0 0" rpy="3.14159 -1.5708 0" />
     <parent link="camera_right_link" />
     <child link="camera_right_optical_link" />
@@ -432,10 +432,10 @@
   <link name="camera_left_link">
     <inertial>
-      <origin xyz="-0.11381 0.0112573 -0.0744097" rpy="-1.5708 0 -0.750492" />
+      <origin xyz="-0.0693851 -0.0744097 -0.0909127" rpy="3.14159 -1.5708 0" />
       <mass value="5.62562911534835" />
       <inertia ixx="0.0504717539490822" ixy="-0.000186491896655198" ixz="-0.0128492795010695" iyy="0.0306330356066479" iyz="-9.711516064215E-05" izz="0.0518045670438135" />
     </inertial>
     <visual>
-      <origin xyz="0 0 0" rpy="-1.5708 0 -0.750492" />
+      <origin xyz="0 0 0" rpy="3.14159 -1.5708 0" />
       <geometry>
         <mesh filename="$(arg model_mesh_dir)/camera_left_link.STL" />
@@ -446,5 +446,5 @@
     </visual>
     <collision name="camera_left_collision_link">
-      <origin xyz="0 0 0" rpy="-1.5708 0 -0.750492" />
+      <origin xyz="0 0 0" rpy="3.14159 -1.5708 0" />
       <geometry>
         <mesh filename="$(arg model_mesh_dir)/camera_left_link.STL" />
@@ -453,5 +453,5 @@
   </link>
   <joint name="camera_left_joint" type="fixed">
-    <origin xyz="0.171841 0.173 -0.0157567" rpy="-1.5708 0 0" />
+    <origin xyz="0.171841 0.173 -0.0157567" rpy="0 0.820305 0" />
     <parent link="head_link" />
     <child link="camera_left_link" />
@@ -460,5 +460,5 @@
   <link name="camera_left_optical_link">
     <visual>
-      <origin xyz="0 0 0" rpy="-0.820305 0 1.5708" />
+      <origin xyz="0 0 0" rpy="0 0 -1.5708" />
       <geometry>
         <box size="0.001 0.001 0.001" /></geometry>
@@ -469,5 +469,5 @@
     </link>
   <joint name="camera_left_optical_joint" type="fixed">
-    <origin xyz="0.0144584 0.0155047 0" rpy="-1.5708 0 -1.5708" />
+    <origin xyz="0.0212 0 0" rpy="0 1.5708 0" />
     <parent link="camera_left_link" />
     <child link="camera_left_optical_link" />
@@ -476,10 +476,10 @@
   <link name="camera_center_link">
     <inertial>
-      <origin xyz="-0.119215 -0.00310706 -0.000590252" rpy="1.5708 0 0.959931" />
+      <origin xyz="-0.0958729 0.000590252 -0.070924" rpy="3.14159 -1.5708 0" />
       <mass value="5.62562911534835" />
       <inertia ixx="0.0557556406323663" ixy="-0.000162225224016438" ixz="-0.0120094528841815" iyy="0.0306330356066479" iyz="-0.000133766806934365" izz="0.0465206803605294" />
     </inertial>
     <visual>
-      <origin xyz="0 0 0" rpy="1.5708 0 0.959931" />
+      <origin xyz="0 0 0" rpy="3.14159 -1.5708 0" />
       <geometry>
         <mesh filename="$(arg model_mesh_dir)/camera_center_link.STL" />
@@ -490,5 +490,5 @@
     </visual>
     <collision name="camera_center_collision_link">
-      <origin xyz="0 0 0" rpy="1.5708 0 0.959931" />
+      <origin xyz="0 0 0" rpy="3.14159 -1.5708 0" />
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