Commit message: camera frame fix

File: stretch4_urdf/SE4_francis/xacro/stretch_main.xacro (robot description, xacro)
@@ -1,12 +1,4 @@
 <robot xmlns:xacro="http://www.ros.org/wiki/xacro" name="stretch">
   <link name="base_footprint">
-    <visual>
-      <origin xyz="0 0 0" rpy="0 0 0" />
-      <geometry>
-        <box size="0.001 0.001 0.001" /></geometry>
-      <material name="">
-        <color rgba="0.752941176470588 0.752941176470588 0.752941176470588 1" />
-      </material>
-    </visual>
     </link>
   <link name="base_link">
@@ -19,5 +11,5 @@
       <origin xyz="0 0 0" rpy="0 0 0" />
       <geometry>
-        <mesh filename="$(arg model_mesh_dir)/base_link.obj" />
+        <mesh filename="$(arg model_mesh_dir)/base_link.OBJ" />
       </geometry>
       <material name="">
@@ -28,5 +20,5 @@
       <origin xyz="0 0 0" rpy="0 0 0" />
       <geometry>
-        <mesh filename="$(arg model_mesh_dir)/base_collision_link.obj" />
+        <mesh filename="$(arg model_mesh_dir)/base_collision_link.OBJ" />
       </geometry>
     </collision>
@@ -44,19 +36,4 @@
       <inertia ixx="2.88698160050487E-07" ixy="-7.07831726662329E-09" ixz="5.64135957062429E-10" iyy="6.64615782289849E-08" iyz="2.73972720709955E-10" izz="2.34959277592962E-07" />
     </inertial>
-    <visual>
-      <origin xyz="0 0 0" rpy="1.5708 0 0" />
-      <geometry>
-        <mesh filename="$(arg model_mesh_dir)/line_sensor_5_link.STL" />
-      </geometry>
-      <material name="">
-        <color rgba="0.792156862745098 0.819607843137255 0.933333333333333 1" />
-      </material>
-    </visual>
-    <collision name="line_sensor_5_collision_link">
-      <origin xyz="0 0 0" rpy="1.5708 0 0" />
-      <geometry>
-        <mesh filename="$(arg model_mesh_dir)/line_sensor_5_link.STL" />
-      </geometry>
-    </collision>
   </link>
   <joint name="line_sensor_5_joint" type="fixed">
@@ -67,12 +44,4 @@
   </joint>
   <link name="line_sensor_5_optical_link">
-    <visual>
-      <origin xyz="0 0 0" rpy="-3.14159 -1.5708 0" />
-      <geometry>
-        <box size="0.001 0.001 0.001" /></geometry>
-      <material name="">
-        <color rgba="0.792156862745098 0.819607843137255 0.933333333333333 1" />
-      </material>
-    </visual>
     </link>
   <joint name="line_sensor_5_optical_joint" type="fixed">
@@ -88,19 +57,4 @@
       <inertia ixx="2.88698160050488E-07" ixy="-7.07831726662323E-09" ixz="5.64135957060017E-10" iyy="6.6461578228985E-08" iyz="2.73972720708404E-10" izz="2.34959277592962E-07" />
     </inertial>
-    <visual>
-      <origin xyz="0 0 0" rpy="1.5708 0 0" />
-      <geometry>
-        <mesh filename="$(arg model_mesh_dir)/line_sensor_4_link.STL" />
-      </geometry>
-      <material name="">
-        <color rgba="0.792156862745098 0.819607843137255 0.933333333333333 1" />
-      </material>
-    </visual>
-    <collision name="line_sensor_4_collision_link">
-      <origin xyz="0 0 0" rpy="1.5708 0 0" />
-      <geometry>
-        <mesh filename="$(arg model_mesh_dir)/line_sensor_4_link.STL" />
-      </geometry>
-    </collision>
   </link>
   <joint name="line_sensor_4_joint" type="fixed">
@@ -111,12 +65,4 @@
   </joint>
   <link name="line_sensor_4_optical_link">
-    <visual>
-      <origin xyz="0 0 0" rpy="3.14159 -1.5708 0" />
-      <geometry>
-        <box size="0.001 0.001 0.001" /></geometry>
-      <material name="">
-        <color rgba="0.792156862745098 0.819607843137255 0.933333333333333 1" />
-      </material>
-    </visual>
     </link>
   <joint name="line_sensor_4_optical_joint" type="fixed">
@@ -132,19 +78,4 @@
       <inertia ixx="2.88698160050477E-07" ixy="-7.07831726660264E-09" ixz="5.64135957061256E-10" iyy="6.64615782289998E-08" iyz="2.73972720709257E-10" izz="2.34959277592965E-07" />
     </inertial>
-    <visual>
-      <origin xyz="0 0 0" rpy="1.5708 0 0" />
-      <geometry>
-        <mesh filename="$(arg model_mesh_dir)/line_sensor_3_link.STL" />
-      </geometry>
-      <material name="">
-        <color rgba="0.792156862745098 0.819607843137255 0.933333333333333 1" />
-      </material>
-    </visual>
-    <collision name="line_sensor_3_collision_link">
-      <origin xyz="0 0 0" rpy="1.5708 0 0" />
-      <geometry>
-        <mesh filename="$(arg model_mesh_dir)/line_sensor_3_link.STL" />
-      </geometry>
-    </collision>
   </link>
   <joint name="line_sensor_3_joint" type="fixed">
@@ -155,12 +86,4 @@
   </joint>
   <link name="line_sensor_3_optical_link">
-    <visual>
-      <origin xyz="0 0 0" rpy="-3.14159 -1.5708 0" />
-      <geometry>
-        <box size="0.001 0.001 0.001" /></geometry>
-      <material name="">
-        <color rgba="0.792156862745098 0.819607843137255 0.933333333333333 1" />
-      </material>
-    </visual>
     </link>
   <joint name="line_sensor_3_optical_joint" type="fixed">
@@ -176,19 +99,4 @@
       <inertia ixx="2.88698160050488E-07" ixy="-7.07831726662343E-09" ixz="5.64135957062436E-10" iyy="6.64615782289851E-08" iyz="2.73972720710034E-10" izz="2.34959277592963E-07" />
     </inertial>
-    <visual>
-      <origin xyz="0 0 0" rpy="1.5708 0 0" />
-      <geometry>
-        <mesh filename="$(arg model_mesh_dir)/line_sensor_2_link.STL" />
-      </geometry>
-      <material name="">
-        <color rgba="0.792156862745098 0.819607843137255 0.933333333333333 1" />
-      </material>
-    </visual>
-    <collision name="line_sensor_2_collision_link">
-      <origin xyz="0 0 0" rpy="1.5708 0 0" />
-      <geometry>
-        <mesh filename="$(arg model_mesh_dir)/line_sensor_2_link.STL" />
-      </geometry>
-    </collision>
   </link>
   <joint name="line_sensor_2_joint" type="fixed">
@@ -199,12 +107,4 @@
   </joint>
   <link name="line_sensor_2_optical_link">
-    <visual>
-      <origin xyz="0 0 0" rpy="-3.14159 -1.5708 0" />
-      <geometry>
-        <box size="0.001 0.001 0.001" /></geometry>
-      <material name="">
-        <color rgba="0.792156862745098 0.819607843137255 0.933333333333333 1" />
-      </material>
-    </visual>
     </link>
   <joint name="line_sensor_2_optical_joint" type="fixed">
@@ -220,19 +120,4 @@
       <inertia ixx="2.88698160050487E-07" ixy="-7.07831726662329E-09" ixz="5.64135957059983E-10" iyy="6.64615782289849E-08" iyz="2.73972720708449E-10" izz="2.34959277592962E-07" />
     </inertial>
-    <visual>
-      <origin xyz="0 0 0" rpy="1.5708 0 0" />
-      <geometry>
-        <mesh filename="$(arg model_mesh_dir)/line_sensor_1_link.STL" />
-      </geometry>
-      <material name="">
-        <color rgba="0.792156862745098 0.819607843137255 0.933333333333333 1" />
-      </material>
-    </visual>
-    <collision name="line_sensor_1_collision_link">
-      <origin xyz="0 0 0" rpy="1.5708 0 0" />
-      <geometry>
-        <mesh filename="$(arg model_mesh_dir)/line_sensor_1_link.STL" />
-      </geometry>
-    </collision>
   </link>
   <joint name="line_sensor_1_joint" type="fixed">
@@ -243,12 +128,4 @@
   </joint>
   <link name="line_sensor_1_optical_link">
-    <visual>
-      <origin xyz="0 0 0" rpy="-3.14159 -1.5708 0" />
-      <geometry>
-        <box size="0.001 0.001 0.001" /></geometry>
-      <material name="">
-        <color rgba="0.792156862745098 0.819607843137255 0.933333333333333 1" />
-      </material>
-    </visual>
     </link>
   <joint name="line_sensor_1_optical_joint" type="fixed">
@@ -264,19 +141,4 @@
       <inertia ixx="2.88698160050477E-07" ixy="-7.07831726660252E-09" ixz="5.64135957061258E-10" iyy="6.64615782290001E-08" iyz="2.73972720709191E-10" izz="2.34959277592965E-07" />
     </inertial>
-    <visual>
-      <origin xyz="0 0 0" rpy="1.5708 0 0" />
-      <geometry>
-        <mesh filename="$(arg model_mesh_dir)/line_sensor_0_link.STL" />
-      </geometry>
-      <material name="">
-        <color rgba="0.792156862745098 0.819607843137255 0.933333333333333 1" />
-      </material>
-    </visual>
-    <collision name="line_sensor_0_collision_link">
-      <origin xyz="0 0 0" rpy="1.5708 0 0" />
-      <geometry>
-        <mesh filename="$(arg model_mesh_dir)/line_sensor_0_link.STL" />
-      </geometry>
-    </collision>
   </link>
   <joint name="line_sensor_0_joint" type="fixed">
@@ -287,12 +149,4 @@
   </joint>
   <link name="line_sensor_0_optical_link">
-    <visual>
-      <origin xyz="0 0 0" rpy="-3.14159 -1.5708 0" />
-      <geometry>
-        <box size="0.001 0.001 0.001" /></geometry>
-      <material name="">
-        <color rgba="0.792156862745098 0.819607843137255 0.933333333333333 1" />
-      </material>
-    </visual>
     </link>
   <joint name="line_sensor_0_optical_joint" type="fixed">
@@ -336,19 +190,4 @@
       <inertia ixx="0.0492829862682945" ixy="-0.00156447943074778" ixz="0.0149316960757035" iyy="0.0349356510816738" iyz="0.00380036130478219" izz="0.0486907192495753" />
     </inertial>
-    <visual>
-      <origin xyz="0 0 0" rpy="0 0 0" />
-      <geometry>
-        <mesh filename="$(arg model_mesh_dir)/lidar_right_link.STL" />
-      </geometry>
-      <material name="">
-        <color rgba="0.752941176470588 0.752941176470588 0.752941176470588 1" />
-      </material>
-    </visual>
-    <collision name="lidar_right_collision_link">
-      <origin xyz="0 0 0" rpy="0 0 0" />
-      <geometry>
-        <mesh filename="$(arg model_mesh_dir)/lidar_right_link.STL" />
-      </geometry>
-    </collision>
   </link>
   <joint name="lidar_right_joint" type="fixed">
@@ -364,19 +203,4 @@
       <inertia ixx="0.0495631509325281" ixy="0.00150375861955282" ixz="-0.0147241234027668" iyy="0.0345419854283597" iyz="0.00388339874340473" izz="0.0488042202386559" />
     </inertial>
-    <visual>
-      <origin xyz="0 0 0" rpy="0 0 0" />
-      <geometry>
-        <mesh filename="$(arg model_mesh_dir)/lidar_left_link.STL" />
-      </geometry>
-      <material name="">
-        <color rgba="0.752941176470588 0.752941176470588 0.752941176470588 1" />
-      </material>
-    </visual>
-    <collision name="lidar_left_collision_link">
-      <origin xyz="0 0 0" rpy="0 0 0" />
-      <geometry>
-        <mesh filename="$(arg model_mesh_dir)/lidar_left_link.STL" />
-      </geometry>
-    </collision>
   </link>
   <joint name="lidar_left_joint" type="fixed">
@@ -388,26 +212,11 @@
   <link name="camera_right_link">
     <inertial>
-      <origin xyz="0.0693851 0.0755903 0.0909127" rpy="0 1.5708 0" />
+      <origin xyz="0.0755903 -0.0693851 0.0909127" rpy="1.5708 0 1.5708" />
       <mass value="5.62562911534835" />
       <inertia ixx="0.0504717539490822" ixy="-0.000186491896655228" ixz="0.0128492795010695" iyy="0.0306330356066479" iyz="9.71151606421086E-05" izz="0.0518045670438135" />
     </inertial>
-    <visual>
-      <origin xyz="0 0 0" rpy="0 1.5708 0" />
-      <geometry>
-        <mesh filename="$(arg model_mesh_dir)/camera_right_link.STL" />
-      </geometry>
-      <material name="">
-        <color rgba="0.752941176470588 0.752941176470588 0.752941176470588 1" />
-      </material>
-    </visual>
-    <collision name="camera_right_collision_link">
-      <origin xyz="0 0 0" rpy="0 1.5708 0" />
-      <geometry>
-        <mesh filename="$(arg model_mesh_dir)/camera_right_link.STL" />
-      </geometry>
-    </collision>
   </link>
   <joint name="camera_right_joint" type="fixed">
-    <origin xyz="0.171841 0.023 -0.0157567" rpy="0 0.820305 0" />
+    <origin xyz="0.171841 0.023 -0.0157567" rpy="-1.5708 0.820305 0" />
     <parent link="head_link" />
     <child link="camera_right_link" />
@@ -415,15 +224,7 @@
   </joint>
   <link name="camera_right_optical_link">
-    <visual>
-      <origin xyz="0 0 0" rpy="0 0 1.5708" />
-      <geometry>
-        <box size="0.001 0.001 0.001" /></geometry>
-      <material name="">
-        <color rgba="0.752941176470588 0.752941176470588 0.752941176470588 1" />
-      </material>
-    </visual>
     </link>
   <joint name="camera_right_optical_joint" type="fixed">
-    <origin xyz="0.0212 0 0" rpy="3.14159 -1.5708 0" />
+    <origin xyz="0.0212 0 0" rpy="-1.5708 0 -1.5708" />
     <parent link="camera_right_link" />
     <child link="camera_right_optical_link" />
@@ -432,26 +233,11 @@
   <link name="camera_left_link">
     <inertial>
-      <origin xyz="-0.0693851 -0.0744097 -0.0909127" rpy="3.14159 -1.5708 0" />
+      <origin xyz="0.0744097 -0.0693851 -0.0909127" rpy="1.5708 0 1.5708" />
       <mass value="5.62562911534835" />
       <inertia ixx="0.0504717539490822" ixy="-0.000186491896655198" ixz="-0.0128492795010695" iyy="0.0306330356066479" iyz="-9.711516064215E-05" izz="0.0518045670438135" />
     </inertial>
-    <visual>
-      <origin xyz="0 0 0" rpy="3.14159 -1.5708 0" />
-      <geometry>
-        <mesh filename="$(arg model_mesh_dir)/camera_left_link.STL" />
-      </geometry>
-      <material name="">
-        <color rgba="0.752941176470588 0.752941176470588 0.752941176470588 1" />
-      </material>
-    </visual>
-    <collision name="camera_left_collision_link">
-      <origin xyz="0 0 0" rpy="3.14159 -1.5708 0" />
-      <geometry>
-        <mesh filename="$(arg model_mesh_dir)/camera_left_link.STL" />
-      </geometry>
-    </collision>
   </link>
   <joint name="camera_left_joint" type="fixed">
-    <origin xyz="0.171841 0.173 -0.0157567" rpy="0 0.820305 0" />
+    <origin xyz="0.171841 0.173 -0.0157567" rpy="1.5708 0.820305 0" />
     <parent link="head_link" />
     <child link="camera_left_link" />
@@ -459,15 +245,7 @@
   </joint>
   <link name="camera_left_optical_link">
-    <visual>
-      <origin xyz="0 0 0" rpy="0 0 -1.5708" />
-      <geometry>
-        <box size="0.001 0.001 0.001" /></geometry>
-      <material name="">
-        <color rgba="0.752941176470588 0.752941176470588 0.752941176470588 1" />
-      </material>
-    </visual>
     </link>
   <joint name="camera_left_optical_joint" type="fixed">
-    <origin xyz="0.0212 0 0" rpy="0 1.5708 0" />
+    <origin xyz="0.0212 0 0" rpy="-1.5708 0 -1.5708" />
     <parent link="camera_left_link" />
     <child link="camera_left_optical_link" />
@@ -476,26 +254,11 @@
   <link name="camera_center_link">
     <inertial>
-      <origin xyz="-0.0958729 0.000590252 -0.070924" rpy="3.14159 -1.5708 0" />
+      <origin xyz="-0.000590252 -0.0958729 -0.070924" rpy="1.5708 0 1.5708" />
       <mass value="5.62562911534835" />
       <inertia ixx="0.0557556406323663" ixy="-0.000162225224016438" ixz="-0.0120094528841815" iyy="0.0306330356066479" iyz="-0.000133766806934365" izz="0.0465206803605294" />
     </inertial>
-    <visual>
-      <origin xyz="0 0 0" rpy="3.14159 -1.5708 0" />
-      <geometry>
-        <mesh filename="$(arg model_mesh_dir)/camera_center_link.STL" />
-      </geometry>
-      <material name="">
-        <color rgba="0.752941176470588 0.752941176470588 0.752941176470588 1" />
-      </material>
-    </visual>
-    <collision name="camera_center_collision_link">
-      <origin xyz="0 0 0" rpy="3.14159 -1.5708 0" />
-      <geometry>
-        <mesh filename="$(arg model_mesh_dir)/camera_center_link.STL" />
-      </geometry>
-    </collision>
   </link>
   <joint name="camera_center_joint" type="fixed">
-    <origin xyz="0.177246 0.098 -0.0239069" rpy="0 0.610865 0" />
+    <origin xyz="0.177246 0.098 -0.0239069" rpy="1.5708 0.610865 0" />
     <parent link="head_link" />
     <child link="camera_center_link" />
@@ -503,15 +266,7 @@
   </joint>
   <link name="camera_center_optical_link">
-    <visual>
-      <origin xyz="0 0 0" rpy="0 0 -1.5708" />
-      <geometry>
-        <box size="0.001 0.001 0.001" /></geometry>
-      <material name="">
-        <color rgba="0.752941176470588 0.752941176470588 0.752941176470588 1" />
-      </material>
-    </visual>
     </link>
   <joint name="camera_center_optical_joint" type="fixed">
-    <origin xyz="0.0017 0 0" rpy="0 1.5708 0" />
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
Commit message: Camera frame fixes

File: stretch4_urdf/SE4_francis/xacro/stretch_main.xacro (robot description, xacro)
@@ -212,5 +212,5 @@
   <link name="camera_right_link">
     <inertial>
-      <origin xyz="0.0755903 -0.0693851 0.0909127" rpy="1.5708 0 1.5708" />
+      <origin xyz="-0.0755903 0.0693851 0.0909127" rpy="-1.5708 0 -1.5708" />
       <mass value="5.62562911534835" />
       <inertia ixx="0.0504717539490822" ixy="-0.000186491896655228" ixz="0.0128492795010695" iyy="0.0306330356066479" iyz="9.71151606421086E-05" izz="0.0518045670438135" />
@@ -218,5 +218,5 @@
   </link>
   <joint name="camera_right_joint" type="fixed">
-    <origin xyz="0.171841 0.023 -0.0157567" rpy="-1.5708 0.820305 0" />
+    <origin xyz="0.171841 0.023 -0.0157567" rpy="1.5708 0.820305 0" />
     <parent link="head_link" />
     <child link="camera_right_link" />
@@ -233,5 +233,5 @@
   <link name="camera_left_link">
     <inertial>
-      <origin xyz="0.0744097 -0.0693851 -0.0909127" rpy="1.5708 0 1.5708" />
+      <origin xyz="-0.0744097 0.0693851 -0.0909127" rpy="-1.5708 0 -1.5708" />
       <mass value="5.62562911534835" />
       <inertia ixx="0.0504717539490822" ixy="-0.000186491896655198" ixz="-0.0128492795010695" iyy="0.0306330356066479" iyz="-9.711516064215E-05" izz="0.0518045670438135" />
@@ -239,5 +239,5 @@
   </link>
   <joint name="camera_left_joint" type="fixed">
-    <origin xyz="0.171841 0.173 -0.0157567" rpy="1.5708 0.820305 0" />
+    <origin xyz="0.171841 0.173 -0.0157567" rpy="-1.5708 0.820305 0" />
     <parent link="head_link" />
     <child link="camera_left_link" />
@@ -254,5 +254,5 @@
   <link name="camera_center_link">
     <inertial>
-      <origin xyz="-0.000590252 -0.0958729 -0.070924" rpy="1.5708 0 1.5708" />
+      <origin xyz="0.000590252 0.0958729 -0.070924" rpy="-1.5708 0 -1.5708" />
       <mass value="5.62562911534835" />
       <inertia ixx="0.0557556406323663" ixy="-0.000162225224016438" ixz="-0.0120094528841815" iyy="0.0306330356066479" iyz="-0.000133766806934365" izz="0.0465206803605294" />
@@ -260,5 +260,5 @@
   </link>
   <joint name="camera_center_joint" type="fixed">
-    <origin xyz="0.177246 0.098 -0.0239069" rpy="1.5708 0.610865 0" />
+    <origin xyz="0.177246 0.098 -0.0239069" rpy="-1.5708 0.610865 0" />
     <parent link="head_link" />
     <child link="camera_center_link" />
