Commit message: New URDF removes the need for manual TF manipulation

File: stretch4_urdf/SE4_francis/xacro/stretch_main.xacro (robot description, xacro)
@@ -1,15 +1,23 @@
 <robot xmlns:xacro="http://www.ros.org/wiki/xacro" name="stretch">
   <link name="base_footprint">
+    <visual>
+      <origin xyz="0 0 0" rpy="0 0 0" />
+      <geometry>
+        <box size="0.001 0.001 0.001" /></geometry>
+      <material name="">
+        <color rgba="0.752941176470588 0.752941176470588 0.752941176470588 1" />
+      </material>
+    </visual>
     </link>
   <link name="base_link">
     <inertial>
-      <origin xyz="0.000438847979959605 -0.00177714773743784 0.0964683588787771" rpy="0 0 0" />
+      <origin xyz="0.000438847979959618 -0.00177714773743785 0.0964683696491897" rpy="0 0 0" />
       <mass value="18.9261042191275" />
-      <inertia ixx="0.214992665976689" ixy="0.000833860434661022" ixz="-0.000588719185644055" iyy="0.223010418927309" iyz="-0.00155067412786045" izz="0.327845794874662" />
-    </inertial>
-    <visual>
-      <origin xyz="0 0 0" rpy="0 0 0" />
-      <geometry>
-        <mesh filename="$(arg model_mesh_dir)/base_link.OBJ" />
+      <inertia ixx="0.214992665976689" ixy="0.000833860434660833" ixz="-0.000588719185644081" iyy="0.223010418927309" iyz="-0.00155067412786042" izz="0.327845794874662" />
+    </inertial>
+    <visual>
+      <origin xyz="0 0 0" rpy="0 0 0" />
+      <geometry>
+        <mesh filename="$(arg model_mesh_dir)/base_link.STL" />
       </geometry>
       <material name="">
@@ -20,10 +28,10 @@
       <origin xyz="0 0 0" rpy="0 0 0" />
       <geometry>
-        <mesh filename="$(arg model_mesh_dir)/base_collision_link.OBJ" />
+        <mesh filename="$(arg model_mesh_dir)/base_collision_link.STL" />
       </geometry>
     </collision>
   </link>
   <joint name="base_ref" type="fixed">
-    <origin xyz="0 0 0.028" rpy="0 0 0" />
+    <origin xyz="0 0 0.027999995691835" rpy="0 0 0" />
     <parent link="base_footprint" />
     <child link="base_link" />
@@ -32,11 +40,17 @@
   <link name="line_sensor_5_link">
     <inertial>
-      <origin xyz="0.00114502 0.000126775 -0.0119762" rpy="1.5708 0 0" />
+      <origin xyz="0.00114502070313141 -0.000126774756058531 0.0119761602719026" rpy="0 0 0" />
       <mass value="0.00213836003346436" />
-      <inertia ixx="2.88698160050487E-07" ixy="-7.07831726662329E-09" ixz="5.64135957062429E-10" iyy="6.64615782289849E-08" iyz="2.73972720709955E-10" izz="2.34959277592962E-07" />
-    </inertial>
+      <inertia ixx="2.88698160050487E-07" ixy="-5.64135957062421E-10" ixz="-7.07831726662328E-09" iyy="2.34959277592962E-07" iyz="-2.73972720709966E-10" izz="6.64615782289848E-08" />
+    </inertial>
+    <collision name="line_sensor_5_collision_link">
+      <origin xyz="0 0 0" rpy="0 0 0" />
+      <geometry>
+        <mesh filename="$(arg model_mesh_dir)/line_sensor_5_link.STL" />
+      </geometry>
+    </collision>
   </link>
   <joint name="line_sensor_5_joint" type="fixed">
-    <origin xyz="0.0613832 0.178319 0.0527014" rpy="0 0.453786 1.0472" />
+    <origin xyz="0.0613832011662534 0.178318823151171 0.0527013981430276" rpy="0 0.453785605518531 1.04719755119659" />
     <parent link="base_link" />
     <child link="line_sensor_5_link" />
@@ -46,5 +60,5 @@
     </link>
   <joint name="line_sensor_5_optical_joint" type="fixed">
-    <origin xyz="0.00286 0 0" rpy="-1.5708 0 -1.5708" />
+    <origin xyz="0.00286000000000003 0 0" rpy="-1.5707963267949 0 -1.5707963267949" />
     <parent link="line_sensor_5_link" />
     <child link="line_sensor_5_optical_link" />
@@ -53,11 +67,17 @@
   <link name="line_sensor_4_link">
     <inertial>
-      <origin xyz="0.00114502 0.000126775 -0.0119762" rpy="1.5708 0 0" />
+      <origin xyz="0.00114502070313141 -0.000126774756058587 0.0119761602719026" rpy="0 0 0" />
       <mass value="0.00213836003346436" />
-      <inertia ixx="2.88698160050488E-07" ixy="-7.07831726662323E-09" ixz="5.64135957060017E-10" iyy="6.6461578228985E-08" iyz="2.73972720708404E-10" izz="2.34959277592962E-07" />
-    </inertial>
+      <inertia ixx="2.88698160050488E-07" ixy="-5.64135957060019E-10" ixz="-7.07831726662323E-09" iyy="2.34959277592962E-07" iyz="-2.7397272070835E-10" izz="6.64615782289851E-08" />
+    </inertial>
+    <collision name="line_sensor_4_collision_link">
+      <origin xyz="0 0 0" rpy="0 0 0" />
+      <geometry>
+        <mesh filename="$(arg model_mesh_dir)/line_sensor_4_link.STL" />
+      </geometry>
+    </collision>
   </link>
   <joint name="line_sensor_4_joint" type="fixed">
-    <origin xyz="-0.0613832 0.178319 0.0527014" rpy="0 0.453786 2.0944" />
+    <origin xyz="-0.0613832011662525 0.178318823151171 0.0527013981430276" rpy="0 0.453785605518532 2.09439510239319" />
     <parent link="base_link" />
     <child link="line_sensor_4_link" />
@@ -67,5 +87,5 @@
     </link>
   <joint name="line_sensor_4_optical_joint" type="fixed">
-    <origin xyz="0.00286 0 0" rpy="-1.5708 0 -1.5708" />
+    <origin xyz="0.00286 0 0" rpy="-1.5707963267949 0 -1.5707963267949" />
     <parent link="line_sensor_4_link" />
     <child link="line_sensor_4_optical_link" />
@@ -74,11 +94,17 @@
   <link name="line_sensor_3_link">
     <inertial>
-      <origin xyz="0.00114502 0.000126775 -0.0119762" rpy="1.5708 0 0" />
+      <origin xyz="0.00114502070313158 -0.000126774756058573 0.0119761602719024" rpy="0 0 0" />
       <mass value="0.00213836003346444" />
-      <inertia ixx="2.88698160050477E-07" ixy="-7.07831726660264E-09" ixz="5.64135957061256E-10" iyy="6.64615782289998E-08" iyz="2.73972720709257E-10" izz="2.34959277592965E-07" />
-    </inertial>
+      <inertia ixx="2.88698160050477E-07" ixy="-5.64135957061258E-10" ixz="-7.07831726660266E-09" iyy="2.34959277592965E-07" iyz="-2.73972720709266E-10" izz="6.64615782289998E-08" />
+    </inertial>
+    <collision name="line_sensor_3_collision_link">
+      <origin xyz="0 0 0" rpy="0 0 0" />
+      <geometry>
+        <mesh filename="$(arg model_mesh_dir)/line_sensor_3_link.STL" />
+      </geometry>
+    </collision>
   </link>
   <joint name="line_sensor_3_joint" type="fixed">
-    <origin xyz="-0.18512 -0.036 0.0527014" rpy="0 0.453786 -3.14159" />
+    <origin xyz="-0.185120231404985 -0.036 0.0527013981430276" rpy="0 0.453785605518531 -3.14159265358979" />
     <parent link="base_link" />
     <child link="line_sensor_3_link" />
@@ -88,5 +114,5 @@
     </link>
   <joint name="line_sensor_3_optical_joint" type="fixed">
-    <origin xyz="0.00286 0 0" rpy="-1.5708 0 -1.5708" />
+    <origin xyz="0.00286 0 0" rpy="-1.5707963267949 0 -1.5707963267949" />
     <parent link="line_sensor_3_link" />
     <child link="line_sensor_3_optical_link" />
@@ -95,11 +121,17 @@
   <link name="line_sensor_2_link">
     <inertial>
-      <origin xyz="0.00114502 0.000126775 -0.0119762" rpy="1.5708 0 0" />
+      <origin xyz="0.00114502070313144 -0.000126774756058531 0.0119761602719027" rpy="0 0 0" />
       <mass value="0.00213836003346437" />
-      <inertia ixx="2.88698160050488E-07" ixy="-7.07831726662343E-09" ixz="5.64135957062436E-10" iyy="6.64615782289851E-08" iyz="2.73972720710034E-10" izz="2.34959277592963E-07" />
-    </inertial>
+      <inertia ixx="2.88698160050489E-07" ixy="-5.64135957062398E-10" ixz="-7.07831726662342E-09" iyy="2.34959277592963E-07" iyz="-2.73972720710033E-10" izz="6.64615782289851E-08" />
+    </inertial>
+    <collision name="line_sensor_2_collision_link">
+      <origin xyz="0 0 0" rpy="0 0 0" />
+      <geometry>
+        <mesh filename="$(arg model_mesh_dir)/line_sensor_2_link.STL" />
+      </geometry>
+    </collision>
   </link>
   <joint name="line_sensor_2_joint" type="fixed">
-    <origin xyz="-0.123737 -0.142319 0.0527014" rpy="0 0.453786 -2.0944" />
+    <origin xyz="-0.123737030238733 -0.14231882315117 0.0527013981430276" rpy="0 0.453785605518531 -2.0943951023932" />
     <parent link="base_link" />
     <child link="line_sensor_2_link" />
@@ -109,5 +141,5 @@
     </link>
   <joint name="line_sensor_2_optical_joint" type="fixed">
-    <origin xyz="0.00286 0 0" rpy="-1.5708 0 -1.5708" />
+    <origin xyz="0.00286 0 0" rpy="-1.5707963267949 0 -1.5707963267949" />
     <parent link="line_sensor_2_link" />
     <child link="line_sensor_2_optical_link" />
@@ -116,11 +148,17 @@
   <link name="line_sensor_1_link">
     <inertial>
-      <origin xyz="0.00114502 0.000126775 -0.0119762" rpy="1.5708 0 0" />
+      <origin xyz="0.00114502070313141 -0.000126774756058601 0.0119761602719027" rpy="0 0 0" />
       <mass value="0.00213836003346436" />
-      <inertia ixx="2.88698160050487E-07" ixy="-7.07831726662329E-09" ixz="5.64135957059983E-10" iyy="6.64615782289849E-08" iyz="2.73972720708449E-10" izz="2.34959277592962E-07" />
-    </inertial>
+      <inertia ixx="2.88698160050487E-07" ixy="-5.64135957059992E-10" ixz="-7.07831726662327E-09" iyy="2.34959277592961E-07" iyz="-2.73972720708435E-10" izz="6.64615782289849E-08" />
+    </inertial>
+    <collision name="line_sensor_1_collision_link">
+      <origin xyz="0 0 0" rpy="0 0 0" />
+      <geometry>
+        <mesh filename="$(arg model_mesh_dir)/line_sensor_1_link.STL" />
+      </geometry>
+    </collision>
   </link>
   <joint name="line_sensor_1_joint" type="fixed">
-    <origin xyz="0.123737 -0.142319 0.0527014" rpy="0 0.453786 -1.0472" />
+    <origin xyz="0.123737030238732 -0.142318823151171 0.0527013981430276" rpy="0 0.453785605518531 -1.0471975511966" />
     <parent link="base_link" />
     <child link="line_sensor_1_link" />
@@ -130,20 +168,35 @@
     </link>
   <joint name="line_sensor_1_optical_joint" type="fixed">
-    <origin xyz="0.00286 0 0" rpy="-1.5708 0 -1.5708" />
+    <origin xyz="0.00286 0 0" rpy="-1.5707963267949 0 -1.5707963267949" />
     <parent link="line_sensor_1_link" />
     <child link="line_sensor_1_optical_link" />
     <axis xyz="0 0 0" />
   </joint>
-  <link name="line_sensor_0_link">
-    <inertial>
-      <origin xyz="0.00114502 0.000126775 -0.0119762" rpy="1.5708 0 0" />
+  <link name="sensor_0_link">
+    <inertial>
+      <origin xyz="0.00114502070313161 -0.000126774756058566 0.0119761602719025" rpy="0 0 0" />
       <mass value="0.00213836003346444" />
-      <inertia ixx="2.88698160050477E-07" ixy="-7.07831726660252E-09" ixz="5.64135957061258E-10" iyy="6.64615782290001E-08" iyz="2.73972720709191E-10" izz="2.34959277592965E-07" />
-    </inertial>
+      <inertia ixx="2.88698160050477E-07" ixy="-5.64135957061261E-10" ixz="-7.0783172666026E-09" iyy="2.34959277592965E-07" iyz="-2.73972720709192E-10" izz="6.6461578229E-08" />
+    </inertial>
+    <visual>
+      <origin xyz="0 0 0" rpy="0 0 0" />
+      <geometry>
+        <mesh filename="$(arg model_mesh_dir)/sensor_0_link.STL" />
+      </geometry>
+      <material name="">
+        <color rgba="0.792156862745098 0.819607843137255 0.933333333333333 1" />
+      </material>
+    </visual>
+    <collision name="sensor_0_collision_link">
+      <origin xyz="0 0 0" rpy="0 0 0" />
+      <geometry>
+        <mesh filename="$(arg model_mesh_dir)/sensor_0_link.STL" />
+      </geometry>
+    </collision>
   </link>
   <joint name="line_sensor_0_joint" type="fixed">
-    <origin xyz="0.18512 -0.036 0.0527014" rpy="0 0.453786 0" />
-    <parent link="base_link" />
-    <child link="line_sensor_0_link" />
+    <origin xyz="0.185120231404985 -0.0360000000000004 0.0527013981430276" rpy="0 0.453785605518531 0" />
+    <parent link="base_link" />
+    <child link="sensor_0_link" />
     <axis xyz="0 0 0" />
   </joint>
@@ -151,6 +204,6 @@
     </link>
   <joint name="line_sensor_0_optical_joint" type="fixed">
-    <origin xyz="0.00286 0 0" rpy="-1.5708 0 -1.5708" />
-    <parent link="line_sensor_0_link" />
+    <origin xyz="0.00286000000000003 0 0" rpy="-1.5707963267949 0 -1.5707963267949" />
+    <parent link="sensor_0_link" />
     <child link="line_sensor_0_optical_link" />
     <axis xyz="0 0 0" />
@@ -158,12 +211,12 @@
   <link name="head_link">
     <inertial>
-      <origin xyz="0.0578831464809341 0.0985910077817881 -0.0270263436790745" rpy="0 0 0" />
-      <mass value="5.618435167362" />
-      <inertia ixx="0.0382731622122869" ixy="0.000202623919235895" ixz="0.000231642202175719" iyy="0.0306326706365949" iyz="5.61616354648268E-05" izz="0.0640020784749226" />
-    </inertial>
-    <visual>
-      <origin xyz="0 0 0" rpy="0 0 0" />
-      <geometry>
-        <mesh filename="$(arg model_mesh_dir)/head_link.obj" />
+      <origin xyz="0.0578831450711745 0.0985910072575782 -0.0270263437535108" rpy="0 0 0" />
+      <mass value="5.61843540939406" />
+      <inertia ixx="0.0382731622600879" ixy="0.000202623770136033" ixz="0.00023164221061037" iyy="0.030632670593406" iyz="5.61616115268146E-05" izz="0.06400207843788" />
+    </inertial>
+    <visual>
+      <origin xyz="0 0 0" rpy="0 0 0" />
+      <geometry>
+        <mesh filename="$(arg model_mesh_dir)/head_link.STL" />
       </geometry>
       <material name="">
@@ -174,10 +227,10 @@
       <origin xyz="0 0 0" rpy="0 0 0" />
       <geometry>
-        <mesh filename="$(arg model_mesh_dir)/head_collision_link.obj" />
+        <mesh filename="$(arg model_mesh_dir)/head_collision_link.STL" />
       </geometry>
     </collision>
   </link>
   <joint name="head_joint" type="fixed">
-    <origin xyz="-0.093 -0.098 1.559" rpy="0 0 0" />
+    <origin xyz="-0.0930000000000002 -0.0979999999999998 1.55900000430817" rpy="0 0 0" />
     <parent link="base_link" />
     <child link="head_link" />
@@ -186,11 +239,17 @@
   <link name="lidar_right_link">
     <inertial>
-      <origin xyz="0.0766909447572703 0.0306840677846499 -0.12335811389925" rpy="0 0 0" />
-      <mass value="5.62562911534835" />
-      <inertia ixx="0.0492829862682945" ixy="-0.00156447943074778" ixz="0.0149316960757035" iyy="0.0349356510816738" iyz="0.00380036130478219" izz="0.0486907192495753" />
-    </inertial>
+      <origin xyz="0.0766909452916591 0.0306840664060522 -0.123358114205568" rpy="0 0 0" />
+      <mass value="5.62562935738041" />
+      <inertia ixx="0.0492829863501232" ixy="-0.0015644794553125" ixz="0.0149316959819941" iyy="0.0349356509390749" iyz="0.0038003613530989" izz="0.048690719277915" />
+    </inertial>
+    <collision name="lidar_right_collision_link">
+      <origin xyz="0 0 0" rpy="0 0 0" />
+      <geometry>
+        <mesh filename="$(arg model_mesh_dir)/lidar_right_link.STL" />
+      </geometry>
+    </collision>
   </link>
   <joint name="lidar_right_joint" type="fixed">
-    <origin xyz="0.131744 -0.0264137 -0.058328" rpy="-3.05466 0.7816 2.39203" />
+    <origin xyz="0.131744211811827 -0.0264137425448753 -0.0583279884119643" rpy="-3.05465659239941 0.781600065124168 2.39203005564319" />
     <parent link="head_link" />
     <child link="lidar_right_link" />
@@ -199,11 +258,17 @@
   <link name="lidar_left_link">
     <inertial>
-      <origin xyz="-0.0761200632210846 0.0298724102181261 -0.122718664121595" rpy="0 0 0" />
-      <mass value="5.62562911534835" />
-      <inertia ixx="0.0495631509325281" ixy="0.00150375861955282" ixz="-0.0147241234027668" iyy="0.0345419854283597" iyz="0.00388339874340473" izz="0.0488042202386559" />
-    </inertial>
+      <origin xyz="-0.0761200642618001 0.0298724095594048 -0.122718664995054" rpy="0 0 0" />
+      <mass value="5.62562935738041" />
+      <inertia ixx="0.0495631508318921" ixy="0.00150375867091916" ixz="-0.0147241234604212" iyy="0.034541985578385" iyz="0.00388339874636518" izz="0.0488042201568361" />
+    </inertial>
+    <collision name="lidar_left_collision_link">
+      <origin xyz="0 0 0" rpy="0 0 0" />
+      <geometry>
+        <mesh filename="$(arg model_mesh_dir)/lidar_left_link.STL" />
+      </geometry>
+    </collision>
   </link>
   <joint name="lidar_left_joint" type="fixed">
-    <origin xyz="0.131744 0.222414 -0.058328" rpy="-3.05466 -0.7816 0.749563" />
+    <origin xyz="0.131744211811846 0.222413742544858 -0.0583279884119634" rpy="-3.05465659239939 -0.781600065124167 0.749562597946573" />
     <parent link="head_link" />
     <child link="lidar_left_link" />
@@ -212,11 +277,17 @@
   <link name="camera_right_link">
     <inertial>
-      <origin xyz="-0.0755903 0.0693851 0.0909127" rpy="-1.5708 0 -1.5708" />
-      <mass value="5.62562911534835" />
-      <inertia ixx="0.0504717539490822" ixy="-0.000186491896655228" ixz="0.0128492795010695" iyy="0.0306330356066479" iyz="9.71151606421086E-05" izz="0.0518045670438135" />
-    </inertial>
+      <origin xyz="-0.0693850700494765 -0.0909126816993031 -0.0755902514887177" rpy="0 0 0" />
+      <mass value="5.62562935738041" />
+      <inertia ixx="0.0518045670378194" ixy="-0.0128492794593393" ixz="-9.71150764634026E-05" iyy="0.0504717539658347" iyz="-0.000186491771284805" izz="0.0306330355634591" />
+    </inertial>
+    <collision name="camera_right_collision_link">
+      <origin xyz="0 0 0" rpy="0 0 0" />
+      <geometry>
+        <mesh filename="$(arg model_mesh_dir)/camera_right_link.STL" />
+      </geometry>
+    </collision>
   </link>
   <joint name="camera_right_joint" type="fixed">
-    <origin xyz="0.171841 0.023 -0.0157567" rpy="1.5708 0.820305 0" />
+    <origin xyz="0.171840602787894 0.0230000000000032 -0.0157566987072475" rpy="1.5707963267949 0.820304748437337 0" />
     <parent link="head_link" />
     <child link="camera_right_link" />
@@ -226,5 +297,5 @@
     </link>
   <joint name="camera_right_optical_joint" type="fixed">
-    <origin xyz="0.0212 0 0" rpy="-1.5708 0 -1.5708" />
+    <origin xyz="0.0212000000000001 0 0" rpy="-1.5707963267949 0 -1.5707963267949" />
     <parent link="camera_right_link" />
     <child link="camera_right_optical_link" />
@@ -233,11 +304,17 @@
   <link name="camera_left_link">
     <inertial>
-      <origin xyz="-0.0744097 0.0693851 -0.0909127" rpy="-1.5708 0 -1.5708" />
-      <mass value="5.62562911534835" />
-      <inertia ixx="0.0504717539490822" ixy="-0.000186491896655198" ixz="-0.0128492795010695" iyy="0.0306330356066479" iyz="-9.711516064215E-05" izz="0.0518045670438135" />
-    </inertial>
+      <origin xyz="-0.0693850700494769 0.0909126816993033 -0.0744097485112792" rpy="0 0 0" />
+      <mass value="5.62562935738041" />
+      <inertia ixx="0.0518045670378194" ixy="0.0128492794593393" ixz="9.71150764634441E-05" iyy="0.0504717539658347" iyz="-0.000186491771284775" izz="0.0306330355634591" />
+    </inertial>
+    <collision name="camera_left_collision_link">
+      <origin xyz="0 0 0" rpy="0 0 0" />
+      <geometry>
+        <mesh filename="$(arg model_mesh_dir)/camera_left_link.STL" />
+      </geometry>
+    </collision>
   </link>
   <joint name="camera_left_joint" type="fixed">
-    <origin xyz="0.171841 0.173 -0.0157567" rpy="-1.5708 0.820305 0" />
+    <origin xyz="0.171840602787895 0.173 -0.0157566987072475" rpy="-1.5707963267949 0.820304748437337 0" />
     <parent link="head_link" />
     <child link="camera_left_link" />
@@ -247,5 +324,5 @@
     </link>
   <joint name="camera_left_optical_joint" type="fixed">
-    <origin xyz="0.0212 0 0" rpy="-1.5708 0 -1.5708" />
+    <origin xyz="0.0211999999999999 0 0" rpy="-1.5707963267949 0 -1.5707963267949" />
     <parent link="camera_left_link" />
     <child link="camera_left_optical_link" />
@@ -254,11 +331,17 @@
   <link name="camera_center_link">
     <inertial>
-      <origin xyz="0.000590252 0.0958729 -0.070924" rpy="-1.5708 0 -1.5708" />
-      <mass value="5.62562911534835" />
-      <inertia ixx="0.0557556406323663" ixy="-0.000162225224016438" ixz="-0.0120094528841815" iyy="0.0306330356066479" iyz="-0.000133766806934365" izz="0.0465206803605294" />
-    </inertial>
+      <origin xyz="-0.0958729354978768 0.0709239731668885 0.000590251488720641" rpy="0 0 0" />
+      <mass value="5.62562935738041" />
+      <inertia ixx="0.0465206803724917" ixy="0.0120094528414331" ixz="0.000133766698529188" iyy="0.0557556406311624" iyz="-0.000162225118887399" izz="0.0306330355634591" />
+    </inertial>
+    <collision name="camera_center_collision_link">
+      <origin xyz="0 0 0" rpy="0 0 0" />
+      <geometry>
+        <mesh filename="$(arg model_mesh_dir)/camera_center_link.STL" />
+      </geometry>
+    </collision>
   </link>
   <joint name="camera_center_joint" type="fixed">
-    <origin xyz="0.177246 0.098 -0.0239069" rpy="-1.5708 0.610865 0" />
+    <origin xyz="0.177245603402412 0.0980000000000004 -0.0239069097938973" rpy="-1.5707963267949 0.610865238198018 0" />
     <parent link="head_link" />
     <child link="camera_center_link" />
@@ -268,5 +351,5 @@
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
File: stretch4_urdf/SE4_tools/eoa_wrist_dw4_tool_sg4/eoa_wrist_dw4_tool_sg4.urdf (robot description, URDF)
Before this commit: robot URDF_DALI_ASSEM_Stretch_Gripper_V4, 8 links, 7 joints
Joints:
- joint aruco_fingertip_left_joint: origin xyz=0.0335358 0.00675395 3.80134e-05 rpy=1.37881 -2.50583e-06 0.62832 -> xyz=3.80423e-05 -0.0335357 -0.00675433 rpy=1.37881 -2.50583e-06 0.62832
- joint aruco_fingertip_right_joint: origin xyz=-0.0335357 0.00675413 3.81175e-05 rpy=1.37881 1.8123e-06 2.51327 -> xyz=-3.81181e-05 0.0335357 0.00675399 rpy=1.37881 1.8123e-06 2.51327
- joint grasp_center_joint: origin xyz=0.234538 0 0 rpy=0 0 -1.5708 -> xyz=-0.234538 0 0 rpy=0 0 0
- joint gripper_finger_left_joint: origin xyz=0.0373909 0.0222607 0 rpy=1.5708 0 3.14159 -> xyz=-0.0373909 -0.0222607 0 rpy=0 0 0
- joint gripper_finger_right_joint: origin xyz=0.0373909 -0.0222607 0 rpy=1.5708 0 3.14159 -> xyz=-0.0373909 0.0222607 0 rpy=0 0 0
- joint gripper_fingertip_left_joint: origin xyz=-0.191008 0 -0.022168 rpy=-1.5708 2.65359e-06 0 -> xyz=-0.191008 0.0221671 0 rpy=0.625614 -1.57079 0.945183
- joint gripper_fingertip_right_joint: origin xyz=-0.191008 0 0.022168 rpy=1.5708 -2.65359e-06 3.14159 -> xyz=-0.191008 -0.0221675 0 rpy=-0.625614 1.57079 -2.19641
