Commit message: Gripper camera fix and new docking contact link

File: stretch4_urdf/SE4_francis/xacro/stretch_main.xacro (robot description, xacro)
@@ -12,7 +12,7 @@
   <link name="base_link">
     <inertial>
-      <origin xyz="0.000438847979959618 -0.00177714773743785 0.0964683696491897" rpy="0 0 0" />
-      <mass value="18.9261042191275" />
-      <inertia ixx="0.214992665976689" ixy="0.000833860434660833" ixz="-0.000588719185644081" iyy="0.223010418927309" iyz="-0.00155067412786042" izz="0.327845794874662" />
+      <origin xyz="0.000438848617413435 -0.00177714671567261 0.0964683686997768" rpy="0 0 0" />
+      <mass value="18.9261039673325" />
+      <inertia ixx="0.214992663147159" ixy="0.00083386140340347" ixz="-0.000588720101362878" iyy="0.22301041696344" iyz="-0.00155067556464412" izz="0.327845792807285" />
     </inertial>
     <visual>
@@ -40,5 +40,5 @@
   <link name="line_sensor_5_link">
     <inertial>
-      <origin xyz="0.00114502070313141 -0.000126774756058531 0.0119761602719026" rpy="0 0 0" />
+      <origin xyz="0.00114502070313141 -0.000126774756058545 0.0119761602719026" rpy="0 0 0" />
       <mass value="0.00213836003346436" />
       <inertia ixx="2.88698160050487E-07" ixy="-5.64135957062421E-10" ixz="-7.07831726662328E-09" iyy="2.34959277592962E-07" iyz="-2.73972720709966E-10" izz="6.64615782289848E-08" />
@@ -67,7 +67,7 @@
   <link name="line_sensor_4_link">
     <inertial>
-      <origin xyz="0.00114502070313141 -0.000126774756058587 0.0119761602719026" rpy="0 0 0" />
+      <origin xyz="0.00114502070313144 -0.000126774756058601 0.0119761602719027" rpy="0 0 0" />
       <mass value="0.00213836003346436" />
-      <inertia ixx="2.88698160050488E-07" ixy="-5.64135957060019E-10" ixz="-7.07831726662323E-09" iyy="2.34959277592962E-07" iyz="-2.7397272070835E-10" izz="6.64615782289851E-08" />
+      <inertia ixx="2.88698160050488E-07" ixy="-5.64135957060042E-10" ixz="-7.07831726662323E-09" iyy="2.34959277592962E-07" iyz="-2.73972720708353E-10" izz="6.6461578228985E-08" />
     </inertial>
     <collision name="line_sensor_4_collision_link">
@@ -96,5 +96,5 @@
       <origin xyz="0.00114502070313158 -0.000126774756058573 0.0119761602719024" rpy="0 0 0" />
       <mass value="0.00213836003346444" />
-      <inertia ixx="2.88698160050477E-07" ixy="-5.64135957061258E-10" ixz="-7.07831726660266E-09" iyy="2.34959277592965E-07" iyz="-2.73972720709266E-10" izz="6.64615782289998E-08" />
+      <inertia ixx="2.88698160050477E-07" ixy="-5.64135957061257E-10" ixz="-7.07831726660265E-09" iyy="2.34959277592965E-07" iyz="-2.73972720709266E-10" izz="6.64615782289998E-08" />
     </inertial>
     <collision name="line_sensor_3_collision_link">
@@ -121,7 +121,7 @@
   <link name="line_sensor_2_link">
     <inertial>
-      <origin xyz="0.00114502070313144 -0.000126774756058531 0.0119761602719027" rpy="0 0 0" />
+      <origin xyz="0.00114502070313144 -0.000126774756058518 0.0119761602719027" rpy="0 0 0" />
       <mass value="0.00213836003346437" />
-      <inertia ixx="2.88698160050489E-07" ixy="-5.64135957062398E-10" ixz="-7.07831726662342E-09" iyy="2.34959277592963E-07" iyz="-2.73972720710033E-10" izz="6.64615782289851E-08" />
+      <inertia ixx="2.88698160050489E-07" ixy="-5.64135957062399E-10" ixz="-7.07831726662342E-09" iyy="2.34959277592963E-07" iyz="-2.73972720710027E-10" izz="6.64615782289852E-08" />
     </inertial>
     <collision name="line_sensor_2_collision_link">
@@ -150,5 +150,5 @@
       <origin xyz="0.00114502070313141 -0.000126774756058601 0.0119761602719027" rpy="0 0 0" />
       <mass value="0.00213836003346436" />
-      <inertia ixx="2.88698160050487E-07" ixy="-5.64135957059992E-10" ixz="-7.07831726662327E-09" iyy="2.34959277592961E-07" iyz="-2.73972720708435E-10" izz="6.64615782289849E-08" />
+      <inertia ixx="2.88698160050487E-07" ixy="-5.64135957060014E-10" ixz="-7.0783172666233E-09" iyy="2.34959277592961E-07" iyz="-2.73972720708438E-10" izz="6.64615782289849E-08" />
     </inertial>
     <collision name="line_sensor_1_collision_link">
@@ -175,7 +175,7 @@
   <link name="sensor_0_link">
     <inertial>
-      <origin xyz="0.00114502070313161 -0.000126774756058566 0.0119761602719025" rpy="0 0 0" />
+      <origin xyz="0.00114502070313158 -0.000126774756058566 0.0119761602719025" rpy="0 0 0" />
       <mass value="0.00213836003346444" />
-      <inertia ixx="2.88698160050477E-07" ixy="-5.64135957061261E-10" ixz="-7.0783172666026E-09" iyy="2.34959277592965E-07" iyz="-2.73972720709192E-10" izz="6.6461578229E-08" />
+      <inertia ixx="2.88698160050477E-07" ixy="-5.64135957061259E-10" ixz="-7.07831726660262E-09" iyy="2.34959277592965E-07" iyz="-2.73972720709195E-10" izz="6.6461578229E-08" />
     </inertial>
     <visual>
@@ -211,7 +211,7 @@
   <link name="head_link">
     <inertial>
-      <origin xyz="0.0578831450711745 0.0985910072575782 -0.0270263437535108" rpy="0 0 0" />
+      <origin xyz="0.0578831450711746 0.0985910072575783 -0.0270263437535101" rpy="0 0 0" />
       <mass value="5.61843540939406" />
-      <inertia ixx="0.0382731622600879" ixy="0.000202623770136033" ixz="0.00023164221061037" iyy="0.030632670593406" iyz="5.61616115268146E-05" izz="0.06400207843788" />
+      <inertia ixx="0.038273162260088" ixy="0.000202623770136025" ixz="0.000231642210610366" iyy="0.030632670593406" iyz="5.61616115268112E-05" izz="0.06400207843788" />
     </inertial>
     <visual>
@@ -239,7 +239,7 @@
   <link name="lidar_right_link">
     <inertial>
-      <origin xyz="0.0766909452916591 0.0306840664060522 -0.123358114205568" rpy="0 0 0" />
+      <origin xyz="0.0766909452916593 0.0306840664060523 -0.123358114205567" rpy="0 0 0" />
       <mass value="5.62562935738041" />
-      <inertia ixx="0.0492829863501232" ixy="-0.0015644794553125" ixz="0.0149316959819941" iyy="0.0349356509390749" iyz="0.0038003613530989" izz="0.048690719277915" />
+      <inertia ixx="0.0492829863501233" ixy="-0.0015644794553125" ixz="0.0149316959819942" iyy="0.0349356509390749" iyz="0.00380036135309891" izz="0.0486907192779151" />
     </inertial>
     <collision name="lidar_right_collision_link">
@@ -260,5 +260,5 @@
       <origin xyz="-0.0761200642618001 0.0298724095594048 -0.122718664995054" rpy="0 0 0" />
       <mass value="5.62562935738041" />
-      <inertia ixx="0.0495631508318921" ixy="0.00150375867091916" ixz="-0.0147241234604212" iyy="0.034541985578385" iyz="0.00388339874636518" izz="0.0488042201568361" />
+      <inertia ixx="0.0495631508318921" ixy="0.00150375867091917" ixz="-0.0147241234604212" iyy="0.034541985578385" iyz="0.00388339874636519" izz="0.0488042201568361" />
     </inertial>
     <collision name="lidar_left_collision_link">
@@ -279,5 +279,5 @@
       <origin xyz="-0.0693850700494765 -0.0909126816993031 -0.0755902514887177" rpy="0 0 0" />
       <mass value="5.62562935738041" />
-      <inertia ixx="0.0518045670378194" ixy="-0.0128492794593393" ixz="-9.71150764634026E-05" iyy="0.0504717539658347" iyz="-0.000186491771284805" izz="0.0306330355634591" />
+      <inertia ixx="0.0518045670378195" ixy="-0.0128492794593393" ixz="-9.71150764633997E-05" iyy="0.0504717539658347" iyz="-0.000186491771284797" izz="0.0306330355634591" />
     </inertial>
     <collision name="camera_right_collision_link">
@@ -306,5 +306,5 @@
       <origin xyz="-0.0693850700494769 0.0909126816993033 -0.0744097485112792" rpy="0 0 0" />
       <mass value="5.62562935738041" />
-      <inertia ixx="0.0518045670378194" ixy="0.0128492794593393" ixz="9.71150764634441E-05" iyy="0.0504717539658347" iyz="-0.000186491771284775" izz="0.0306330355634591" />
+      <inertia ixx="0.0518045670378195" ixy="0.0128492794593393" ixz="9.71150764634412E-05" iyy="0.0504717539658347" iyz="-0.000186491771284767" izz="0.0306330355634591" />
     </inertial>
     <collision name="camera_left_collision_link">
@@ -331,7 +331,7 @@
   <link name="camera_center_link">
     <inertial>
-      <origin xyz="-0.0958729354978768 0.0709239731668885 0.000590251488720641" rpy="0 0 0" />
+      <origin xyz="-0.0958729354978766 0.0709239731668887 0.000590251488720675" rpy="0 0 0" />
       <mass value="5.62562935738041" />
-      <inertia ixx="0.0465206803724917" ixy="0.0120094528414331" ixz="0.000133766698529188" iyy="0.0557556406311624" iyz="-0.000162225118887399" izz="0.0306330355634591" />
+      <inertia ixx="0.0465206803724917" ixy="0.0120094528414331" ixz="0.000133766698529184" iyy="0.0557556406311624" iyz="-0.000162225118887392" izz="0.0306330355634591" />
     </inertial>
     <collision name="camera_center_collision_link">
@@ -360,5 +360,5 @@
       <origin xyz="2.77555756156289E-17 -0.00165282700965368 0.815" rpy="0 0 0" />
       <mass value="10.8924861076487" />
-      <inertia ixx="1.96276319417158" ixy="-4.91253888692586E-18" ixz="-1.21184210498761E-16" iyy="1.96594229514087" iyz="-3.35011521318398E-18" izz="0.00577661764276332" />
+      <inertia ixx="1.96276319417158" ixy="-4.74739862687269E-18" ixz="-1.24526930733894E-16" iyy="1.96594229514087" iyz="-1.7420761023809E-18" izz="0.00577661764276332" />
     </inertial>
     <visual>
@@ -386,7 +386,7 @@
   <link name="lift_link">
     <inertial>
-      <origin xyz="-0.0148722581318623 0.0596072894254191 0.00542773918494444" rpy="0 0 0" />
+      <origin xyz="-0.0148722581318624 0.0596072894254191 0.00542773918494432" rpy="0 0 0" />
       <mass value="2.95349364666659" />
-      <inertia ixx="0.0117399464230091" ixy="0.000875437380496019" ixz="0.000164784888522663" iyy="0.0102748963241433" iyz="-0.00101918054718661" izz="0.0139841484528854" />
+      <inertia ixx="0.0117399464230091" ixy="0.000875437380496019" ixz="0.000164784888522662" iyy="0.0102748963241433" iyz="-0.00101918054718661" izz="0.0139841484528854" />
     </inertial>
     <visual>
@@ -415,5 +415,5 @@
   <link name="arm_l0_link">
     <inertial>
-      <origin xyz="-0.0316222581318623 -0.039792710574581 0.0182872881301621" rpy="0 0 0" />
+      <origin xyz="-0.0316222581318624 -0.0397927105745811 0.0182872881301621" rpy="0 0 0" />
       <mass value="2.95349364666659" />
       <inertia ixx="0.0117399464230091" ixy="0.000875437380496019" ixz="0.000164784888522662" iyy="0.0102748963241433" iyz="-0.00101918054718661" izz="0.0139841484528854" />
@@ -443,7 +443,7 @@
   <link name="arm_l1_link">
     <inertial>
-      <origin xyz="0.0983194277508772 -6.17042026110449E-17 0.00214616065125611" rpy="0 0 0" />
+      <origin xyz="0.0983194277508772 -4.84141562609803E-17 0.00214616065125611" rpy="0 0 0" />
       <mass value="0.211728696447344" />
-      <inertia ixx="0.000227675228746485" ixy="1.42790510359093E-19" ixz="1.46222263181723E-10" iyy="0.000730798627565317" iyz="2.71815409206256E-21" izz="0.000759408092665036" />
+      <inertia ixx="0.000227675228746485" ixy="1.74505747014533E-19" ixz="1.46222263149901E-10" iyy="0.000730798627565317" iyz="1.04945328084606E-20" izz="0.000759408092665037" />
     </inertial>
     <visual>
@@ -472,7 +472,7 @@
   <link name="arm_l2_link">
     <inertial>
-      <origin xyz="0.126544808120785 -5.28822009914513E-17 0.00212532899607004" rpy="0 0 0" />
+      <origin xyz="0.126544808120785 -4.72555604260908E-17 0.00212532899607004" rpy="0 0 0" />
       <mass value="0.197181391808907" />
-      <inertia ixx="0.000180704361161813" ixy="1.40253445285864E-19" ixz="1.56735722637944E-10" iyy="0.000676905139492615" iyz="-3.72122630710006E-21" izz="0.000701571828521803" />
+      <inertia ixx="0.000180704361161813" ixy="1.07026638037563E-19" ixz="1.56735722682903E-10" iyy="0.000676905139492615" iyz="-8.22433526184444E-21" izz="0.000701571828521803" />
     </inertial>
     <visual>
@@ -501,7 +501,7 @@
   <link name="arm_l3_link">
     <inertial>
-      <origin xyz="0.154805576226277 -2.99487980435997E-17 0.00210076275486304" rpy="0 0 0" />
+      <origin xyz="0.154805576226277 -3.07037539647458E-17 0.00210076275486304" rpy="0 0 0" />
       <mass value="0.182379618165529" />
-      <inertia ixx="0.000140464382352664" ixy="2.14407536327449E-19" ixz="1.68878152445003E-10" iyy="0.00062371110107317" iyz="-1.10859874912867E-20" izz="0.000644687237937217" />
+      <inertia ixx="0.000140464382352664" ixy="2.1435437078952E-19" ixz="1.68878152441465E-10" iyy="0.00062371110107317" iyz="-9.8151250050676E-21" izz="0.000644687237937217" />
     </inertial>
     <visual>
@@ -530,7 +530,7 @@
   <link name="arm_l4_link">
     <inertial>
-      <origin xyz="0.15125 3.35236566452435E-16 0.00206007053977714" rpy="0 0 0" />
+      <origin xyz="0.15125 3.40653404230178E-16 0.00206007053977714" rpy="0 0 0" />
       <mass value="0.131482025176648" />
-      <inertia ixx="7.61244098718923E-05" ixy="8.57509226382842E-20" ixz="-6.85841251548587E-20" iyy="0.00051464101554282" iyz="-4.71969502254436E-21" izz="0.000527876279377434" />
+      <inertia ixx="7.61244098718923E-05" ixy="9.69178609077501E-20" ixz="-4.66991036331849E-20" iyy="0.00051464101554282" iyz="6.30460018301958E-22" izz="0.000527876279377434" />
     </inertial>
     <visual>
@@ -559,7 +559,7 @@
   <link name="wrist_link">
     <inertial>
-      <origin xyz="-0.00943224270685236 -2.24072494908036E-08 0.0350669907502222" rpy="0 0 0" />
+      <origin xyz="-0.00943224270685253 -2.24072505584934E-08 0.0350669907502222" rpy="0 0 0" />
       <mass value="0.228848612237181" />
-      <inertia ixx="0.000122470482540944" ixy="-1.07472717291765E-10" ixz="1.16790939209657E-05" iyy="0.0001715213303575" iyz="-9.50304167695345E-11" izz="0.000141511317394913" />
+      <inertia ixx="0.000122470482540944" ixy="-1.07472717309855E-10" ixz="1.16790939209657E-05" iyy="0.0001715213303575" iyz="-9.50304167649752E-11" izz="0.000141511317394913" />
     </inertial>
     <visual>
@@ -637,15 +637,15 @@
   </link>
   <joint name="wrist_pitch_joint" type="revolute">
-    <origin xyz="0 -0.0422200000000001 -0.0452000000000001" rpy="0 0 0" />
+    <origin xyz="0 -0.04222 -0.0452" rpy="0 0 0" />
     <parent link="wrist_yaw_link" />
     <child link="wrist_pitch_link" />
-    <axis xyz="0 -1 0" />
-    <limit lower="-4.276" upper="1.135" effort="0" velocity="0" />
+    <axis xyz="0 1 0" />
+    <limit lower="-1.135" upper="4.276" effort="0" velocity="0" />
   </joint>
   <link name="wrist_roll_link">
     <inertial>
-      <origin xyz="0.0125796209584655 0.00139059549833792 0.012231226279655" rpy="0 0 0" />
+      <origin xyz="0.0125796209584655 0.00139059549833795 0.012231226279655" rpy="0 0 0" />
       <mass value="0.0875518779599177" />
-      <inertia ixx="7.36573009473639E-05" ixy="1.09648627072304E-11" ixz="3.93918627087478E-06" iyy="5.3109684066939E-05" iyz="2.53579489920842E-10" izz="2.50172844184434E-05" />
+      <inertia ixx="7.36573009473639E-05" ixy="1.09648627072382E-11" ixz="3.93918627087477E-06" iyy="5.3109684066939E-05" iyz="2.53579489921485E-10" izz="2.50172844184434E-05" />
     </inertial>
     <visual>
@@ -670,11 +670,11 @@
     <child link="wrist_roll_link" />
     <axis xyz="1 0 0" />
-    <limit lower="-1.135" upper="4.276" effort="0" velocity="0" />
+    <limit lower="-4.276" upper="1.135" effort="0" velocity="0" />
   </joint>
   <link name="gripper_camera_link">
     <inertial>
-      <origin xyz="-0.0121348322776446 -1.38777878078145E-17 0.00187096264569653" rpy="0 0 0" />
+      <origin xyz="-0.0121348322776446 0 0.00187096264569653" rpy="0 0 0" />
       <mass value="0.0447759731526001" />
-      <inertia ixx="1.60194001393268E-05" ixy="9.36418181523527E-22" ixz="9.91050471819132E-08" iyy="6.92267971098109E-06" iyz="-4.69734902377389E-22" izz="1.36285341071377E-05" />
+      <inertia ixx="1.60194001393268E-05" ixy="9.03146096735839E-22" ixz="9.91050471819132E-08" iyy="6.92267971098109E-06" iyz="-4.42031565006143E-22" izz="1.36285341071377E-05" />
     </inertial>
     <visual>
@@ -711,5 +711,5 @@
     </link>
   <joint name="gripper_stereo_camera_color_optical_joint" type="fixed">
-    <origin xyz="0 0 0" rpy="-1.5707963267949 -0.0523598775598298 0" />
+    <origin xyz="0 0 0" rpy="-1.51843644923507 0 -1.5707963267949" />
     <parent link="gripper_camera_link" />
     <child link="gripper_stereo_camera_color_optical_frame" />
@@ -727,5 +727,5 @@
     </link>
   <joint name="gripper_right_camera_color_optical_joint" type="fixed">
-    <origin xyz="0 -0.01 0" rpy="-1.5707963267949 -0.0523598775598298 0" />
+    <origin xyz="0 -0.01 0" rpy="-1.51843644923507 0 -1.5707963267949" />
     <parent link="gripper_camera_link" />
     <child link="gripper_right_camera_color_optical_frame" />
@@ -743,5 +743,5 @@
     </link>
   <joint name="gripper_left_camera_color_optical_joint" type="fixed">
-    <origin xyz="0 0.01 0" rpy="-1.5707963267949 -0.0523598775598298 0" />
+    <origin xyz="0 0.01 0" rpy="-1.51843644923507 0 -1.5707963267949" />
     <parent link="gripper_camera_link" />
     <child link="gripper_left_camera_color_optical_frame" />
@@ -752,5 +752,5 @@
       <origin xyz="-0.00602037904153455 0.00139059549833791 0.012231226279655" rpy="0 0 0" />
       <mass value="0.0875518779599177" />
-      <inertia ixx="7.36573009473639E-05" ixy="1.09648627076813E-11" ixz="3.93918627087477E-06" iyy="5.3109684066939E-05" iyz="2.5357948992143E-10" izz="2.50172844184434E-05" />
+      <inertia ixx="7.36573009473639E-05" ixy="1.09648627077354E-11" ixz="3.93918627087477E-06" iyy="5.3109684066939E-05" iyz="2.535794899228E-10" izz="2.50172844184434E-05" />
     </inertial>
     <visual>
@@ -778,7 +778,7 @@
   <link name="wrist_aruco_link">
     <inertial>
-      <origin xyz="-8.97014059894619E-06 2.99075835221763E-06 -0.000313517411967446" rpy="0 0 0" />
+      <origin xyz="-8.97014059911272E-06 2.99075835115259E-06 -0.000313517411967557" rpy="0 0 0" />
       <mass value="0.000520487721584508" />
-      <inertia ixx="3.834908442783E-08" ixy="-1.23630345810507E-14" ixz="1.34704395412492E-12" iyy="3.83685013633507E-08" iyz="-4.4912149519828E-13" izz="7.66888919510146E-08" />
+      <inertia ixx="3.834908442783E-08" ixy="-1.23630345809062E-14" ixz="1.34704395412487E-12" iyy="3.83685013633507E-08" iyz="-4.49121495198314E-13" izz="7.66888919510146E-08" />
     </inertial>
     <visual>
@@ -806,7 +806,7 @@
   <link name="wrist_reflector_link">
     <inertial>
-      <origin xyz="0.00377531872412074 -3.85449981286527E-12 0.00351760915937299" rpy="0 0 0" />
+      <origin xyz="0.00377531872412057 -3.85556475255951E-12 0.00351760915937294" rpy="0 0 0" />
       <mass value="0.00171618092746856" />
-      <inertia ixx="1.51127728759546E-07" ixy="1.29437561169358E-17" ixz="-1.24862425165547E-09" iyy="1.64146246077095E-08" iyz="-2.00458483084907E-17" izz="1.47242352409892E-07" />
+      <inertia ixx="1.51127728759546E-07" ixy="1.29437519397159E-17" ixz="-1.24862425165547E-09" iyy="1.64146246077095E-08" iyz="-2.00458419822811E-17" izz="1.47242352409892E-07" />
     </inertial>
     <visual>
@@ -834,7 +834,7 @@
   <link name="wheel_2_link">
     <inertial>
-      <origin xyz="1.25476756894562E-05 5.22307168604463E-06 -0.000275017600766342" rpy="0 0 0" />
+      <origin xyz="1.25476756894564E-05 5.22307168604463E-06 -0.000275017600766314" rpy="0 0 0" />
       <mass value="6.0682081887272" />
-      <inertia ixx="0.0154034644119385" ixy="-2.22604627484569E-06" ixz="5.21108774696477E-09" iyy="0.0154080256643557" iyz="5.27262855355176E-09" izz="0.029708346400951" />
+      <inertia ixx="0.0154034644119385" ixy="-2.22604627484544E-06" ixz="5.21108774702054E-09" iyy="0.0154080256643557" iyz="5.27262855356307E-09" izz="0.029708346400951" />
     </inertial>
     <visual>
@@ -862,7 +862,7 @@
   <link name="wheel_1_link">
     <inertial>
-      <origin xyz="1.25478060125916E-05 5.22294298858916E-06 -0.00027501693981774" rpy="0 0 0" />
-      <mass value="6.06820810020003" />
-      <inertia ixx="0.0154034651258546" ixy="-2.22604258302274E-06" ixz="5.22035462687677E-09" iyy="0.0154080256614686" iyz="5.28562094393514E-09" izz="0.0297083471319844" />
+      <origin xyz="1.2547806012661E-05 5.22294298857529E-06 -0.00027501693981774" rpy="0 0 0" />
+      <mass value="6.06820810020002" />
+      <inertia ixx="0.0154034651258547" ixy="-2.22604258305555E-06" ixz="5.22035462340732E-09" iyy="0.0154080256614685" iyz="5.28562094397411E-09" izz="0.0297083471319844" />
     </inertial>
     <visual>
@@ -892,5 +892,5 @@
       <origin xyz="1.25474646742035E-05 5.22291550456022E-06 -0.000275016877356288" rpy="0 0 0" />
       <mass value="6.06820808425982" />
-      <inertia ixx="0.0154034651445229" ixy="-2.22601000971658E-06" ixz="5.20622353301233E-09" iyy="0.0154080256540422" iyz="5.28522507564306E-09" izz="0.0297083471441777" />
+      <inertia ixx="0.0154034651445229" ixy="-2.22601000971664E-06" ixz="5.20622353301233E-09" iyy="0.0154080256540422" iyz="5.28522507559181E-09" izz="0.0297083471441777" />
     </inertial>
     <visual>
@@ -916,3 +916,31 @@
     <axis xyz="0 0 1" />
   </joint>
+  <link name="docking_contact_link">
+    <inertial>
+      <origin xyz="0.000438848617413434 -0.178577146715673 -0.0110316356083883" rpy="0 0 0" />
+      <mass value="18.9261039673325" />
+      <inertia ixx="0.214992663147159" ixy="0.00083386140340347" ixz="-0.000588720101362879" iyy="0.22301041696344" iyz="-0.00155067556464412" izz="0.327845792807285" />
+    </inertial>
+    <visual>
+      <origin xyz="0 0 0" rpy="0 0 0" />
+      <geometry>
+        <mesh filename="$(arg model_mesh_dir)/docking_contact_link.STL" />
+      </geometry>
+      <material name="">
+        <color rgba="0.752941176470588 0.752941176470588 0.752941176470588 1" />
+      </material>
+    </visual>
+    <collision name="docking_contact_collision_link">
+      <origin xyz="0 0 0" rpy="0 0 0" />
+      <geometry>
+        <mesh filename="$(arg model_mesh_dir)/docking_contact_link.STL" />
+      </geometry>
+    </collision>
+  </link>
+  <joint name="docking_contact_frame" type="fixed">
+    <origin xyz="0 0.1768 0.107500004308165" rpy="0 0 0" />
+    <parent link="base_link" />
+    <child link="docking_contact_link" />
+    <axis xyz="0 0 0" />
+  </joint>
 </robot>

File: stretch4_urdf/SE4_tools/eoa_wrist_dw4_tool_sg4/eoa_wrist_dw4_tool_sg4.urdf (robot description, URDF)
Before this commit: robot URDF_DALI_ASSEM_Stretch_Gripper_V4, 8 links, 7 joints
Joints:
- joint aruco_fingertip_left_joint: origin xyz=3.80423e-05 -0.0335357 -0.00675433 rpy=1.37881 -2.50583e-06 0.62832 -> xyz=0.0335358 0.00675395 3.80134e-05 rpy=1.37881 -2.50583e-06 0.62832
- joint aruco_fingertip_right_joint: origin xyz=-3.81181e-05 0.0335357 0.00675399 rpy=1.37881 1.8123e-06 2.51327 -> xyz=-0.0335357 0.00675413 3.81175e-05 rpy=1.37881 1.8123e-06 2.51327
- joint grasp_center_joint: origin xyz=-0.234538 0 0 rpy=0 0 0 -> xyz=0.234538 0 0 rpy=0 0 -1.5708
- joint gripper_finger_left_joint: origin xyz=-0.0373909 -0.0222607 0 rpy=0 0 0 -> xyz=0.0373909 0.0222607 0 rpy=1.5708 0 3.14159
- joint gripper_finger_right_joint: origin xyz=-0.0373909 0.0222607 0 rpy=0 0 0 -> xyz=0.0373909 -0.0222607 0 rpy=1.5708 0 3.14159
- joint gripper_fingertip_left_joint: origin xyz=-0.191008 0.0221671 0 rpy=0.625614 -1.57079 0.945183 -> xyz=-0.191008 0 -0.022168 rpy=-1.5708 2.65359e-06 0
- joint gripper_fingertip_right_joint: origin xyz=-0.191008 -0.0221675 0 rpy=-0.625614 1.57079 -2.19641 -> xyz=-0.191008 0 0.022168 rpy=1.5708 -2.65359e-06 3.14159
