Commit message: Reducing manual changes to URDFs (#22)
* New URDF removes the need for manual TF manipulation

* Gripper camera fix and new docking contact link

* New surface-only mesh for sg4 gripper

* tablet and calibration board orientations

* Tool URDF updates

* Finger frame corrections for sg4

File: stretch4_urdf/SE4_tools/eoa_wrist_dw4_tool_sg4/eoa_wrist_dw4_tool_sg4.urdf (robot description, URDF)
Before this commit: robot URDF_DALI_ASSEM_Stretch_Gripper_V4, 8 links, 7 joints
Links:
- link aruco_fingertip_left_link: mass 0.000123521493853862 -> 0.000123521493853863
- link gripper_finger_left_link: mass 0.0196491261592472 -> 0.0196452088457426
- link gripper_finger_right_link: mass 0.0196451967584484 -> 0.0196451967584486
- link gripper_fingertip_left_link: mass 0.0147998681120424 -> 0.0155504911063414
- link gripper_fingertip_right_link: mass 0.0147998807271023 -> 0.0155505328279169
- link quick_connect_interface_link: mass 0.0917733059735497 -> 0.268266990446664
Joints:
- joint aruco_fingertip_left_joint: origin xyz=0.0335358 0.00675395 3.80134e-05 rpy=1.37881 -2.50583e-06 0.62832 -> xyz=-0.00441710992520833 -0.0320457043432331 0 rpy=1.37881010907552 0 0.698131700797736
- joint aruco_fingertip_right_joint: origin xyz=-0.0335357 0.00675413 3.81175e-05 rpy=1.37881 1.8123e-06 2.51327 -> xyz=-0.00441710992520835 0.0320457043432331 0 rpy=1.37881010907552 0 2.44346095279206
- joint grasp_center_joint: origin xyz=0.234538 0 0 rpy=0 0 -1.5708 -> xyz=0.23496234568483 0 0 rpy=0 0 0
- joint gripper_finger_left_joint: axis 0 1 0 -> 0 0 1; limit lower=0.0 upper=0.5 effort=0 velocity=0 -> lower=0 upper=0.5 effort=0 velocity=0; origin xyz=0.0373909 0.0222607 0 rpy=1.5708 0 3.14159 -> xyz=0.0378 0.022121 0 rpy=0 0 0
- joint gripper_finger_right_joint: axis 0 -1 0 -> 0 0 1; limit lower=0.0 upper=0.5 effort=0 velocity=0 -> lower=0 upper=0.5 effort=0 velocity=0; origin xyz=0.0373909 -0.0222607 0 rpy=1.5708 0 3.14159 -> xyz=0.0377995041255281 -0.0221213818384166 0 rpy=3.14159265358979 0 0
- joint gripper_fingertip_left_joint: origin xyz=-0.191008 0 -0.022168 rpy=-1.5708 2.65359e-06 0 -> xyz=0.191008332164325 -0.0221679999883927 0 rpy=0 0 -1.29154364647581
- joint gripper_fingertip_right_joint: origin xyz=-0.191008 0 0.022168 rpy=1.5708 -2.65359e-06 3.14159 -> xyz=0.191008332164326 -0.0221679999883885 0 rpy=3.14159265358979 0 -1.29154364647579

File: stretch4_urdf/SE4_tools/eoa_wrist_dw4_tool_tablet/eoa_wrist_dw4_tool_tablet.urdf (robot description, URDF)
Before this commit: robot URDF_DALI_ASSEM_Tablet_Mount_V3, 1 links, 0 joints
Links:
- link quick_connect_interface_link: mass 0.774816112828515 -> 0.755969840555698

Commit message: change sensor_0 name to line_sensor_0

File: stretch4_urdf/SE4_francis/xacro/stretch_main.xacro (robot description, xacro)
@@ -173,5 +173,5 @@
     <axis xyz="0 0 0" />
   </joint>
-  <link name="sensor_0_link">
+  <link name="line_sensor_0_link">
     <inertial>
       <origin xyz="0.00114502070313158 -0.000126774756058566 0.0119761602719025" rpy="0 0 0" />
@@ -182,5 +182,5 @@
       <origin xyz="0 0 0" rpy="0 0 0" />
       <geometry>
-        <mesh filename="$(arg model_mesh_dir)/sensor_0_link.STL" />
+        <mesh filename="$(arg model_mesh_dir)/line_sensor_0_link.STL" />
       </geometry>
       <material name="">
@@ -188,8 +188,8 @@
       </material>
     </visual>
-    <collision name="sensor_0_collision_link">
-      <origin xyz="0 0 0" rpy="0 0 0" />
-      <geometry>
-        <mesh filename="$(arg model_mesh_dir)/sensor_0_link.STL" />
+    <collision name="line_sensor_0_collision_link">
+      <origin xyz="0 0 0" rpy="0 0 0" />
+      <geometry>
+        <mesh filename="$(arg model_mesh_dir)/line_sensor_0_link.STL" />
       </geometry>
     </collision>
@@ -198,5 +198,5 @@
     <origin xyz="0.185120231404985 -0.0360000000000004 0.0527013981430276" rpy="0 0.453785605518531 0" />
     <parent link="base_link" />
-    <child link="sensor_0_link" />
+    <child link="line_sensor_0_link" />
     <axis xyz="0 0 0" />
   </joint>
@@ -205,5 +205,5 @@
   <joint name="line_sensor_0_optical_joint" type="fixed">
     <origin xyz="0.00286000000000003 0 0" rpy="-1.5707963267949 0 -1.5707963267949" />
-    <parent link="sensor_0_link" />
+    <parent link="line_sensor_0_link" />
     <child link="line_sensor_0_optical_link" />
     <axis xyz="0 0 0" />
