Commit message: Remove line_sensor_0 from visuals

File: stretch4_urdf/SE4_francis/xacro/stretch_main.xacro (robot description, xacro)
@@ -179,13 +179,4 @@
       <inertia ixx="2.88698160050477E-07" ixy="-5.64135957061259E-10" ixz="-7.07831726660262E-09" iyy="2.34959277592965E-07" iyz="-2.73972720709195E-10" izz="6.6461578229E-08" />
     </inertial>
-    <visual>
-      <origin xyz="0 0 0" rpy="0 0 0" />
-      <geometry>
-        <mesh filename="$(arg model_mesh_dir)/line_sensor_0_link.STL" />
-      </geometry>
-      <material name="">
-        <color rgba="0.792156862745098 0.819607843137255 0.933333333333333 1" />
-      </material>
-    </visual>
     <collision name="line_sensor_0_collision_link">
       <origin xyz="0 0 0" rpy="0 0 0" />

Commit message: Remove line_sensor_0 from collision

File: stretch4_urdf/SE4_francis/xacro/stretch_main.xacro (robot description, xacro)
@@ -179,10 +179,4 @@
       <inertia ixx="2.88698160050477E-07" ixy="-5.64135957061259E-10" ixz="-7.07831726660262E-09" iyy="2.34959277592965E-07" iyz="-2.73972720709195E-10" izz="6.6461578229E-08" />
     </inertial>
-    <collision name="line_sensor_0_collision_link">
-      <origin xyz="0 0 0" rpy="0 0 0" />
-      <geometry>
-        <mesh filename="$(arg model_mesh_dir)/line_sensor_0_link.STL" />
-      </geometry>
-    </collision>
   </link>
   <joint name="line_sensor_0_joint" type="fixed">

Commit message: Remove extra sensor meshes but leave lidar bounding boxes

File: stretch4_urdf/SE4_francis/xacro/stretch_main.xacro (robot description, xacro)
@@ -44,11 +44,5 @@
       <inertia ixx="2.88698160050487E-07" ixy="-5.64135957062421E-10" ixz="-7.07831726662328E-09" iyy="2.34959277592962E-07" iyz="-2.73972720709966E-10" izz="6.64615782289848E-08" />
     </inertial>
-    <collision name="line_sensor_5_collision_link">
-      <origin xyz="0 0 0" rpy="0 0 0" />
-      <geometry>
-        <mesh filename="$(arg model_mesh_dir)/line_sensor_5_link.STL" />
-      </geometry>
-    </collision>
-  </link>
+    </link>
   <joint name="line_sensor_5_joint" type="fixed">
     <origin xyz="0.0613832011662534 0.178318823151171 0.0527013981430276" rpy="0 0.453785605518531 1.04719755119659" />
@@ -71,11 +65,5 @@
       <inertia ixx="2.88698160050488E-07" ixy="-5.64135957060042E-10" ixz="-7.07831726662323E-09" iyy="2.34959277592962E-07" iyz="-2.73972720708353E-10" izz="6.6461578228985E-08" />
     </inertial>
-    <collision name="line_sensor_4_collision_link">
-      <origin xyz="0 0 0" rpy="0 0 0" />
-      <geometry>
-        <mesh filename="$(arg model_mesh_dir)/line_sensor_4_link.STL" />
-      </geometry>
-    </collision>
-  </link>
+    </link>
   <joint name="line_sensor_4_joint" type="fixed">
     <origin xyz="-0.0613832011662525 0.178318823151171 0.0527013981430276" rpy="0 0.453785605518532 2.09439510239319" />
@@ -98,11 +86,5 @@
       <inertia ixx="2.88698160050477E-07" ixy="-5.64135957061257E-10" ixz="-7.07831726660265E-09" iyy="2.34959277592965E-07" iyz="-2.73972720709266E-10" izz="6.64615782289998E-08" />
     </inertial>
-    <collision name="line_sensor_3_collision_link">
-      <origin xyz="0 0 0" rpy="0 0 0" />
-      <geometry>
-        <mesh filename="$(arg model_mesh_dir)/line_sensor_3_link.STL" />
-      </geometry>
-    </collision>
-  </link>
+    </link>
   <joint name="line_sensor_3_joint" type="fixed">
     <origin xyz="-0.185120231404985 -0.036 0.0527013981430276" rpy="0 0.453785605518531 -3.14159265358979" />
@@ -125,11 +107,5 @@
       <inertia ixx="2.88698160050489E-07" ixy="-5.64135957062399E-10" ixz="-7.07831726662342E-09" iyy="2.34959277592963E-07" iyz="-2.73972720710027E-10" izz="6.64615782289852E-08" />
     </inertial>
-    <collision name="line_sensor_2_collision_link">
-      <origin xyz="0 0 0" rpy="0 0 0" />
-      <geometry>
-        <mesh filename="$(arg model_mesh_dir)/line_sensor_2_link.STL" />
-      </geometry>
-    </collision>
-  </link>
+    </link>
   <joint name="line_sensor_2_joint" type="fixed">
     <origin xyz="-0.123737030238733 -0.14231882315117 0.0527013981430276" rpy="0 0.453785605518531 -2.0943951023932" />
@@ -152,11 +128,5 @@
       <inertia ixx="2.88698160050487E-07" ixy="-5.64135957060014E-10" ixz="-7.0783172666233E-09" iyy="2.34959277592961E-07" iyz="-2.73972720708438E-10" izz="6.64615782289849E-08" />
     </inertial>
-    <collision name="line_sensor_1_collision_link">
-      <origin xyz="0 0 0" rpy="0 0 0" />
-      <geometry>
-        <mesh filename="$(arg model_mesh_dir)/line_sensor_1_link.STL" />
-      </geometry>
-    </collision>
-  </link>
+    </link>
   <joint name="line_sensor_1_joint" type="fixed">
     <origin xyz="0.123737030238732 -0.142318823151171 0.0527013981430276" rpy="0 0.453785605518531 -1.0471975511966" />
@@ -179,5 +149,5 @@
       <inertia ixx="2.88698160050477E-07" ixy="-5.64135957061259E-10" ixz="-7.07831726660262E-09" iyy="2.34959277592965E-07" iyz="-2.73972720709195E-10" izz="6.6461578229E-08" />
     </inertial>
-  </link>
+    </link>
   <joint name="line_sensor_0_joint" type="fixed">
     <origin xyz="0.185120231404985 -0.0360000000000004 0.0527013981430276" rpy="0 0.453785605518531 0" />
@@ -231,5 +201,5 @@
       <origin xyz="0 0 0" rpy="0 0 0" />
       <geometry>
-        <mesh filename="$(arg model_mesh_dir)/lidar_right_link.STL" />
+        <mesh filename="$(arg model_mesh_dir)/lidar_right_collision_link.STL" />
       </geometry>
     </collision>
@@ -250,5 +220,5 @@
       <origin xyz="0 0 0" rpy="0 0 0" />
       <geometry>
-        <mesh filename="$(arg model_mesh_dir)/lidar_left_link.STL" />
+        <mesh filename="$(arg model_mesh_dir)/lidar_left_collision_link.STL" />
       </geometry>
     </collision>
@@ -266,11 +236,5 @@
       <inertia ixx="0.0518045670378195" ixy="-0.0128492794593393" ixz="-9.71150764633997E-05" iyy="0.0504717539658347" iyz="-0.000186491771284797" izz="0.0306330355634591" />
     </inertial>
-    <collision name="camera_right_collision_link">
-      <origin xyz="0 0 0" rpy="0 0 0" />
-      <geometry>
-        <mesh filename="$(arg model_mesh_dir)/camera_right_link.STL" />
-      </geometry>
-    </collision>
-  </link>
+    </link>
   <joint name="camera_right_joint" type="fixed">
     <origin xyz="0.171840602787894 0.0230000000000032 -0.0157566987072475" rpy="1.5707963267949 0.820304748437337 0" />
@@ -293,11 +257,5 @@
       <inertia ixx="0.0518045670378195" ixy="0.0128492794593393" ixz="9.71150764634412E-05" iyy="0.0504717539658347" iyz="-0.000186491771284767" izz="0.0306330355634591" />
     </inertial>
-    <collision name="camera_left_collision_link">
-      <origin xyz="0 0 0" rpy="0 0 0" />
-      <geometry>
-        <mesh filename="$(arg model_mesh_dir)/camera_left_link.STL" />
-      </geometry>
-    </collision>
-  </link>
+    </link>
   <joint name="camera_left_joint" type="fixed">
     <origin xyz="0.171840602787895 0.173 -0.0157566987072475" rpy="-1.5707963267949 0.820304748437337 0" />
@@ -320,11 +278,5 @@
       <inertia ixx="0.0465206803724917" ixy="0.0120094528414331" ixz="0.000133766698529184" iyy="0.0557556406311624" iyz="-0.000162225118887392" izz="0.0306330355634591" />
     </inertial>
-    <collision name="camera_center_collision_link">
-      <origin xyz="0 0 0" rpy="0 0 0" />
-      <geometry>
-        <mesh filename="$(arg model_mesh_dir)/camera_center_link.STL" />
-      </geometry>
-    </collision>
-  </link>
+    </link>
   <joint name="camera_center_joint" type="fixed">
     <origin xyz="0.177245603402412 0.0980000000000004 -0.0239069097938973" rpy="-1.5707963267949 0.610865238198018 0" />

Commit message: Remove all sensor links + collisions, make the head a bounding box

File: stretch4_urdf/SE4_francis/xacro/stretch_main.xacro (robot description, xacro)
@@ -198,11 +198,5 @@
       <inertia ixx="0.0492829863501233" ixy="-0.0015644794553125" ixz="0.0149316959819942" iyy="0.0349356509390749" iyz="0.00380036135309891" izz="0.0486907192779151" />
     </inertial>
-    <collision name="lidar_right_collision_link">
-      <origin xyz="0 0 0" rpy="0 0 0" />
-      <geometry>
-        <mesh filename="$(arg model_mesh_dir)/lidar_right_collision_link.STL" />
-      </geometry>
-    </collision>
-  </link>
+    </link>
   <joint name="lidar_right_joint" type="fixed">
     <origin xyz="0.131744211811827 -0.0264137425448753 -0.0583279884119643" rpy="-3.05465659239941 0.781600065124168 2.39203005564319" />
@@ -217,11 +211,5 @@
       <inertia ixx="0.0495631508318921" ixy="0.00150375867091917" ixz="-0.0147241234604212" iyy="0.034541985578385" iyz="0.00388339874636519" izz="0.0488042201568361" />
     </inertial>
-    <collision name="lidar_left_collision_link">
-      <origin xyz="0 0 0" rpy="0 0 0" />
-      <geometry>
-        <mesh filename="$(arg model_mesh_dir)/lidar_left_collision_link.STL" />
-      </geometry>
-    </collision>
-  </link>
+    </link>
   <joint name="lidar_left_joint" type="fixed">
     <origin xyz="0.131744211811846 0.222413742544858 -0.0583279884119634" rpy="-3.05465659239939 -0.781600065124167 0.749562597946573" />

Commit message: head+lift collision fix (#33)
* Remove all sensor visuals + collisions, make the head a bounding box

File: stretch4_urdf/SE4_francis/xacro/stretch_main.xacro (robot description, xacro)
@@ -44,11 +44,5 @@
       <inertia ixx="2.88698160050487E-07" ixy="-5.64135957062421E-10" ixz="-7.07831726662328E-09" iyy="2.34959277592962E-07" iyz="-2.73972720709966E-10" izz="6.64615782289848E-08" />
     </inertial>
-    <collision name="line_sensor_5_collision_link">
-      <origin xyz="0 0 0" rpy="0 0 0" />
-      <geometry>
-        <mesh filename="$(arg model_mesh_dir)/line_sensor_5_link.STL" />
-      </geometry>
-    </collision>
-  </link>
+    </link>
   <joint name="line_sensor_5_joint" type="fixed">
     <origin xyz="0.0613832011662534 0.178318823151171 0.0527013981430276" rpy="0 0.453785605518531 1.04719755119659" />
@@ -71,11 +65,5 @@
       <inertia ixx="2.88698160050488E-07" ixy="-5.64135957060042E-10" ixz="-7.07831726662323E-09" iyy="2.34959277592962E-07" iyz="-2.73972720708353E-10" izz="6.6461578228985E-08" />
     </inertial>
-    <collision name="line_sensor_4_collision_link">
-      <origin xyz="0 0 0" rpy="0 0 0" />
-      <geometry>
-        <mesh filename="$(arg model_mesh_dir)/line_sensor_4_link.STL" />
-      </geometry>
-    </collision>
-  </link>
+    </link>
   <joint name="line_sensor_4_joint" type="fixed">
     <origin xyz="-0.0613832011662525 0.178318823151171 0.0527013981430276" rpy="0 0.453785605518532 2.09439510239319" />
@@ -98,11 +86,5 @@
       <inertia ixx="2.88698160050477E-07" ixy="-5.64135957061257E-10" ixz="-7.07831726660265E-09" iyy="2.34959277592965E-07" iyz="-2.73972720709266E-10" izz="6.64615782289998E-08" />
     </inertial>
-    <collision name="line_sensor_3_collision_link">
-      <origin xyz="0 0 0" rpy="0 0 0" />
-      <geometry>
-        <mesh filename="$(arg model_mesh_dir)/line_sensor_3_link.STL" />
-      </geometry>
-    </collision>
-  </link>
+    </link>
   <joint name="line_sensor_3_joint" type="fixed">
     <origin xyz="-0.185120231404985 -0.036 0.0527013981430276" rpy="0 0.453785605518531 -3.14159265358979" />
@@ -125,11 +107,5 @@
       <inertia ixx="2.88698160050489E-07" ixy="-5.64135957062399E-10" ixz="-7.07831726662342E-09" iyy="2.34959277592963E-07" iyz="-2.73972720710027E-10" izz="6.64615782289852E-08" />
     </inertial>
-    <collision name="line_sensor_2_collision_link">
-      <origin xyz="0 0 0" rpy="0 0 0" />
-      <geometry>
-        <mesh filename="$(arg model_mesh_dir)/line_sensor_2_link.STL" />
-      </geometry>
-    </collision>
-  </link>
+    </link>
   <joint name="line_sensor_2_joint" type="fixed">
     <origin xyz="-0.123737030238733 -0.14231882315117 0.0527013981430276" rpy="0 0.453785605518531 -2.0943951023932" />
@@ -152,11 +128,5 @@
       <inertia ixx="2.88698160050487E-07" ixy="-5.64135957060014E-10" ixz="-7.0783172666233E-09" iyy="2.34959277592961E-07" iyz="-2.73972720708438E-10" izz="6.64615782289849E-08" />
     </inertial>
-    <collision name="line_sensor_1_collision_link">
-      <origin xyz="0 0 0" rpy="0 0 0" />
-      <geometry>
-        <mesh filename="$(arg model_mesh_dir)/line_sensor_1_link.STL" />
-      </geometry>
-    </collision>
-  </link>
+    </link>
   <joint name="line_sensor_1_joint" type="fixed">
     <origin xyz="0.123737030238732 -0.142318823151171 0.0527013981430276" rpy="0 0.453785605518531 -1.0471975511966" />
@@ -179,20 +149,5 @@
       <inertia ixx="2.88698160050477E-07" ixy="-5.64135957061259E-10" ixz="-7.07831726660262E-09" iyy="2.34959277592965E-07" iyz="-2.73972720709195E-10" izz="6.6461578229E-08" />
     </inertial>
-    <visual>
-      <origin xyz="0 0 0" rpy="0 0 0" />
-      <geometry>
-        <mesh filename="$(arg model_mesh_dir)/line_sensor_0_link.STL" />
-      </geometry>
-      <material name="">
-        <color rgba="0.792156862745098 0.819607843137255 0.933333333333333 1" />
-      </material>
-    </visual>
-    <collision name="line_sensor_0_collision_link">
-      <origin xyz="0 0 0" rpy="0 0 0" />
-      <geometry>
-        <mesh filename="$(arg model_mesh_dir)/line_sensor_0_link.STL" />
-      </geometry>
-    </collision>
-  </link>
+    </link>
   <joint name="line_sensor_0_joint" type="fixed">
     <origin xyz="0.185120231404985 -0.0360000000000004 0.0527013981430276" rpy="0 0.453785605518531 0" />
@@ -243,11 +198,5 @@
       <inertia ixx="0.0492829863501233" ixy="-0.0015644794553125" ixz="0.0149316959819942" iyy="0.0349356509390749" iyz="0.00380036135309891" izz="0.0486907192779151" />
     </inertial>
-    <collision name="lidar_right_collision_link">
-      <origin xyz="0 0 0" rpy="0 0 0" />
-      <geometry>
-        <mesh filename="$(arg model_mesh_dir)/lidar_right_link.STL" />
-      </geometry>
-    </collision>
-  </link>
+    </link>
   <joint name="lidar_right_joint" type="fixed">
     <origin xyz="0.131744211811827 -0.0264137425448753 -0.0583279884119643" rpy="-3.05465659239941 0.781600065124168 2.39203005564319" />
@@ -262,11 +211,5 @@
       <inertia ixx="0.0495631508318921" ixy="0.00150375867091917" ixz="-0.0147241234604212" iyy="0.034541985578385" iyz="0.00388339874636519" izz="0.0488042201568361" />
     </inertial>
-    <collision name="lidar_left_collision_link">
-      <origin xyz="0 0 0" rpy="0 0 0" />
-      <geometry>
-        <mesh filename="$(arg model_mesh_dir)/lidar_left_link.STL" />
-      </geometry>
-    </collision>
-  </link>
+    </link>
   <joint name="lidar_left_joint" type="fixed">
     <origin xyz="0.131744211811846 0.222413742544858 -0.0583279884119634" rpy="-3.05465659239939 -0.781600065124167 0.749562597946573" />
@@ -281,11 +224,5 @@
       <inertia ixx="0.0518045670378195" ixy="-0.0128492794593393" ixz="-9.71150764633997E-05" iyy="0.0504717539658347" iyz="-0.000186491771284797" izz="0.0306330355634591" />
     </inertial>
-    <collision name="camera_right_collision_link">
-      <origin xyz="0 0 0" rpy="0 0 0" />
-      <geometry>
-        <mesh filename="$(arg model_mesh_dir)/camera_right_link.STL" />
-      </geometry>
-    </collision>
-  </link>
+    </link>
   <joint name="camera_right_joint" type="fixed">
     <origin xyz="0.171840602787894 0.0230000000000032 -0.0157566987072475" rpy="1.5707963267949 0.820304748437337 0" />
@@ -308,11 +245,5 @@
       <inertia ixx="0.0518045670378195" ixy="0.0128492794593393" ixz="9.71150764634412E-05" iyy="0.0504717539658347" iyz="-0.000186491771284767" izz="0.0306330355634591" />
     </inertial>
-    <collision name="camera_left_collision_link">
-      <origin xyz="0 0 0" rpy="0 0 0" />
-      <geometry>
-        <mesh filename="$(arg model_mesh_dir)/camera_left_link.STL" />
-      </geometry>
-    </collision>
-  </link>
+    </link>
   <joint name="camera_left_joint" type="fixed">
     <origin xyz="0.171840602787895 0.173 -0.0157566987072475" rpy="-1.5707963267949 0.820304748437337 0" />
@@ -335,11 +266,5 @@
       <inertia ixx="0.0465206803724917" ixy="0.0120094528414331" ixz="0.000133766698529184" iyy="0.0557556406311624" iyz="-0.000162225118887392" izz="0.0306330355634591" />
     </inertial>
-    <collision name="camera_center_collision_link">
-      <origin xyz="0 0 0" rpy="0 0 0" />
-      <geometry>
-        <mesh filename="$(arg model_mesh_dir)/camera_center_link.STL" />
-      </geometry>
-    </collision>
-  </link>
+    </link>
   <joint name="camera_center_joint" type="fixed">
     <origin xyz="0.177245603402412 0.0980000000000004 -0.0239069097938973" rpy="-1.5707963267949 0.610865238198018 0" />

Commit message: SE4_francis joint limits

File: stretch4_urdf/SE4_francis/xacro/stretch_main.xacro (robot description, xacro)
@@ -4,10 +4,11 @@
       <origin xyz="0 0 0" rpy="0 0 0" />
       <geometry>
-        <box size="0.001 0.001 0.001" /></geometry>
-      <material name="">
-        <color rgba="0.752941176470588 0.752941176470588 0.752941176470588 1" />
-      </material>
-    </visual>
-    </link>
+        <box size="0.001 0.001 0.001" />
+      </geometry>
+      <material name="">
+        <color rgba="0.752941176470588 0.752941176470588 0.752941176470588 1" />
+      </material>
+    </visual>
+  </link>
   <link name="base_link">
     <inertial>
@@ -349,21 +350,10 @@
     </collision>
   </link>
-  <joint
-    name="lift_joint"
-    type="prismatic">
-    <origin
-      xyz="0 -0.00140000000000005 0.241"
-      rpy="0 0 0" />
-    <parent
-      link="mast_link" />
-    <child
-      link="lift_link" />
-    <axis
-      xyz="0 0 1" />
-    <limit
-      lower="0"
-      upper="1.2"
-      effort="0"
-      velocity="0" />
+  <joint name="lift_joint" type="prismatic">
+    <origin xyz="0 -0.00140000000000005 0.241" rpy="0 0 0" />
+    <parent link="mast_link" />
+    <child link="lift_link" />
+    <axis xyz="0 0 1" />
+    <limit lower="0" upper="1.2" effort="0" velocity="0.5" />
   </joint>
   <link
@@ -447,5 +437,5 @@
     <child link="arm_l1_link" />
     <axis xyz="1 0 0" />
-    <limit lower="0" upper="0.13" effort="0" velocity="0" />
+    <limit lower="0" upper="0.13" effort="0" velocity="0.7" />
   </joint>
   <link name="arm_l2_link">
@@ -476,5 +466,5 @@
     <child link="arm_l2_link" />
     <axis xyz="1 0 0" />
-    <limit lower="0" upper="0.13" effort="0" velocity="0" />
+    <limit lower="0" upper="0.13" effort="0" velocity="0.7" />
   </joint>
   <link name="arm_l3_link">
@@ -505,5 +495,5 @@
     <child link="arm_l3_link" />
     <axis xyz="1 0 0" />
-    <limit lower="0" upper="0.13" effort="0" velocity="0" />
+    <limit lower="0" upper="0.13" effort="0" velocity="0.7" />
   </joint>
   <link name="arm_l4_link">
@@ -534,5 +524,5 @@
     <child link="arm_l4_link" />
     <axis xyz="1 0 0" />
-    <limit lower="0" upper="0.13" effort="0" velocity="0" />
+    <limit lower="0" upper="0.13" effort="0" velocity="0.7" />
   </joint>
   <link name="wrist_link">
@@ -591,5 +581,5 @@
     <child link="wrist_yaw_link" />
     <axis xyz="0 0 1" />
-    <limit lower="-1.135" upper="4.276" effort="0" velocity="0" />
+    <limit lower="-1.135" upper="4.276" effort="20.0" velocity="12.0" />
   </joint>
   <link name="wrist_pitch_link">
@@ -620,5 +610,5 @@
     <child link="wrist_pitch_link" />
     <axis xyz="0 1 0" />
-    <limit lower="-1.135" upper="4.276" effort="0" velocity="0" />
+    <limit lower="-1.135" upper="4.276" effort="20.0" velocity="12.0" />
   </joint>
   <link name="wrist_roll_link">
@@ -649,5 +639,5 @@
     <child link="wrist_roll_link" />
     <axis xyz="1 0 0" />
-    <limit lower="-4.276" upper="1.135" effort="0" velocity="0" />
+    <limit lower="-4.276" upper="1.135" effort="20.0" velocity="12.0" />
   </joint>
   <link name="gripper_camera_link">
@@ -683,10 +673,11 @@
       <origin xyz="0 0 0" rpy="0 0 0" />
       <geometry>
-        <box size="0.001 0.001 0.001" /></geometry>
+        <box size="0.001 0.001 0.001" />
+      </geometry>
       <material name="">
         <color rgba="0.792156862745098 0.819607843137255 0.933333333333333 1" />
       </material>
     </visual>
-    </link>
+  </link>
   <joint name="gripper_stereo_camera_color_optical_joint" type="fixed">
     <origin xyz="0 0 0" rpy="-1.51843644923507 0 -1.5707963267949" />
@@ -699,10 +690,11 @@
       <origin xyz="0 0 0" rpy="0 0 0" />
       <geometry>
-        <box size="0.001 0.001 0.001" /></geometry>
+        <box size="0.001 0.001 0.001" />
+      </geometry>
       <material name="">
         <color rgba="0.792156862745098 0.819607843137255 0.933333333333333 1" />
       </material>
     </visual>
-    </link>
+  </link>
   <joint name="gripper_right_camera_color_optical_joint" type="fixed">
     <origin xyz="0 -0.01 0" rpy="-1.51843644923507 0 -1.5707963267949" />
@@ -715,10 +707,11 @@
       <origin xyz="0 0 0" rpy="0 0 0" />
       <geometry>
-        <box size="0.001 0.001 0.001" /></geometry>
+        <box size="0.001 0.001 0.001" />
+      </geometry>
       <material name="">
         <color rgba="0.792156862745098 0.819607843137255 0.933333333333333 1" />
       </material>
     </visual>
-    </link>
+  </link>
   <joint name="gripper_left_camera_color_optical_joint" type="fixed">
     <origin xyz="0 0.01 0" rpy="-1.51843644923507 0 -1.5707963267949" />
@@ -838,4 +831,5 @@
     <child link="wheel_2_link" />
     <axis xyz="0 0 1" />
+    <limit />
   </joint>
   <link name="wheel_1_link">
@@ -866,4 +860,5 @@
     <child link="wheel_1_link" />
     <axis xyz="0 0 1" />
+    <limit />
   </joint>
   <link name="wheel_0_link">
@@ -894,4 +889,5 @@
     <child link="wheel_0_link" />
     <axis xyz="0 0 1" />
+    <limit />
   </joint>
   <link name="docking_contact_link">
