Commit message: SE4_francis joint limits

File: stretch4_urdf/SE4_francis/xacro/stretch_main.xacro (robot description, xacro)
@@ -4,10 +4,11 @@
       <origin xyz="0 0 0" rpy="0 0 0" />
       <geometry>
-        <box size="0.001 0.001 0.001" /></geometry>
-      <material name="">
-        <color rgba="0.752941176470588 0.752941176470588 0.752941176470588 1" />
-      </material>
-    </visual>
-    </link>
+        <box size="0.001 0.001 0.001" />
+      </geometry>
+      <material name="">
+        <color rgba="0.752941176470588 0.752941176470588 0.752941176470588 1" />
+      </material>
+    </visual>
+  </link>
   <link name="base_link">
     <inertial>
@@ -336,5 +337,5 @@
     <child link="lift_link" />
     <axis xyz="0 0 1" />
-    <limit lower="0" upper="1.2" effort="0" velocity="0" />
+    <limit lower="0" upper="1.2" effort="0" velocity="0.5" />
   </joint>
   <link name="arm_l0_link">
@@ -393,5 +394,5 @@
     <child link="arm_l1_link" />
     <axis xyz="1 0 0" />
-    <limit lower="0" upper="0.13" effort="0" velocity="0" />
+    <limit lower="0" upper="0.13" effort="0" velocity="0.7" />
   </joint>
   <link name="arm_l2_link">
@@ -422,5 +423,5 @@
     <child link="arm_l2_link" />
     <axis xyz="1 0 0" />
-    <limit lower="0" upper="0.13" effort="0" velocity="0" />
+    <limit lower="0" upper="0.13" effort="0" velocity="0.7" />
   </joint>
   <link name="arm_l3_link">
@@ -451,5 +452,5 @@
     <child link="arm_l3_link" />
     <axis xyz="1 0 0" />
-    <limit lower="0" upper="0.13" effort="0" velocity="0" />
+    <limit lower="0" upper="0.13" effort="0" velocity="0.7" />
   </joint>
   <link name="arm_l4_link">
@@ -480,5 +481,5 @@
     <child link="arm_l4_link" />
     <axis xyz="1 0 0" />
-    <limit lower="0" upper="0.13" effort="0" velocity="0" />
+    <limit lower="0" upper="0.13" effort="0" velocity="0.7" />
   </joint>
   <link name="wrist_link">
@@ -537,5 +538,5 @@
     <child link="wrist_yaw_link" />
     <axis xyz="0 0 1" />
-    <limit lower="-1.135" upper="4.276" effort="0" velocity="0" />
+    <limit lower="-1.135" upper="4.276" effort="20.0" velocity="12.0" />
   </joint>
   <link name="wrist_pitch_link">
@@ -566,5 +567,5 @@
     <child link="wrist_pitch_link" />
     <axis xyz="0 1 0" />
-    <limit lower="-1.135" upper="4.276" effort="0" velocity="0" />
+    <limit lower="-1.135" upper="4.276" effort="20.0" velocity="12.0" />
   </joint>
   <link name="wrist_roll_link">
@@ -595,5 +596,5 @@
     <child link="wrist_roll_link" />
     <axis xyz="1 0 0" />
-    <limit lower="-4.276" upper="1.135" effort="0" velocity="0" />
+    <limit lower="-4.276" upper="1.135" effort="20.0" velocity="12.0" />
   </joint>
   <link name="gripper_camera_link">
@@ -629,10 +630,11 @@
       <origin xyz="0 0 0" rpy="0 0 0" />
       <geometry>
-        <box size="0.001 0.001 0.001" /></geometry>
+        <box size="0.001 0.001 0.001" />
+      </geometry>
       <material name="">
         <color rgba="0.792156862745098 0.819607843137255 0.933333333333333 1" />
       </material>
     </visual>
-    </link>
+  </link>
   <joint name="gripper_stereo_camera_color_optical_joint" type="fixed">
     <origin xyz="0 0 0" rpy="-1.51843644923507 0 -1.5707963267949" />
@@ -645,10 +647,11 @@
       <origin xyz="0 0 0" rpy="0 0 0" />
       <geometry>
-        <box size="0.001 0.001 0.001" /></geometry>
+        <box size="0.001 0.001 0.001" />
+      </geometry>
       <material name="">
         <color rgba="0.792156862745098 0.819607843137255 0.933333333333333 1" />
       </material>
     </visual>
-    </link>
+  </link>
   <joint name="gripper_right_camera_color_optical_joint" type="fixed">
     <origin xyz="0 -0.01 0" rpy="-1.51843644923507 0 -1.5707963267949" />
@@ -661,10 +664,11 @@
       <origin xyz="0 0 0" rpy="0 0 0" />
       <geometry>
-        <box size="0.001 0.001 0.001" /></geometry>
+        <box size="0.001 0.001 0.001" />
+      </geometry>
       <material name="">
         <color rgba="0.792156862745098 0.819607843137255 0.933333333333333 1" />
       </material>
     </visual>
-    </link>
+  </link>
   <joint name="gripper_left_camera_color_optical_joint" type="fixed">
     <origin xyz="0 0.01 0" rpy="-1.51843644923507 0 -1.5707963267949" />
@@ -784,4 +788,5 @@
     <child link="wheel_2_link" />
     <axis xyz="0 0 1" />
+    <limit />
   </joint>
   <link name="wheel_1_link">
@@ -812,4 +817,5 @@
     <child link="wheel_1_link" />
     <axis xyz="0 0 1" />
+    <limit />
   </joint>
   <link name="wheel_0_link">
@@ -840,4 +846,5 @@
     <child link="wheel_0_link" />
     <axis xyz="0 0 1" />
+    <limit />
   </joint>
   <link name="docking_contact_link">

Commit message: Do not add empty limit tags

File: stretch4_urdf/SE4_francis/xacro/stretch_main.xacro (robot description, xacro)
@@ -788,5 +788,4 @@
     <child link="wheel_2_link" />
     <axis xyz="0 0 1" />
-    <limit />
   </joint>
   <link name="wheel_1_link">
@@ -817,5 +816,4 @@
     <child link="wheel_1_link" />
     <axis xyz="0 0 1" />
-    <limit />
   </joint>
   <link name="wheel_0_link">
@@ -846,5 +844,4 @@
     <child link="wheel_0_link" />
     <axis xyz="0 0 1" />
-    <limit />
   </joint>
   <link name="docking_contact_link">

Commit message: Do not add empty limit tags

File: stretch4_urdf/SE4_francis/xacro/stretch_main.xacro (robot description, xacro)
@@ -831,5 +831,4 @@
     <child link="wheel_2_link" />
     <axis xyz="0 0 1" />
-    <limit />
   </joint>
   <link name="wheel_1_link">
@@ -860,5 +859,4 @@
     <child link="wheel_1_link" />
     <axis xyz="0 0 1" />
-    <limit />
   </joint>
   <link name="wheel_0_link">
@@ -889,5 +887,4 @@
     <child link="wheel_0_link" />
     <axis xyz="0 0 1" />
-    <limit />
   </joint>
   <link name="docking_contact_link">

Commit message: New camera optical frame definitions

File: stretch4_urdf/SE4_francis/xacro/stretch_main.xacro (robot description, xacro)
@@ -226,5 +226,5 @@
     </link>
   <joint name="camera_right_joint" type="fixed">
-    <origin xyz="0.171840602787894 0.0230000000000032 -0.0157566987072475" rpy="1.5707963267949 0.820304748437337 0" />
+    <origin xyz="0.171840602787894 0.0230000000000032 -0.0157566987072475" rpy="0 0.820304748437337 0" />
     <parent link="head_link" />
     <child link="camera_right_link" />
@@ -234,5 +234,5 @@
     </link>
   <joint name="camera_right_optical_joint" type="fixed">
-    <origin xyz="0.0212000000000001 0 0" rpy="-1.5707963267949 0 -1.5707963267949" />
+    <origin xyz="0.0212000000000001 0 0" rpy="0 1.5707963267948966 0" />
     <parent link="camera_right_link" />
     <child link="camera_right_optical_link" />
@@ -247,5 +247,5 @@
     </link>
   <joint name="camera_left_joint" type="fixed">
-    <origin xyz="0.171840602787895 0.173 -0.0157566987072475" rpy="-1.5707963267949 0.820304748437337 0" />
+    <origin xyz="0.171840602787895 0.173 -0.0157566987072475" rpy="0 0.820304748437337 0" />
     <parent link="head_link" />
     <child link="camera_left_link" />
@@ -255,5 +255,5 @@
     </link>
   <joint name="camera_left_optical_joint" type="fixed">
-    <origin xyz="0.0211999999999999 0 0" rpy="-1.5707963267949 0 -1.5707963267949" />
+    <origin xyz="0.0211999999999999 0 0" rpy="3.141592653589793 -1.5707963267948966 0" />
     <parent link="camera_left_link" />
     <child link="camera_left_optical_link" />
@@ -268,5 +268,5 @@
     </link>
   <joint name="camera_center_joint" type="fixed">
-    <origin xyz="0.177245603402412 0.0980000000000004 -0.0239069097938973" rpy="-1.5707963267949 0.610865238198018 0" />
+    <origin xyz="0.177245603402412 0.0980000000000004 -0.0239069097938973" rpy="0 0.610865238198018 0" />
     <parent link="head_link" />
     <child link="camera_center_link" />
@@ -276,5 +276,5 @@
     </link>
   <joint name="camera_center_optical_joint" type="fixed">
-    <origin xyz="0.00170000000000003 0 0" rpy="-1.5707963267949 0 -1.5707963267949" />
+    <origin xyz="0.00170000000000003 0 0" rpy="0 1.5707963267948966 0" />
     <parent link="camera_center_link" />
     <child link="camera_center_optical_link" />

Commit message: Rename optical links to use expected luxonis names

File: stretch4_urdf/SE4_francis/xacro/stretch_main.xacro (robot description, xacro)
@@ -231,10 +231,10 @@
     <axis xyz="0 0 0" />
   </joint>
-  <link name="camera_right_optical_link">
+  <link name="cameras_head_right_camera_optical_frame">
     </link>
   <joint name="camera_right_optical_joint" type="fixed">
     <origin xyz="0.0212000000000001 0 0" rpy="0 1.5707963267948966 0" />
     <parent link="camera_right_link" />
-    <child link="camera_right_optical_link" />
+    <child link="cameras_head_right_camera_optical_frame" />
     <axis xyz="0 0 0" />
   </joint>
@@ -252,10 +252,10 @@
     <axis xyz="0 0 0" />
   </joint>
-  <link name="camera_left_optical_link">
+  <link name="cameras_head_left_camera_optical_frame">
     </link>
   <joint name="camera_left_optical_joint" type="fixed">
     <origin xyz="0.0211999999999999 0 0" rpy="3.141592653589793 -1.5707963267948966 0" />
     <parent link="camera_left_link" />
-    <child link="camera_left_optical_link" />
+    <child link="cameras_head_left_camera_optical_frame" />
     <axis xyz="0 0 0" />
   </joint>
@@ -273,10 +273,10 @@
     <axis xyz="0 0 0" />
   </joint>
-  <link name="camera_center_optical_link">
+  <link name="cameras_head_center_camera_optical_frame">
     </link>
   <joint name="camera_center_optical_joint" type="fixed">
     <origin xyz="0.00170000000000003 0 0" rpy="0 1.5707963267948966 0" />
     <parent link="camera_center_link" />
-    <child link="camera_center_optical_link" />
+    <child link="cameras_head_center_camera_optical_frame" />
     <axis xyz="0 0 0" />
   </joint>

Commit message: I think I understand opencv now

File: stretch4_urdf/SE4_francis/xacro/stretch_main.xacro (robot description, xacro)
@@ -234,5 +234,5 @@
     </link>
   <joint name="camera_right_optical_joint" type="fixed">
-    <origin xyz="0.0212000000000001 0 0" rpy="0 1.5707963267948966 0" />
+    <origin xyz="0.0212000000000001 0 0" rpy="3.141592653589793 -1.5707963267948966 0" />
     <parent link="camera_right_link" />
     <child link="cameras_head_right_camera_optical_frame" />
@@ -255,5 +255,5 @@
     </link>
   <joint name="camera_left_optical_joint" type="fixed">
-    <origin xyz="0.0211999999999999 0 0" rpy="3.141592653589793 -1.5707963267948966 0" />
+    <origin xyz="0.0211999999999999 0 0" rpy="0 1.5707963267948966 0" />
     <parent link="camera_left_link" />
     <child link="cameras_head_left_camera_optical_frame" />
@@ -276,5 +276,5 @@
     </link>
   <joint name="camera_center_optical_joint" type="fixed">
-    <origin xyz="0.00170000000000003 0 0" rpy="0 1.5707963267948966 0" />
+    <origin xyz="0.00170000000000003 0 0" rpy="3.141592653589793 -1.5707963267948966 0" />
     <parent link="camera_center_link" />
     <child link="cameras_head_center_camera_optical_frame" />

Commit message: Changed the optical frame links back to their original urdf names instead of the luxonis ros names

File: stretch4_urdf/SE4_francis/xacro/stretch_main.xacro (robot description, xacro)
@@ -231,10 +231,10 @@
     <axis xyz="0 0 0" />
   </joint>
-  <link name="cameras_head_right_camera_optical_frame">
+  <link name="camera_right_optical_link">
     </link>
   <joint name="camera_right_optical_joint" type="fixed">
     <origin xyz="0.0212000000000001 0 0" rpy="3.141592653589793 -1.5707963267948966 0" />
     <parent link="camera_right_link" />
-    <child link="cameras_head_right_camera_optical_frame" />
+    <child link="camera_right_optical_link" />
     <axis xyz="0 0 0" />
   </joint>
@@ -252,10 +252,10 @@
     <axis xyz="0 0 0" />
   </joint>
-  <link name="cameras_head_left_camera_optical_frame">
+  <link name="camera_left_optical_link">
     </link>
   <joint name="camera_left_optical_joint" type="fixed">
     <origin xyz="0.0211999999999999 0 0" rpy="0 1.5707963267948966 0" />
     <parent link="camera_left_link" />
-    <child link="cameras_head_left_camera_optical_frame" />
+    <child link="camera_left_optical_link" />
     <axis xyz="0 0 0" />
   </joint>
@@ -273,10 +273,10 @@
     <axis xyz="0 0 0" />
   </joint>
-  <link name="cameras_head_center_camera_optical_frame">
+  <link name="camera_center_optical_link">
     </link>
   <joint name="camera_center_optical_joint" type="fixed">
     <origin xyz="0.00170000000000003 0 0" rpy="3.141592653589793 -1.5707963267948966 0" />
     <parent link="camera_center_link" />
-    <child link="cameras_head_center_camera_optical_frame" />
+    <child link="camera_center_optical_link" />
     <axis xyz="0 0 0" />
   </joint>

Commit message: Flipped center-camera rotation about z axis, and put back camera_link rotations

File: stretch4_urdf/SE4_francis/xacro/stretch_main.xacro (robot description, xacro)
@@ -226,5 +226,5 @@
     </link>
   <joint name="camera_right_joint" type="fixed">
-    <origin xyz="0.171840602787894 0.0230000000000032 -0.0157566987072475" rpy="0 0.820304748437337 0" />
+    <origin xyz="0.171840602787894 0.0230000000000032 -0.0157566987072475" rpy="1.5707963267949 0.820304748437337 0" />
     <parent link="head_link" />
     <child link="camera_right_link" />
@@ -234,5 +234,5 @@
     </link>
   <joint name="camera_right_optical_joint" type="fixed">
-    <origin xyz="0.0212000000000001 0 0" rpy="3.141592653589793 -1.5707963267948966 0" />
+    <origin xyz="0.0212000000000001 0 0" rpy="-1.5707963267949 0 -1.5707963267949" />
     <parent link="camera_right_link" />
     <child link="camera_right_optical_link" />
@@ -247,5 +247,5 @@
     </link>
   <joint name="camera_left_joint" type="fixed">
-    <origin xyz="0.171840602787895 0.173 -0.0157566987072475" rpy="0 0.820304748437337 0" />
+    <origin xyz="0.171840602787895 0.173 -0.0157566987072475" rpy="-1.5707963267949 0.820304748437337 0" />
     <parent link="head_link" />
     <child link="camera_left_link" />
@@ -255,5 +255,5 @@
     </link>
   <joint name="camera_left_optical_joint" type="fixed">
-    <origin xyz="0.0211999999999999 0 0" rpy="0 1.5707963267948966 0" />
+    <origin xyz="0.0211999999999999 0 0" rpy="-1.5707963267949 0 -1.5707963267949" />
     <parent link="camera_left_link" />
     <child link="camera_left_optical_link" />
@@ -268,5 +268,5 @@
     </link>
   <joint name="camera_center_joint" type="fixed">
-    <origin xyz="0.177245603402412 0.0980000000000004 -0.0239069097938973" rpy="0 0.610865238198018 0" />
+    <origin xyz="0.177245603402412 0.0980000000000004 -0.0239069097938973" rpy="1.5707963267949 0.610865238198018 0" />
     <parent link="head_link" />
     <child link="camera_center_link" />
@@ -276,5 +276,5 @@
     </link>
   <joint name="camera_center_optical_joint" type="fixed">
-    <origin xyz="0.00170000000000003 0 0" rpy="3.141592653589793 -1.5707963267948966 0" />
+    <origin xyz="0.00170000000000003 0 0" rpy="-1.5707963267949 0 -1.5707963267949" />
     <parent link="camera_center_link" />
     <child link="camera_center_optical_link" />

Commit message: New camera optical frame definitions (#40)
* New camera optical frame definitions

* Rename optical links to use expected luxonis names

* I think I understand opencv now

* docs

* docs

* docs

* docs

* Changed the optical frame links back to their original urdf names instead of the luxonis ros names

* Flipped center-camera rotation about z axis, and put back camera_link rotations

---------

Co-authored-by: Shehab Attia <sattia@hello-robot.com>

File: stretch4_urdf/SE4_francis/xacro/stretch_main.xacro (robot description, xacro)
@@ -268,5 +268,5 @@
     </link>
   <joint name="camera_center_joint" type="fixed">
-    <origin xyz="0.177245603402412 0.0980000000000004 -0.0239069097938973" rpy="-1.5707963267949 0.610865238198018 0" />
+    <origin xyz="0.177245603402412 0.0980000000000004 -0.0239069097938973" rpy="1.5707963267949 0.610865238198018 0" />
     <parent link="head_link" />
     <child link="camera_center_link" />

Commit message: Removed collision from arm_l0

File: stretch4_urdf/SE4_francis/xacro/stretch_main.xacro (robot description, xacro)
@@ -339,9 +339,4 @@
   </joint>
   <link name="arm_l0_link">
-    <inertial>
-      <origin xyz="-0.0316222581318624 -0.0397927105745811 0.0182872881301621" rpy="0 0 0" />
-      <mass value="2.95349364666659" />
-      <inertia ixx="0.0117399464230091" ixy="0.000875437380496019" ixz="0.000164784888522662" iyy="0.0102748963241433" iyz="-0.00101918054718661" izz="0.0139841484528854" />
-    </inertial>
     <visual>
       <origin xyz="0 0 0" rpy="0 0 0" />
@@ -353,10 +348,4 @@
       </material>
     </visual>
-    <collision name="arm_l0_collision_link">
-      <origin xyz="0 0 0" rpy="0 0 0" />
-      <geometry>
-        <mesh filename="$(arg model_mesh_dir)/arm_l0_collision_link.STL" />
-      </geometry>
-    </collision>
   </link>
   <joint name="arm_l0_joint" type="fixed">

Commit message: arm_l0 mesh is now separated from lift mesh

File: stretch4_urdf/SE4_francis/xacro/stretch_main.xacro (robot description, xacro)
@@ -309,60 +309,114 @@
     <axis xyz="0 0 0" />
   </joint>
-  <link name="lift_link">
-    <inertial>
-      <origin xyz="-0.0148722581318624 0.0596072894254191 0.00542773918494432" rpy="0 0 0" />
-      <mass value="2.95349364666659" />
-      <inertia ixx="0.0117399464230091" ixy="0.000875437380496019" ixz="0.000164784888522662" iyy="0.0102748963241433" iyz="-0.00101918054718661" izz="0.0139841484528854" />
-    </inertial>
-    <visual>
-      <origin xyz="0 0 0" rpy="0 0 0" />
-      <geometry>
-        <mesh filename="$(arg model_mesh_dir)/lift_link.STL" />
-      </geometry>
-      <material name="">
-        <color rgba="0.752941176470588 0.752941176470588 0.752941176470588 1" />
-      </material>
-    </visual>
-    <collision name="lift_collision_link">
-      <origin xyz="0 0 0" rpy="0 0 0" />
-      <geometry>
-        <mesh filename="$(arg model_mesh_dir)/lift_collision_link.STL" />
-      </geometry>
-    </collision>
-  </link>
-  <joint name="lift_joint" type="prismatic">
-    <origin xyz="0 -0.00140000000000005 0.241" rpy="0 0 0" />
-    <parent link="mast_link" />
-    <child link="lift_link" />
-    <axis xyz="0 0 1" />
-    <limit lower="0" upper="1.2" effort="0" velocity="0" />
-  </joint>
-  <link name="arm_l0_link">
-    <inertial>
-      <origin xyz="-0.0316222581318624 -0.0397927105745811 0.0182872881301621" rpy="0 0 0" />
-      <mass value="2.95349364666659" />
-      <inertia ixx="0.0117399464230091" ixy="0.000875437380496019" ixz="0.000164784888522662" iyy="0.0102748963241433" iyz="-0.00101918054718661" izz="0.0139841484528854" />
-    </inertial>
-    <visual>
-      <origin xyz="0 0 0" rpy="0 0 0" />
-      <geometry>
-        <mesh filename="$(arg model_mesh_dir)/arm_l0_link.STL" />
-      </geometry>
-      <material name="">
-        <color rgba="0.752941176470588 0.752941176470588 0.752941176470588 1" />
-      </material>
-    </visual>
-    <collision name="arm_l0_collision_link">
-      <origin xyz="0 0 0" rpy="0 0 0" />
-      <geometry>
-        <mesh filename="$(arg model_mesh_dir)/arm_l0_collision_link.STL" />
-      </geometry>
-    </collision>
-  </link>
-  <joint name="arm_l0_joint" type="fixed">
-    <origin xyz="0.01675 0.0994000000000002 -0.0128595489452177" rpy="0 0 0" />
-    <parent link="lift_link" />
-    <child link="arm_l0_link" />
-    <axis xyz="0 0 0" />
+  <link
+    name="lift_link">
+    <inertial>
+      <origin
+        xyz="-0.0233092431932026 0.0564207351004435 0.00671885423980972"
+        rpy="0 0 0" />
+      <mass
+        value="2.73451670567963" />
+      <inertia
+        ixx="0.011466385458167"
+        ixy="0.000875437380496019"
+        ixz="0.000164784751492084"
+        iyy="0.00956613602133992"
+        iyz="-0.00101918054718662"
+        izz="0.0132435850196122" />
+    </inertial>
+    <visual>
+      <origin
+        xyz="0 0 0"
+        rpy="0 0 0" />
+      <geometry>
+        <mesh
+          filename="$(arg model_mesh_dir)/lift_link.STL" />
+      </geometry>
+      <material
+        name="">
+        <color
+          rgba="0.752941176470588 0.752941176470588 0.752941176470588 1" />
+      </material>
+    </visual>
+    <collision>
+      <origin
+        xyz="0 0 0"
+        rpy="0 0 0" />
+      <geometry>
+        <mesh
+          filename="$(arg model_mesh_dir)/lift_collision_link.STL" />
+      </geometry>
+    </collision>
+  </link>
+  <joint
+    name="lift_joint"
+    type="prismatic">
+    <origin
+      xyz="0 -0.00140000000000005 0.241"
+      rpy="0 0 0" />
+    <parent
+      link="mast_link" />
+    <child
+      link="lift_link" />
+    <axis
+      xyz="0 0 1" />
+    <limit
+      lower="0"
+      upper="1.2"
+      effort="0"
+      velocity="0" />
+  </joint>
+  <link
+    name="arm_l0_link">
+    <inertial>
+      <origin
+        xyz="0.0737362170199923 -1.74714644470479E-16 0.0021642403308329"
+        rpy="0 0 0" />
+      <mass
+        value="0.218976940986966" />
+      <inertia
+        ixx="0.000273560964842063"
+        ixy="-6.26647189332688E-19"
+        ixz="1.37030578374227E-10"
+        iyy="0.000708760302803403"
+        iyz="-8.66022937939828E-20"
+        izz="0.000740563433273204" />
+    </inertial>
+    <visual>
+      <origin
+        xyz="0 0 0"
+        rpy="0 0 0" />
+      <geometry>
+        <mesh
+          filename="$(arg model_mesh_dir)/arm_l0_link.STL" />
+      </geometry>
+      <material
+        name="">
+        <color
+          rgba="0.752941176470588 0.752941176470588 0.752941176470588 1" />
+      </material>
+    </visual>
+    <collision>
+      <origin
+        xyz="0 0 0"
+        rpy="0 0 0" />
+      <geometry>
+        <mesh
+          filename="$(arg model_mesh_dir)/arm_l0_collision_link.STL" />
+      </geometry>
+    </collision>
+  </link>
+  <joint
+    name="arm_l0_joint"
+    type="fixed">
+    <origin
+      xyz="0.01675 0.0994000000000002 -0.0128595489452177"
+      rpy="0 0 0" />
+    <parent
+      link="lift_link" />
+    <child
+      link="arm_l0_link" />
+    <axis
+      xyz="0 0 0" />
   </joint>
   <link name="arm_l1_link">
