Commit message: fix the direction in which the joints move

File: stretch4_urdf/SE4_tools/eoa_wrist_dw4_tool_pg4/eoa_wrist_dw4_tool_pg4.urdf (robot description, URDF)
Before this commit: robot URDF_DALI_ASSEM_Parallel_Jaw_Gripper_V2, 7 links, 6 joints
Joints:
- joint finger_left_joint: axis 0 0 1 -> -1 0 0
- joint finger_right_joint: axis 0 0 1 -> 1 0 0

Commit message: Rename pg4 grasp link so it matches sg4

File: stretch4_urdf/SE4_tools/eoa_wrist_dw4_tool_pg4/eoa_wrist_dw4_tool_pg4.urdf (robot description, URDF)
Before this commit: robot URDF_FRANCIS_ASSEM_Parallel_Jaw_Gripper_V3, 7 links, 6 joints
Links:
- removed link grasp_frame_link
- added link grasp_center_link, mass 6.54498469497874E-05; collision mesh filename=$(arg tool_mesh_dir)/grasp_center_collision_link.STL; visual mesh filename=$(arg tool_mesh_dir)/grasp_center_link.STL
Joints:
- removed joint grasp_frame_joint
- added joint grasp_center_joint: type fixed, parent pjg_body_link, child grasp_center_link, origin xyz=0.166855269271506 0 0 rpy=0 0 0, axis 0 0 0

Commit message: Removed collision and visualization from grasp_center_link. Renamed PJG grasp_frame_link -> grasp_center_link

File: stretch4_urdf/SE4_tools/eoa_wrist_dw4_tool_pg4/eoa_wrist_dw4_tool_pg4.urdf (robot description, URDF)
Before this commit: robot URDF_FRANCIS_ASSEM_Parallel_Jaw_Gripper_V3, 7 links, 6 joints
Links:
- removed link grasp_frame_link
- added link grasp_center_link
Joints:
- removed joint grasp_frame_joint
- added joint grasp_center_joint: type fixed, parent pjg_body_link, child grasp_center_link, origin xyz=0.166855269271506 0 0 rpy=0 0 0, axis 0 0 0

File: stretch4_urdf/SE4_tools/eoa_wrist_dw4_tool_sg4/eoa_wrist_dw4_tool_sg4.urdf (robot description, URDF)
Before this commit: robot URDF_FRANCIS_ASSEM_Stretch_Gripper_V6, 8 links, 7 joints
Links:
- link grasp_center_link: mass 6.54498469497874E-05 -> None; geometry 
