Commit message: Update generated robot models with velocity and effort limits from robot params

File: stretch4_urdf/SE4_tools/eoa_wrist_dw4_tool_pg4/eoa_wrist_dw4_tool_pg4.urdf (robot description, URDF)
Before this commit: robot URDF_FRANCIS_ASSEM_Parallel_Jaw_Gripper_V3, 7 links, 6 joints
Joints:
- joint finger_left_joint: limit lower=-0.04 upper=0 effort=0 velocity=0 -> lower=-0.04 upper=0 effort=20.0 velocity=6.0
- joint finger_right_joint: limit lower=-0.04 upper=0 effort=0 velocity=0 -> lower=-0.04 upper=0 effort=20.0 velocity=6.0

File: stretch4_urdf/SE4_tools/eoa_wrist_dw4_tool_sg4/eoa_wrist_dw4_tool_sg4.urdf (robot description, URDF)
Before this commit: robot URDF_FRANCIS_ASSEM_Stretch_Gripper_V6, 8 links, 7 joints
Joints:
- joint gripper_finger_left_joint: limit lower=0 upper=0.5 effort=0 velocity=0 -> lower=0 upper=0.5 effort=20.0 velocity=6.0
- joint gripper_finger_right_joint: limit lower=0 upper=0.5 effort=0 velocity=0 -> lower=0 upper=0.5 effort=20.0 velocity=6.0

Commit message: Updated URDF for the PJG v2

File: stretch4_urdf/SE4_tools/eoa_wrist_dw4_tool_pg4/eoa_wrist_dw4_tool_pg4.urdf (robot description, URDF)
Before this commit: robot URDF_FRANCIS_ASSEM_Parallel_Jaw_Gripper_V3, 7 links, 6 joints
Links:
- removed link grasp_center_link
- added link grasp_frame_link
- link aruco_fingertip_left_link: mass 0.000123521493853863 -> 0.000132188497698026
- link aruco_fingertip_right_link: mass 0.000123521493853863 -> 0.000132188497698027
- link finger_left_link: mass 0.0246520031759402 -> 0.0284304473699516
- link finger_right_link: mass 0.0246520031759402 -> 0.0284304100497672
- link pjg_body_link: mass 0.381434237025036 -> 0.392020130813208
Joints:
- removed joint grasp_center_joint
- added joint grasp_frame_joint: type fixed, parent pjg_body_link, child grasp_frame_link, origin xyz=0.166875269271506 0 0 rpy=0 0 0, axis 0 0 0
- joint aruco_fingertip_left_joint: origin xyz=-0.01225 -0.0670400491408859 0.0170000000000008 rpy=0 0 0 -> xyz=-0.0132499999999998 -0.0705221070892628 0.0197477319374844 rpy=0.174532925199433 0 0
- joint aruco_fingertip_right_joint: origin xyz=-0.0122499999999998 0.0670400491408858 0.0169999999999987 rpy=0 0 -3.14159265358979 -> xyz=-0.01325 0.0705221070892628 0.0197477319374859 rpy=0.174532925199433 0 -3.14159265358979
- joint finger_left_joint: limit lower=-0.04 upper=0 effort=20.0 velocity=6.0 -> lower=-0.0385 upper=0 effort=0 velocity=0; origin xyz=0.166855269271506 0 0 rpy=0 0 -1.5707963267949 -> xyz=0.16688 -0.0005 0 rpy=0 0 -1.5708
- joint finger_right_joint: limit lower=-0.04 upper=0 effort=20.0 velocity=6.0 -> lower=-0.0385 upper=0 effort=0 velocity=0; origin xyz=0.166855269271506 0 0 rpy=0 0 1.5707963267949 -> xyz=0.16688 0.0005 0 rpy=0 0 1.5708

Commit message: grasp_frame_link -> grasp_center_link

File: stretch4_urdf/SE4_tools/eoa_wrist_dw4_tool_pg4/eoa_wrist_dw4_tool_pg4.urdf (robot description, URDF)
Before this commit: robot URDF_FRANCIS_ASSEM_Parallel_Jaw_Gripper_V4, 7 links, 6 joints
Links:
- removed link grasp_frame_link
- added link grasp_center_link
Joints:
- removed joint grasp_frame_joint
- added joint grasp_center_joint: type fixed, parent pjg_body_link, child grasp_center_link, origin xyz=0.166875269271506 0 0 rpy=0 0 0, axis 0 0 0
