Commit message: Misc fixes

File: stretch4_urdf/SE4OMNI_francis/xacro/stretch_main.xacro (robot description, xacro)
@@ -251,4 +251,32 @@
     <axis xyz="0 0 0" />
   </joint>
+  <link name="mast_link">
+    <inertial>
+      <origin xyz="2.77555756156289E-17 -0.00165282700965368 0.815" rpy="0 0 0" />
+      <mass value="10.8924861076487" />
+      <inertia ixx="1.96276319417158" ixy="-4.74739862687269E-18" ixz="-1.24526930733894E-16" iyy="1.96594229514087" iyz="-1.7420761023809E-18" izz="0.00577661764276332" />
+    </inertial>
+    <visual>
+      <origin xyz="0 0 0" rpy="0 0 0" />
+      <geometry>
+        <mesh filename="$(arg model_mesh_dir)/mast_link.STL" />
+      </geometry>
+      <material name="">
+        <color rgba="0.752941176470588 0.752941176470588 0.752941176470588 1" />
+      </material>
+    </visual>
+    <collision name="mast_collision_link">
+      <origin xyz="0 0 0" rpy="0 0 0" />
+      <geometry>
+        <mesh filename="$(arg model_mesh_dir)/mast_collision_link.STL" />
+      </geometry>
+    </collision>
+  </link>
+  <joint name="mast_joint" type="fixed">
+    <origin xyz="-0.0930000000000002 -0.0979999999999998 0.00400000430816486" rpy="0 0 0" />
+    <parent link="base_link" />
+    <child link="mast_link" />
+    <axis xyz="0 0 0" />
+  </joint>
   <link name="wheel_2_link">
     <inertial>

File: stretch4_urdf/SE4OMNI_tools/whole_arm_nil/whole_arm_nil.urdf (robot description, URDF)
Before this commit: robot stretch_tool_tablet, 1 links, 0 joints
Joints:
- added joint nop_joint: type fixed, parent base_link, child nop
